File: electronics/local_oscillator_test/local_oscillator_test.sch (KiCad schematic (older format))
At the start: 2 parts, among them U1 CE3520K3

Commit message: Something resembling an impulse
Connections:
- wire segments 3 -> 6
Changed lines of the file:
@@
 $EndComp
 Wire Wire Line
-	2850 3300 2550 3300
+	2850 3300 2650 3300
 Wire Wire Line
-	2550 3000 3100 3000
+	2550 3000 2650 3000
 Wire Wire Line
 	3100 3000 3100 3100
@@
 $EndComp
 $Comp
-L power:GND #PWR?
+L power:GND #PWR0101
 U 1 1 5E8F6624
 P 3100 3500
-F 0 "#PWR?" H 3100 3500 30  0001 C CNN
+F 0 "#PWR0101" H 3100 3500 30  0001 C CNN
 F 1 "GND" H 3100 3430 30  0001 C CNN
 F 2 "" H 3100 3500 50  0001 C CNN
@@
 $EndComp
 $Comp
-L power:GND #PWR?
+L power:GND #PWR0102
 U 1 1 5E8F663A
 P 3200 3500
-F 0 "#PWR?" H 3200 3500 30  0001 C CNN
+F 0 "#PWR0102" H 3200 3500 30  0001 C CNN
 F 1 "GND" H 3200 3430 30  0001 C CNN
 F 2 "" H 3200 3500 50  0001 C CNN
@@
 Text Label 2600 3300 0    50   ~ 0
 GATE
+Wire Wire Line
+	2650 3000 2650 3300
+Connection ~ 2650 3000
+Wire Wire Line
+	2650 3000 3100 3000
+Connection ~ 2650 3300
+Wire Wire Line
+	2650 3300 2550 3300
 $EndSCHEMATC

Commit message: LO works!
Parts:
- added L?: INDUCTOR-0402-3.9NH, 0402, symbol SparkFun-Coils:INDUCTOR-0402-3.9NH
- C1: value 1pF -> 4pF
Connections:
- wire segments 6 -> 3
Changed lines of the file:
@@
 	1    0    0    -1
 $EndComp
-Wire Wire Line
-	2850 3300 2650 3300
-Wire Wire Line
-	2550 3000 2650 3000
-Wire Wire Line
-	3100 3000 3100 3100
 $Comp
 L SparkFun-Capacitors:1.0UF-0402-16V-10% C1
@@
 P 2550 3100
 F 0 "C1" H 2442 3055 45  0000 R CNN
-F 1 "1pF" H 2750 3050 45  0000 R CNN
+F 1 "4pF" H 2750 3050 45  0000 R CNN
 F 2 "0402" H 2550 3350 20  0001 C CNN
 F 3 "" H 2550 3100 50  0001 C CNN
@@
 L power:GND #PWR0101
 U 1 1 5E8F6624
-P 3100 3500
-F 0 "#PWR0101" H 3100 3500 30  0001 C CNN
-F 1 "GND" H 3100 3430 30  0001 C CNN
-F 2 "" H 3100 3500 50  0001 C CNN
-F 3 "" H 3100 3500 50  0001 C CNN
-	1    3100 3500
+P 3100 3900
+F 0 "#PWR0101" H 3100 3900 30  0001 C CNN
+F 1 "GND" H 3100 3830 30  0001 C CNN
+F 2 "" H 3100 3900 50  0001 C CNN
+F 3 "" H 3100 3900 50  0001 C CNN
+	1    3100 3900
 	1    0    0    -1
 $EndComp
@@
 L power:GND #PWR0102
 U 1 1 5E8F663A
-P 3200 3500
-F 0 "#PWR0102" H 3200 3500 30  0001 C CNN
-F 1 "GND" H 3200 3430 30  0001 C CNN
-F 2 "" H 3200 3500 50  0001 C CNN
-F 3 "" H 3200 3500 50  0001 C CNN
-	1    3200 3500
+P 3200 3900
+F 0 "#PWR0102" H 3200 3900 30  0001 C CNN
+F 1 "GND" H 3200 3830 30  0001 C CNN
+F 2 "" H 3200 3900 50  0001 C CNN
+F 3 "" H 3200 3900 50  0001 C CNN
+	1    3200 3900
 	1    0    0    -1
 $EndComp
@@
 GATE
 Wire Wire Line
-	2650 3000 2650 3300
-Connection ~ 2650 3000
+	2550 3300 2850 3300
 Wire Wire Line
-	2650 3000 3100 3000
-Connection ~ 2650 3300
+	3100 2850 3100 3100
+$Comp
+L SparkFun-Coils:INDUCTOR-0402-3.9NH L?
+U 1 1 5E90A22B
+P 3200 3700
+F 0 "L?" H 3253 3700 45  0000 L CNN
+F 1 "INDUCTOR-0402-3.9NH" H 3253 3711 45  0001 L CNN
+F 2 "0402" H 3200 3950 20  0001 C CNN
+F 3 "" H 3200 3700 50  0001 C CNN
+F 4 "NDUC-13457" H 3253 3658 60  0001 L CNN "Field4"
+	1    3200 3700
+	-1   0    0    1
+$EndComp
 Wire Wire Line
-	2650 3300 2550 3300
+	3100 3900 3200 3900
+Connection ~ 3200 3900
 $EndSCHEMATC

Commit message: Vortexer
Parts:
- added C2: 0.1 uF, 0402, symbol SparkFun-Capacitors:1.0UF-0402-16V-10%
- added C3: 10 uF, 0402, symbol SparkFun-Capacitors:1.0UF-0402-16V-10%
- added L2: INDUCTOR-0402-3.9NH, symbol SparkFun-Coils:INDUCTOR-0402-3.9NH
- L1: renamed from L?; footprint 0402 -> (none)
Connections:
- wire segments 3 -> 10
Changed lines of the file:
@@
 	3100 2850 3100 3100
 $Comp
-L SparkFun-Coils:INDUCTOR-0402-3.9NH L?
+L SparkFun-Coils:INDUCTOR-0402-3.9NH L1
 U 1 1 5E90A22B
 P 3200 3700
-F 0 "L?" H 3253 3700 45  0000 L CNN
+F 0 "L1" H 3159 3700 45  0000 R CNN
 F 1 "INDUCTOR-0402-3.9NH" H 3253 3711 45  0001 L CNN
-F 2 "0402" H 3200 3950 20  0001 C CNN
+F 2 "" H 3200 3950 20  0001 C CNN
 F 3 "" H 3200 3700 50  0001 C CNN
 F 4 "NDUC-13457" H 3253 3658 60  0001 L CNN "Field4"
@@
 	3100 3900 3200 3900
 Connection ~ 3200 3900
+Wire Wire Line
+	2550 3000 2550 2850
+Wire Wire Line
+	2550 2850 3100 2850
+$Comp
+L SparkFun-Capacitors:1.0UF-0402-16V-10% C2
+U 1 1 5E925DB1
+P 3650 3050
+F 0 "C2" H 3758 3142 45  0000 L CNN
+F 1 "0.1 uF" H 3758 3058 45  0000 L CNN
+F 2 "0402" H 3650 3300 20  0001 C CNN
+F 3 "" H 3650 3050 50  0001 C CNN
+F 4 "CAP-12417" H 3758 3016 60  0001 L CNN "Field4"
+	1    3650 3050
+	1    0    0    -1
+$EndComp
+$Comp
+L SparkFun-Capacitors:1.0UF-0402-16V-10% C3
+U 1 1 5E925F97
+P 4000 3050
+F 0 "C3" H 4108 3142 45  0000 L CNN
+F 1 "10 uF" H 4108 3058 45  0000 L CNN
+F 2 "0402" H 4000 3300 20  0001 C CNN
+F 3 "" H 4000 3050 50  0001 C CNN
+F 4 "CAP-12417" H 4108 3016 60  0001 L CNN "Field4"
+	1    4000 3050
+	1    0    0    -1
+$EndComp
+Wire Wire Line
+	4000 2850 3650 2850
+$Comp
+L SparkFun-Coils:INDUCTOR-0402-3.9NH L2
+U 1 1 5E926007
+P 3400 2850
+F 0 "L2" V 3495 2850 45  0000 C CNN
+F 1 "INDUCTOR-0402-3.9NH" H 3453 2861 45  0001 L CNN
+F 2 "" H 3400 3100 20  0001 C CNN
+F 3 "" H 3400 2850 50  0001 C CNN
+F 4 "NDUC-13457" H 3453 2808 60  0001 L CNN "Field4"
+	1    3400 2850
+	0    -1   -1   0
+$EndComp
+Wire Wire Line
+	3650 2850 3600 2850
+Connection ~ 3650 2850
+Wire Wire Line
+	3200 2850 3100 2850
+Connection ~ 3100 2850
+$Comp
+L power:GND #PWR0103
+U 1 1 5E9261AD
+P 3650 3150
+F 0 "#PWR0103" H 3650 3150 30  0001 C CNN
+F 1 "GND" H 3650 3080 30  0001 C CNN
+F 2 "" H 3650 3150 50  0001 C CNN
+F 3 "" H 3650 3150 50  0001 C CNN
+	1    3650 3150
+	1    0    0    -1
+$EndComp
+$Comp
+L power:GND #PWR0104
+U 1 1 5E9261C4
+P 4000 3150
+F 0 "#PWR0104" H 4000 3150 30  0001 C CNN
+F 1 "GND" H 4000 3080 30  0001 C CNN
+F 2 "" H 4000 3150 50  0001 C CNN
+F 3 "" H 4000 3150 50  0001 C CNN
+	1    4000 3150
+	1    0    0    -1
+$EndComp
+Wire Wire Line
+	3100 3500 3200 3500
+Connection ~ 3200 3500
+Wire Wire Line
+	3200 2850 3600 2850
+Connection ~ 3200 2850
+Connection ~ 3600 2850
 $EndSCHEMATC

Commit message: Phage propagation!
Connections:
- wire segments 10 -> 11
Other:
- note added: "Transmission line with 50 R impedance and 180 deg phase shift"
Changed lines of the file:
@@
 Connection ~ 3200 2850
 Connection ~ 3600 2850
+Wire Wire Line
+	3200 3500 3200 3900
+Text Notes 1050 2450 0    50   ~ 0
+Transmission line with 50 R impedance and 180 deg phase shift
 $EndSCHEMATC
