File: electronics/kicad/downconverter/image_reject_filter.kicad_pcb (KiCad board)
At the start: 2 copper layers, 0 parts

Commit message: Crashed and burned there, but I think we're back.
Parts:
- added MS1: microstrip_line, MLIN, F.Cu at (2.96, 5.59)
- added MS11: microstrip_tee, MTEE, F.Cu at (11.1, 5.59)
- added MS12: microstrip_tee, MTEE, F.Cu at (21.2, 5.59)
- added MS2: microstrip_line, MLIN, F.Cu at (5.21, 2.96)
- added MS3: microstrip_line, MLIN, F.Cu at (7.45, 5.59)
- added MS4: microstrip_line, MLIN, F.Cu at (11.1, 2.96)
- added MS5: microstrip_line, MLIN, F.Cu at (14.7, 5.59)
- added MS6: microstrip_line, MLIN, F.Cu at (21.2, 2.96)
- added MS7: microstrip_line, MLIN, F.Cu at (27.8, 5.59)
- added MS8: microstrip_tee, MTEE, F.Cu at (5.21, 5.59)
Changed lines of the file:
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@@
-(kicad_pcb (version 20171130) (host pcbnew 5.0.0)
+(kicad_pcb (version 20171130) (host pcbnew 5.0.1-33cea8e~67~ubuntu18.04.1)
   (general
     (thickness 1.6)
@@
     (uvia_drill 0.1)
   )
+  (module MLIN (layer F.Cu)
+    (at 21.247 2.963 90)
+    (fp_text reference MS6 (at 0 0.5) (layer F.SilkS)
+      (effects (font (size 0.25 0.25) (thickness 0.05)))
+    )
+    (fp_text value microstrip_line (at 0 -0.5) (layer F.Fab)
+      (effects (font (size 0.25 0.25) (thickness 0.05)))
+    )
+    (fp_poly (pts
+      (xy -1.963 4.588)
+      (xy 1.963 4.588)
+      (xy 1.963 -4.588)
+      (xy -1.963 -4.588)
+      ) (layer F.Cu) (width 0)
+    )
+  )
+  (module MLIN (layer F.Cu)
+    (at 27.798 5.588 0)
+    (fp_text reference MS7 (at 0 0.5) (layer F.SilkS)
+      (effects (font (size 0.25 0.25) (thickness 0.05)))
+    )
+    (fp_text value microstrip_line (at 0 -0.5) (layer F.Fab)
+      (effects (font (size 0.25 0.25) (thickness 0.05)))
+    )
+    (fp_poly (pts
+      (xy -1.963 0.662)
+      (xy 1.963 0.662)
+      (xy 1.963 -0.662)
+      (xy -1.963 -0.662)
+      ) (layer F.Cu) (width 0)
+    )
+  )
+  (module MLIN (layer F.Cu)
+    (at 7.449 5.588 0)
+    (fp_text reference MS3 (at 0 0.5) (layer F.SilkS)
+      (effects (font (size 0.25 0.25) (thickness 0.05)))
+    )
+    (fp_text value microstrip_line (at 0 -0.5) (layer F.Fab)
+      (effects (font (size 0.25 0.25) (thickness 0.05)))
+    )
+    (fp_poly (pts
+      (xy -1.963 0.662)
+      (xy 1.963 0.662)
+      (xy 1.963 -0.662)
+      (xy -1.963 -0.662)
+      ) (layer F.Cu) (width 0)
+    )
+  )
+  (module MTEE (layer F.Cu)
+    (at 11.0725 5.588 180)
+    (fp_text reference MS11 (at 0 0.5) (layer F.SilkS)
+      (effects (font (size 0.25 0.25) (thickness 0.05)))
+    )
+    (fp_text value microstrip_tee (at 0 -0.5) (layer F.Fab)
+      (effects (font (size 0.25 0.25) (thickness 0.05)))
+    )
+    (fp_poly (pts
+      (xy -1.6605 0.662)
+      (xy 1.6605 0.662)
+      (xy 1.6605 -0.662)
+      (xy 0 -0.662)
+      (xy 0 -0)
+      (xy -1.6605 -0)
+      ) (layer F.Cu) (width 0)
+    )
+  )
+  (module MTEE (layer F.Cu)
+    (at 21.247 5.588 180)
+    (fp_text reference MS12 (at 0 0.5) (layer F.SilkS)
+      (effects (font (size 0.25 0.25) (thickness 0.05)))
+    )
+    (fp_text value microstrip_tee (at 0 -0.5) (layer F.Fab)
+      (effects (font (size 0.25 0.25) (thickness 0.05)))
+    )
+    (fp_poly (pts
+      (xy -4.588 0.662)
+      (xy 4.588 0.662)
+      (xy 4.588 -0.662)
+      (xy 0 -0.662)
+      (xy 0 -0)
+      (xy -4.588 -0)
+      ) (layer F.Cu) (width 0)
+    )
+  )
+  (module MLIN (layer F.Cu)
+    (at 14.696 5.588 0)
+    (fp_text reference MS5 (at 0 0.5) (layer F.SilkS)
+      (effects (font (size 0.25 0.25) (thickness 0.05)))
+    )
+    (fp_text value microstrip_line (at 0 -0.5) (layer F.Fab)
+      (effects (font (size 0.25 0.25) (thickness 0.05)))
+    )
+    (fp_poly (pts
+      (xy -1.963 0.662)
+      (xy 1.963 0.662)
+      (xy 1.963 -0.662)
+      (xy -1.963 -0.662)
+      ) (layer F.Cu) (width 0)
+    )
+  )
+  (module MLIN (layer F.Cu)
+    (at 2.963 5.588 0)
+    (fp_text reference MS1 (at 0 0.5) (layer F.SilkS)
+      (effects (font (size 0.25 0.25) (thickness 0.05)))
+    )
+    (fp_text value microstrip_line (at 0 -0.5) (layer F.Fab)
+      (effects (font (size 0.25 0.25) (thickness 0.05)))
+    )
+    (fp_poly (pts
+      (xy -1.963 0.662)
+      (xy 1.963 0.662)
+      (xy 1.963 -0.662)
+      (xy -1.963 -0.662)
+      ) (layer F.Cu) (width 0)
+    )
+  )
+  (module MTEE (layer F.Cu)
+    (at 5.206 5.588 180)
+    (fp_text reference MS8 (at 0 0.5) (layer F.SilkS)
+      (effects (font (size 0.25 0.25) (thickness 0.05)))
+    )
+    (fp_text value microstrip_tee (at 0 -0.5) (layer F.Fab)
+      (effects (font (size 0.25 0.25) (thickness 0.05)))
+    )
+    (fp_poly (pts
+      (xy -0.28 0.662)
+      (xy 0.28 0.662)
+      (xy 0.28 -0.662)
+      (xy 0 -0.662)
+      (xy 0 -0)
+      (xy -0.28 -0)
+      ) (layer F.Cu) (width 0)
+    )
+  )
+  (module MLIN (layer F.Cu)
+    (at 5.206 2.963 90)
+    (fp_text reference MS2 (at 0 0.5) (layer F.SilkS)
+      (effects (font (size 0.25 0.25) (thickness 0.05)))
+    )
+    (fp_text value microstrip_line (at 0 -0.5) (layer F.Fab)
+      (effects (font (size 0.25 0.25) (thickness 0.05)))
+    )
+    (fp_poly (pts
+      (xy -1.963 0.28035)
+      (xy 1.963 0.28035)
+      (xy 1.963 -0.28035)
+      (xy -1.963 -0.28035)
+      ) (layer F.Cu) (width 0)
+    )
+  )
+  (module MLIN (layer F.Cu)
+    (at 11.0725 2.963 90)
+    (fp_text reference MS4 (at 0 0.5) (layer F.SilkS)
+      (effects (font (size 0.25 0.25) (thickness 0.05)))
+    )
+    (fp_text value microstrip_line (at 0 -0.5) (layer F.Fab)
+      (effects (font (size 0.25 0.25) (thickness 0.05)))
+    )
+    (fp_poly (pts
+      (xy -1.963 1.6605)
+      (xy 1.963 1.6605)
+      (xy 1.963 -1.6605)
+      (xy -1.963 -1.6605)
+      ) (layer F.Cu) (width 0)
+    )
+  )
 )
