File: electronics/kicad/downconverter/downconverter.kicad_pcb (KiCad board)
At the start: 2 copper layers, 28 parts

Commit message: Crashed and burned there, but I think we're back.
Parts:
- removed MS1, MS13, MS14, MS15, MS18, MS2, MS21, MS22, MS23, MS24, MS25, MS28, MS3, MS30, MS31, MS4, MS5, MS6, MS7: microstrip_line, MLIN
- removed MS11, MS12, MS16, MS17, MS20, MS26, MS27, MS29, MS8: microstrip_tee, MTEE
- added J1: CONN_01, TestPoint:TestPoint_Pad_1.0x1.0mm, F.Cu at (46.5, 40.2)
- added J2: CONN_01, TestPoint:TestPoint_Pad_1.0x1.0mm, F.Cu at (60.2, 40.2)
- added J3: CONN_01, TestPoint:TestPoint_Pad_1.0x1.0mm, F.Cu at (55.8, 60.8)
- added U1: HMC220B, Package_SO:MSOP-8-1EP_3x3mm_P0.65mm_EP1.68x1.88mm, F.Cu at (53.5, 51.0)
Routing:
- net GND: track 0.00 -> 18.7 mm, vias 0 -> 2
- net Net-(J1-Pad1): track 0.00 -> 11.2 mm
- net Net-(J2-Pad1): track 0.00 -> 11.1 mm
- net Net-(J3-Pad1): track 0.00 -> 8.12 mm
- added copper zone on F.Cu, net GND

Commit message: Downconverter board!
Routing:
- net GND: track 18.7 -> 19.5 mm
Changed lines of the file:
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@@
     (thickness 1.6)
     (drawings 0)
-    (tracks 19)
+    (tracks 21)
     (zones 0)
     (modules 4)
@@
     (last_trace_width 0.25)
     (trace_clearance 0.2)
-    (zone_clearance 0.1)
+    (zone_clearance 3)
     (zone_45_only no)
     (trace_min 0.2)
@@
     (pad_drill 0.762)
     (pad_to_mask_clearance 0.2)
-    (aux_axis_origin 0 0)
+    (aux_axis_origin 39.7 37.8)
     (visible_elements FFFFFF7F)
     (pcbplotparams
-      (layerselection 0x010fc_ffffffff)
+      (layerselection 0x00000_7fffffff)
       (usegerberextensions false)
       (usegerberattributes false)
@@
       (outputformat 1)
       (mirror false)
-      (drillshape 1)
+      (drillshape 0)
       (scaleselection 1)
-      (outputdirectory ""))
+      (outputdirectory "CAD/"))
   )
   (net 0 "")
@@
     )
   )
+  (segment (start 53.4 43.1) (end 53.4 42.4) (width 0.25) (layer F.Cu) (net 1))
   (segment (start 50.7 50.675) (end 50.275 51.1) (width 0.25) (layer F.Cu) (net 1))
   (segment (start 51.395 50.675) (end 50.7 50.675) (width 0.25) (layer F.Cu) (net 1))
@@
   (via (at 49.9 51.1) (size 0.8) (drill 0.4) (layers F.Cu B.Cu) (net 1))
   (segment (start 51.395 51.975) (end 51.395 51.325) (width 0.25) (layer F.Cu) (net 1))
+  (segment (start 53.4 43.1) (end 53.5 43.2) (width 0.25) (layer F.Cu) (net 1))
   (segment (start 55.75 53.7) (end 55.75 52.625) (width 1.487) (layer F.Cu) (net 3))
   (segment (start 60.25 43.675) (end 60.25 40.25) (width 1.487) (layer F.Cu) (net 4))
