File: electronics/kicad/downconverter/downconverter.kicad_pcb (KiCad board)
At the start: 2 copper layers, 4 parts, among them J1 CONN_01, J2 CONN_01, J3 CONN_01, U1 HMC220B

Commit message: Spectrum analyzer progress
Parts:
- added J4: CONSMA001-SMD-G, digikey-footprints:RF_SMA_Receptical_Vertical_CONSMA001-SMD-G, F.Cu at (55.8, 59.2)
- moved J1 5.51 mm to (42.2, 43.8)
Routing:
- net Net-(J1-Pad1): track 11.2 -> 12.0 mm
- net GND: track 19.5 -> 20.2 mm, vias 2 -> 3
Changed lines of the file:
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@@
-(kicad_pcb (version 20171130) (host pcbnew 5.0.0)
+(kicad_pcb (version 20171130) (host pcbnew 5.1.5+dfsg1-2~bpo9+1)
   (general
     (thickness 1.6)
     (drawings 0)
-    (tracks 21)
+    (tracks 22)
     (zones 0)
-    (modules 4)
-    (nets 5)
+    (modules 5)
+    (nets 7)
   )
   (page A4)
@@
     (zone_45_only no)
     (trace_min 0.2)
-    (segment_width 0.2)
-    (edge_width 0.15)
     (via_size 0.8)
     (via_drill 0.4)
@@
     (uvia_min_size 0.2)
     (uvia_min_drill 0.1)
+    (edge_width 0.15)
+    (segment_width 0.2)
     (pcb_text_width 0.3)
     (pcb_text_size 1.5 1.5)
@@
   (net 3 "Net-(J3-Pad1)")
   (net 4 "Net-(J2-Pad1)")
+  (net 5 "Net-(J4-Pad2)")
+  (net 6 "Net-(J4-Pad1)")
   (net_class Default "This is the default net class."
     (clearance 0.2)
@@
     (add_net "Net-(J2-Pad1)")
     (add_net "Net-(J3-Pad1)")
+    (add_net "Net-(J4-Pad1)")
+    (add_net "Net-(J4-Pad2)")
+  )
+  (module digikey-footprints:RF_SMA_Receptical_Vertical_CONSMA001-SMD-G (layer F.Cu)
+    (at 55.75 59.25)
+    (fp_text reference J4 (at 0.3 -4.8) (layer F.SilkS)
+      (effects (font (size 1 1) (thickness 0.15)))
+    )
+    (fp_text value CONSMA001-SMD-G (at 0.01778 5.15112) (layer F.Fab)
+      (effects (font (size 1 1) (thickness 0.15)))
+    )
+    (fp_line (start -3.88 -3.88) (end 3.88 -3.88) (layer F.Fab) (width 0.1))
+    (fp_line (start 3.88 -3.88) (end 3.88 3.88) (layer F.Fab) (width 0.1))
+    (fp_line (start 3.88 3.88) (end -3.88 3.88) (layer F.Fab) (width 0.1))
+    (fp_line (start -3.88 -3.88) (end -3.88 3.88) (layer F.Fab) (width 0.1))
+    (fp_line (start -4.13 -4.13) (end 4.13 -4.13) (layer F.CrtYd) (width 0.05))
+    (fp_line (start 4.13 -4.13) (end 4.13 4.13) (layer F.CrtYd) (width 0.05))
+    (fp_line (start 4.13 4.13) (end -4.13 4.13) (layer F.CrtYd) (width 0.05))
+    (fp_line (start -4.13 4.13) (end -4.13 -4.13) (layer F.CrtYd) (width 0.05))
+    (fp_line (start 4 -4) (end 4 -3.525) (layer F.SilkS) (width 0.1))
+    (fp_line (start 3.4 -4) (end 4 -4) (layer F.SilkS) (width 0.1))
+    (fp_line (start -4 -4) (end -4 -3.35) (layer F.SilkS) (width 0.1))
+    (fp_line (start -3.2 -4) (end -4 -4) (layer F.SilkS) (width 0.1))
+    (fp_line (start 4 4) (end 3.425 4) (layer F.SilkS) (width 0.1))
+    (fp_line (start 4 3.475) (end 4 4) (layer F.SilkS) (width 0.1))
+    (fp_line (start -4 4) (end -4 3.55) (layer F.SilkS) (width 0.1))
+    (fp_line (start -3.5 4) (end -4 4) (layer F.SilkS) (width 0.1))
+    (fp_line (start -3.6 4) (end -3.4 4) (layer F.SilkS) (width 0.1))
+    (fp_text user %R (at -0.075 -2.675) (layer F.Fab)
+      (effects (font (size 0.75 0.75) (thickness 0.075)))
+    )
+    (pad 2 smd circle (at 0.025 -0.1) (size 2.05 2.05) (layers F.Cu F.Paste F.Mask)
+      (net 5 "Net-(J4-Pad2)"))
+    (pad 1 smd rect (at 2.55 2.55) (size 1.5 1.5) (layers F.Cu F.Paste F.Mask)
+      (net 6 "Net-(J4-Pad1)"))
+    (pad 1 smd rect (at 2.55 -2.55) (size 1.5 1.5) (layers F.Cu F.Paste F.Mask)
+      (net 6 "Net-(J4-Pad1)"))
+    (pad 1 smd rect (at -2.55 -2.55) (size 1.5 1.5) (layers F.Cu F.Paste F.Mask)
+      (net 6 "Net-(J4-Pad1)"))
+    (pad 1 smd rect (at -2.55 2.55) (size 1.5 1.5) (layers F.Cu F.Paste F.Mask)
+      (net 6 "Net-(J4-Pad1)"))
   )
   (module TestPoint:TestPoint_Pad_1.0x1.0mm (layer F.Cu)
@@
   )
   (module TestPoint:TestPoint_Pad_1.0x1.0mm (layer F.Cu)
-    (at 46.5 40.25 90)
+    (at 42.25 43.75 90)
     (descr "SMD rectangular pad as test Point, square 1.0mm side length")
     (tags "test point SMD pad rectangle square")
@@
     )
   )
-  (segment (start 53.4 43.1) (end 53.4 42.4) (width 0.25) (layer F.Cu) (net 1))
+  (via (at 53.5 42.75) (size 0.8) (drill 0.4) (layers F.Cu B.Cu) (net 1))
   (segment (start 50.7 50.675) (end 50.275 51.1) (width 0.25) (layer F.Cu) (net 1))
   (segment (start 51.395 50.675) (end 50.7 50.675) (width 0.25) (layer F.Cu) (net 1))
@@
   (via (at 49.9 51.1) (size 0.8) (drill 0.4) (layers F.Cu B.Cu) (net 1))
   (segment (start 51.395 51.975) (end 51.395 51.325) (width 0.25) (layer F.Cu) (net 1))
-  (segment (start 53.4 43.1) (end 53.5 43.2) (width 0.25) (layer F.Cu) (net 1))
+  (segment (start 53.100001 42.350001) (end 52.149999 42.350001) (width 0.25) (layer F.Cu) (net 1))
+  (segment (start 53.5 42.75) (end 53.100001 42.350001) (width 0.25) (layer F.Cu) (net 1))
+  (segment (start 51.25 49.5) (end 51.25 48.425) (width 1.487) (layer F.Cu) (net 2))
+  (segment (start 51.25 48.425) (end 46.5 43.675) (width 1.487) (layer F.Cu) (net 2))
+  (segment (start 46.5 43.675) (end 42.325 43.675) (width 1.5) (layer F.Cu) (net 2))
   (segment (start 55.75 53.7) (end 55.75 52.625) (width 1.487) (layer F.Cu) (net 3))
+  (segment (start 55.75 53.7) (end 55.75 60.75) (width 1.487) (layer F.Cu) (net 3))
   (segment (start 60.25 43.675) (end 60.25 40.25) (width 1.487) (layer F.Cu) (net 4))
   (segment (start 55.75 49.5) (end 55.75 48.425) (width 1.487) (layer F.Cu) (net 4))
-  (segment (start 51.25 49.5) (end 51.25 48.425) (width 1.487) (layer F.Cu) (net 2))
-  (segment (start 46.5 43.675) (end 46.5 40.25) (width 1.487) (layer F.Cu) (net 2))
-  (segment (start 51.25 48.425) (end 46.5 43.675) (width 1.487) (layer F.Cu) (net 2))
-  (segment (start 55.75 53.7) (end 55.75 60.75) (width 1.487) (layer F.Cu) (net 3))
   (segment (start 55.75 48.175) (end 60.25 43.675) (width 1.487) (layer F.Cu) (net 4))
   (segment (start 55.75 48.425) (end 55.75 48.175) (width 0.25) (layer F.Cu) (net 4))
