File: electronics/kicad/downconverter/downconverter.sch (KiCad schematic (older format))
At the start: 1 part, among them U1 HMC220B

Commit message: Crashed and burned there, but I think we're back.
Parts:
- added J1, J2, J3: CONN_01, TestPoint:TestPoint_Pad_1.0x1.0mm, symbol SparkFun-Connectors:CONN_01
- U1: footprint (none) -> Package_SO:MSOP-8-1EP_3x3mm_P0.65mm_EP1.68x1.88mm
Connections:
- net GND: now also U1.4 (NC)
- net at U1.1 (LO): now also J1.1
- net at U1.5 (IF): now also J3.1
- net at U1.8 (RF): now also J2.1
Changed lines of the file:
@@
 F 0 "U1" H 3450 2875 50  0000 C CNN
 F 1 "HMC220B" H 3450 2784 50  0000 C CNN
-F 2 "" H 3450 2250 50  0001 C CNN
+F 2 "Package_SO:MSOP-8-1EP_3x3mm_P0.65mm_EP1.68x1.88mm" H 3450 2250 50  0001 C CNN
 F 3 "" H 3450 2250 50  0001 C CNN
 	1    3450 2800
@@
 	0    -1   -1   0
 $EndComp
+Wire Wire Line
+	3150 2950 2850 2950
+Wire Wire Line
+	4000 3250 3750 3250
+$Comp
+L SparkFun-Connectors:CONN_01 J1
+U 1 1 5EA728FD
+P 2750 2950
+F 0 "J1" H 2706 3260 45  0000 C CNN
+F 1 "CONN_01" H 2706 3176 45  0000 C CNN
+F 2 "TestPoint:TestPoint_Pad_1.0x1.0mm" H 2750 3150 20  0001 C CNN
+F 3 "" H 2750 2950 50  0001 C CNN
+F 4 "XXX-00000" H 2706 3081 60  0000 C CNN "Field4"
+	1    2750 2950
+	1    0    0    -1
+$EndComp
+$Comp
+L SparkFun-Connectors:CONN_01 J3
+U 1 1 5EA72B6A
+P 4100 3250
+F 0 "J3" H 4057 2940 45  0000 C CNN
+F 1 "CONN_01" H 4057 3024 45  0000 C CNN
+F 2 "TestPoint:TestPoint_Pad_1.0x1.0mm" H 4100 3450 20  0001 C CNN
+F 3 "" H 4100 3250 50  0001 C CNN
+F 4 "XXX-00000" H 4057 3119 60  0000 C CNN "Field4"
+	1    4100 3250
+	-1   0    0    1
+$EndComp
+$Comp
+L SparkFun-Connectors:CONN_01 J2
+U 1 1 5EA729ED
+P 3850 2950
+F 0 "J2" H 3807 2640 45  0000 C CNN
+F 1 "CONN_01" H 3807 2724 45  0000 C CNN
+F 2 "TestPoint:TestPoint_Pad_1.0x1.0mm" H 3850 3150 20  0001 C CNN
+F 3 "" H 3850 2950 50  0001 C CNN
+F 4 "XXX-00000" H 3807 2819 60  0000 C CNN "Field4"
+	1    3850 2950
+	-1   0    0    1
+$EndComp
+$Comp
+L power:GND #PWR?
+U 1 1 5EA7383E
+P 3150 3200
+F 0 "#PWR?" H 3150 3200 30  0001 C CNN
+F 1 "GND" H 3150 3130 30  0001 C CNN
+F 2 "" H 3150 3200 50  0001 C CNN
+F 3 "" H 3150 3200 50  0001 C CNN
+	1    3150 3200
+	0    1    1    0
+$EndComp
+$Comp
+L power:GND #PWR?
+U 1 1 5EA73896
+P 3150 3250
+F 0 "#PWR?" H 3150 3250 30  0001 C CNN
+F 1 "GND" H 3150 3180 30  0001 C CNN
+F 2 "" H 3150 3250 50  0001 C CNN
+F 3 "" H 3150 3250 50  0001 C CNN
+	1    3150 3250
+	0    1    1    0
+$EndComp
 $EndSCHEMATC

Commit message: Spectrum analyzer progress
Parts:
- added J?: CONSMA001-SMD-G, digikey-footprints:RF_SMA_Receptical_Vertical_CONSMA001-SMD-G, symbol dk_Coaxial-Connectors-RF:CONSMA001-SMD-G
Changed lines of the file:
@@
 EESchema Schematic File Version 4
-EELAYER 26 0
+EELAYER 30 0
 EELAYER END
 $Descr A4 11693 8268
@@
 $EndComp
 $Comp
-L power:GND #PWR?
+L power:GND #PWR0106
 U 1 1 5EA7383E
 P 3150 3200
-F 0 "#PWR?" H 3150 3200 30  0001 C CNN
+F 0 "#PWR0106" H 3150 3200 30  0001 C CNN
 F 1 "GND" H 3150 3130 30  0001 C CNN
 F 2 "" H 3150 3200 50  0001 C CNN
@@
 $EndComp
 $Comp
-L power:GND #PWR?
+L power:GND #PWR0107
 U 1 1 5EA73896
 P 3150 3250
-F 0 "#PWR?" H 3150 3250 30  0001 C CNN
+F 0 "#PWR0107" H 3150 3250 30  0001 C CNN
 F 1 "GND" H 3150 3180 30  0001 C CNN
 F 2 "" H 3150 3250 50  0001 C CNN
@@
 	0    1    1    0
 $EndComp
+$Comp
+L dk_Coaxial-Connectors-RF:CONSMA001-SMD-G J?
+U 1 1 5F1B7015
+P 4550 4200
+F 0 "J?" H 4628 4447 60  0000 C CNN
+F 1 "CONSMA001-SMD-G" H 4628 4341 60  0000 C CNN
+F 2 "digikey-footprints:RF_SMA_Receptical_Vertical_CONSMA001-SMD-G" H 4750 4400 60  0001 L CNN
+F 3 "https://linxtechnologies.com/wp/wp-content/uploads/consma001-smd-g.pdf" H 4750 4500 60  0001 L CNN
+F 4 "CONSMA001-SMD-G-ND" H 4750 4600 60  0001 L CNN "Digi-Key_PN"
+F 5 "CONSMA001-SMD-G" H 4750 4700 60  0001 L CNN "MPN"
+F 6 "Connectors, Interconnects" H 4750 4800 60  0001 L CNN "Category"
+F 7 "Coaxial Connectors (RF)" H 4750 4900 60  0001 L CNN "Family"
+F 8 "https://linxtechnologies.com/wp/wp-content/uploads/consma001-smd-g.pdf" H 4750 5000 60  0001 L CNN "DK_Datasheet_Link"
+F 9 "/product-detail/en/linx-technologies-inc/CONSMA001-SMD-G/CONSMA001-SMD-G-ND/4496569" H 4750 5100 60  0001 L CNN "DK_Detail_Page"
+F 10 "CONN SMA RCPT STR 50 OHM SMD" H 4750 5200 60  0001 L CNN "Description"
+F 11 "Linx Technologies Inc." H 4750 5300 60  0001 L CNN "Manufacturer"
+F 12 "Active" H 4750 5400 60  0001 L CNN "Status"
+	1    4550 4200
+	1    0    0    -1
+$EndComp
 $EndSCHEMATC
