File: electronics/qucs/image_reject_filter.kicad_pcb (KiCad board)
At the start: 2 copper layers, 28 parts

Commit message: Crashed and burned there, but I think we're back.
Parts:
- removed MS13, MS14, MS15, MS18, MS21, MS22, MS23, MS24, MS25, MS28, MS30, MS31: microstrip_line, MLIN
- removed MS16, MS17, MS20, MS26, MS27, MS29: microstrip_tee, MTEE
