File: electronics/kicad/local_oscillator/local_oscillator.sch (KiCad schematic (older format))
At the start: 2 parts

Commit message: Feedback loop looks great now
Connections:
- wire segments 0 -> 3
Changed lines of the file:
@@
 	1    0    0    -1
 $EndComp
+Wire Wire Line
+	5650 4450 4650 4450
+Wire Wire Line
+	4650 4450 4650 4550
+Wire Wire Line
+	4650 4850 5650 4850
 $EndSCHEMATC

Commit message: Largely working feedback loop, but going to try phase shifter.
Parts:
- added D?: D_Capacitance, symbol Device:D_Capacitance
Connections:
- net labels added: GND
- wire segments 3 -> 11
Other:
- note added: "Strap tightly down to GND"
Changed lines of the file:
@@
 L SparkFun-Capacitors:10NF-0603-50V-10% C?
 U 1 1 5EAA1C32
-P 4650 4750
-F 0 "C?" H 4758 4842 45  0000 L CNN
-F 1 "4.7 pF" H 4758 4758 45  0000 L CNN
-F 2 "0603" H 4650 5000 20  0001 C CNN
-F 3 "" H 4650 4750 50  0001 C CNN
-F 4 "" H 4758 4716 60  0000 L CNN "Field4"
-	1    4650 4750
+P 4750 4050
+F 0 "C?" H 4858 4142 45  0000 L CNN
+F 1 "4.7 pF" H 4858 4058 45  0000 L CNN
+F 2 "0603" H 4750 4300 20  0001 C CNN
+F 3 "" H 4750 4050 50  0001 C CNN
+F 4 "" H 4858 4016 60  0000 L CNN "Field4"
+	1    4750 4050
 	1    0    0    -1
 $EndComp
 Wire Wire Line
-	5650 4450 4650 4450
+	4750 3750 4750 3850
+$Comp
+L Device:D_Capacitance D?
+U 1 1 5EAB375D
+P 4750 4450
+F 0 "D?" V 4704 4529 50  0000 L CNN
+F 1 "D_Capacitance" V 4795 4529 50  0000 L CNN
+F 2 "" H 4750 4450 50  0001 C CNN
+F 3 "~" H 4750 4450 50  0001 C CNN
+	1    4750 4450
+	0    1    1    0
+$EndComp
 Wire Wire Line
-	4650 4450 4650 4550
+	5650 4850 5750 4850
+Connection ~ 5650 4850
+$Comp
+L power:GND #PWR?
+U 1 1 5EAB3B29
+P 5750 4850
+F 0 "#PWR?" H 5750 4850 30  0001 C CNN
+F 1 "GND" H 5750 4780 30  0001 C CNN
+F 2 "" H 5750 4850 50  0001 C CNN
+F 3 "" H 5750 4850 50  0001 C CNN
+	1    5750 4850
+	1    0    0    -1
+$EndComp
+Connection ~ 5750 4850
+$Comp
+L power:GND #PWR?
+U 1 1 5EAB3B63
+P 5650 4850
+F 0 "#PWR?" H 5650 4850 30  0001 C CNN
+F 1 "GND" H 5650 4780 30  0001 C CNN
+F 2 "" H 5650 4850 50  0001 C CNN
+F 3 "" H 5650 4850 50  0001 C CNN
+	1    5650 4850
+	1    0    0    -1
+$EndComp
+Text Notes 5350 5100 0    50   ~ 0
+Strap tightly down to GND
 Wire Wire Line
-	4650 4850 5650 4850
+	5400 4650 4750 4650
+Wire Wire Line
+	4750 4150 4750 4300
+Wire Wire Line
+	5650 4450 5650 3750
+Wire Wire Line
+	5650 3750 4750 3750
+Connection ~ 4750 4300
+Wire Wire Line
+	4750 4300 4750 4350
+Wire Wire Line
+	4750 4650 4750 4600
+Wire Wire Line
+	4750 4300 4450 4300
+Wire Wire Line
+	4450 4300 4450 4650
+Wire Wire Line
+	4450 4650 4750 4650
+Connection ~ 4750 4650
 $EndSCHEMATC

Commit message: PIN diode Fb loop actually working
Parts:
- removed C?: 4.7 pF, 0603, symbol SparkFun-Capacitors:10NF-0603-50V-10%
- removed D?: D_Capacitance, symbol Device:D_Capacitance
- added C? (x3): 4.7 pF, 0402, symbol SparkFun-Capacitors:6PF-0402-50V-0.5%
- added D?: DIODE, symbol w_device:DIODE
Connections:
- net labels added: VCC, VCO
- wire segments 11 -> 12
Changed lines of the file:
@@
 	1    0    0    -1
-$EndComp
-$Comp
-L SparkFun-Capacitors:10NF-0603-50V-10% C?
-U 1 1 5EAA1C32
-P 4750 4050
-F 0 "C?" H 4858 4142 45  0000 L CNN
-F 1 "4.7 pF" H 4858 4058 45  0000 L CNN
-F 2 "0603" H 4750 4300 20  0001 C CNN
-F 3 "" H 4750 4050 50  0001 C CNN
-F 4 "" H 4858 4016 60  0000 L CNN "Field4"
-	1    4750 4050
-	1    0    0    -1
-$EndComp
-Wire Wire Line
-	4750 3750 4750 3850
-$Comp
-L Device:D_Capacitance D?
-U 1 1 5EAB375D
-P 4750 4450
-F 0 "D?" V 4704 4529 50  0000 L CNN
-F 1 "D_Capacitance" V 4795 4529 50  0000 L CNN
-F 2 "" H 4750 4450 50  0001 C CNN
-F 3 "~" H 4750 4450 50  0001 C CNN
-	1    4750 4450
-	0    1    1    0
 $EndComp
 Wire Wire Line
@@
 Strap tightly down to GND
 Wire Wire Line
-	5400 4650 4750 4650
+	4750 4000 4450 4000
 Wire Wire Line
-	4750 4150 4750 4300
+	4450 4350 4750 4350
+Connection ~ 4750 4350
+$Comp
+L w_device:DIODE D?
+U 1 1 5EAC4B0B
+P 4750 4200
+F 0 "D?" H 4775 4367 40  0000 C CNN
+F 1 "DIODE" H 4775 4291 40  0000 C CNN
+F 2 "" H 4750 4200 60  0000 C CNN
+F 3 "" H 4750 4200 60  0000 C CNN
+	1    4750 4200
+	0    -1   -1   0
+$EndComp
 Wire Wire Line
-	5650 4450 5650 3750
+	4750 4000 4750 4100
 Wire Wire Line
-	5650 3750 4750 3750
-Connection ~ 4750 4300
+	4750 4250 4750 4350
+$Comp
+L SparkFun-Capacitors:6PF-0402-50V-0.5% C?
+U 1 1 5EAC501D
+P 4750 4450
+F 0 "C?" H 4643 4458 45  0000 R CNN
+F 1 "4.7 pF" H 4643 4542 45  0000 R CNN
+F 2 "0402" H 4750 4700 20  0001 C CNN
+F 3 "" H 4750 4450 50  0001 C CNN
+F 4 "" H 4643 4584 60  0000 R CNN "Field4"
+	1    4750 4450
+	1    0    0    1
+$EndComp
 Wire Wire Line
-	4750 4300 4750 4350
+	4750 4650 5400 4650
 Wire Wire Line
-	4750 4650 4750 4600
+	4750 3700 5350 3700
 Wire Wire Line
-	4750 4300 4450 4300
+	5650 3700 5650 4450
+$Comp
+L SparkFun-Capacitors:6PF-0402-50V-0.5% C?
+U 1 1 5EAC5CD0
+P 4450 4100
+F 0 "C?" H 4343 4108 45  0000 R CNN
+F 1 "4.7 pF" H 4343 4192 45  0000 R CNN
+F 2 "0402" H 4450 4350 20  0001 C CNN
+F 3 "" H 4450 4100 50  0001 C CNN
+F 4 "" H 4343 4234 60  0000 R CNN "Field4"
+	1    4450 4100
+	1    0    0    1
+$EndComp
 Wire Wire Line
-	4450 4300 4450 4650
+	4450 4350 4450 4300
+Connection ~ 4750 4000
 Wire Wire Line
-	4450 4650 4750 4650
-Connection ~ 4750 4650
+	5350 3700 5350 3200
+Connection ~ 5350 3700
+Wire Wire Line
+	5350 3700 5650 3700
+$Comp
+L power:VCC #PWR?
+U 1 1 5EAC60CF
+P 5350 3200
+F 0 "#PWR?" H 5350 3300 30  0001 C CNN
+F 1 "VCC" H 5353 3328 30  0000 C CNN
+F 2 "" H 5350 3200 50  0001 C CNN
+F 3 "" H 5350 3200 50  0001 C CNN
+	1    5350 3200
+	1    0    0    -1
+$EndComp
+Text GLabel 4350 4350 0    50   Input ~ 0
+VCO
+Wire Wire Line
+	4350 4350 4450 4350
+Connection ~ 4450 4350
+$Comp
+L SparkFun-Capacitors:6PF-0402-50V-0.5% C?
+U 1 1 5EAC63C2
+P 4750 3800
+F 0 "C?" H 4643 3808 45  0000 R CNN
+F 1 "4.7 pF" H 4643 3892 45  0000 R CNN
+F 2 "0402" H 4750 4050 20  0001 C CNN
+F 3 "" H 4750 3800 50  0001 C CNN
+F 4 "" H 4643 3934 60  0000 R CNN "Field4"
+	1    4750 3800
+	1    0    0    1
+$EndComp
 $EndSCHEMATC

Commit message: Upgrading kicad
Parts:
- added TP1: SMA, TestPoint:TestPoint_Pad_1.5x1.5mm, symbol SparkFun-Connectors:TEST-POINT3X4
- D1: renamed from D?; footprint (none) -> Diode_SMD:D_SOD-523
- U1: renamed from U?; footprint (none) -> 0xDBFB7:4-Micro-X
- gave numbers to parts that had none: 3
Connections:
- wire segments 12 -> 13
Changed lines of the file:
@@
 $EndDescr
 $Comp
-L 0xDBFB7:CE3520K3 U?
+L 0xDBFB7:CE3520K3 U1
 U 1 1 5EAA1A86
 P 5650 4650
-F 0 "U?" H 5791 4696 50  0000 L CNN
+F 0 "U1" H 5791 4696 50  0000 L CNN
 F 1 "CE3520K3" H 5791 4605 50  0000 L CNN
-F 2 "" H 5650 4650 50  0001 C CNN
+F 2 "0xDBFB7:4-Micro-X" H 5650 4650 50  0001 C CNN
 F 3 "" H 5650 4650 50  0001 C CNN
 	1    5650 4650
@@
 Connection ~ 5650 4850
 $Comp
-L power:GND #PWR?
+L power:GND #PWR0101
 U 1 1 5EAB3B29
 P 5750 4850
-F 0 "#PWR?" H 5750 4850 30  0001 C CNN
+F 0 "#PWR0101" H 5750 4850 30  0001 C CNN
 F 1 "GND" H 5750 4780 30  0001 C CNN
 F 2 "" H 5750 4850 50  0001 C CNN
@@
 Connection ~ 5750 4850
 $Comp
-L power:GND #PWR?
+L power:GND #PWR0102
 U 1 1 5EAB3B63
 P 5650 4850
-F 0 "#PWR?" H 5650 4850 30  0001 C CNN
+F 0 "#PWR0102" H 5650 4850 30  0001 C CNN
 F 1 "GND" H 5650 4780 30  0001 C CNN
 F 2 "" H 5650 4850 50  0001 C CNN
@@
 Connection ~ 4750 4350
 $Comp
-L w_device:DIODE D?
+L w_device:DIODE D1
 U 1 1 5EAC4B0B
 P 4750 4200
-F 0 "D?" H 4775 4367 40  0000 C CNN
-F 1 "DIODE" H 4775 4291 40  0000 C CNN
-F 2 "" H 4750 4200 60  0000 C CNN
+F 0 "D1" V 4866 4147 40  0000 R CNN
+F 1 "DIODE" V 4790 4147 40  0000 R CNN
+F 2 "Diode_SMD:D_SOD-523" V 4699 4147 60  0000 R CNN
 F 3 "" H 4750 4200 60  0000 C CNN
 	1    4750 4200
@@
 	4750 4250 4750 4350
 $Comp
-L SparkFun-Capacitors:6PF-0402-50V-0.5% C?
+L SparkFun-Capacitors:6PF-0402-50V-0.5% C3
 U 1 1 5EAC501D
 P 4750 4450
-F 0 "C?" H 4643 4458 45  0000 R CNN
+F 0 "C3" H 4643 4458 45  0000 R CNN
 F 1 "4.7 pF" H 4643 4542 45  0000 R CNN
 F 2 "0402" H 4750 4700 20  0001 C CNN
@@
 	4750 3700 5350 3700
 Wire Wire Line
-	5650 3700 5650 4450
+	5650 3700 5650 3850
 $Comp
-L SparkFun-Capacitors:6PF-0402-50V-0.5% C?
+L SparkFun-Capacitors:6PF-0402-50V-0.5% C1
 U 1 1 5EAC5CD0
 P 4450 4100
-F 0 "C?" H 4343 4108 45  0000 R CNN
+F 0 "C1" H 4343 4108 45  0000 R CNN
 F 1 "4.7 pF" H 4343 4192 45  0000 R CNN
 F 2 "0402" H 4450 4350 20  0001 C CNN
@@
 	5350 3700 5650 3700
 $Comp
-L power:VCC #PWR?
+L power:VCC #PWR0103
 U 1 1 5EAC60CF
 P 5350 3200
-F 0 "#PWR?" H 5350 3300 30  0001 C CNN
+F 0 "#PWR0103" H 5350 3300 30  0001 C CNN
 F 1 "VCC" H 5353 3328 30  0000 C CNN
 F 2 "" H 5350 3200 50  0001 C CNN
@@
 Connection ~ 4450 4350
 $Comp
-L SparkFun-Capacitors:6PF-0402-50V-0.5% C?
+L SparkFun-Capacitors:6PF-0402-50V-0.5% C2
 U 1 1 5EAC63C2
 P 4750 3800
-F 0 "C?" H 4643 3808 45  0000 R CNN
+F 0 "C2" H 4643 3808 45  0000 R CNN
 F 1 "4.7 pF" H 4643 3892 45  0000 R CNN
 F 2 "0402" H 4750 4050 20  0001 C CNN
@@
 	1    0    0    1
 $EndComp
+$Comp
+L SparkFun-Connectors:TEST-POINT3X4 TP1
+U 1 1 5EAC6ADE
+P 5650 3850
+F 0 "TP1" H 5714 4034 45  0000 C CNN
+F 1 "SMA" H 5714 3950 45  0000 C CNN
+F 2 "TestPoint:TestPoint_Pad_1.5x1.5mm" H 5650 4050 20  0001 C CNN
+F 3 "" H 5650 3850 50  0001 C CNN
+F 4 "" H 5714 3961 60  0000 C CNN "Field4"
+	1    5650 3850
+	1    0    0    -1
+$EndComp
+Connection ~ 5650 3850
+Wire Wire Line
+	5650 3850 5650 4450
 $EndSCHEMATC

Commit message: Somewhat altered fb loop
Parts:
- removed D1: DIODE, Diode_SMD:D_SOD-523, symbol w_device:DIODE
- added C4, C5: 0.1 uF, 0603, symbol SparkFun-Capacitors:4.7UF0603
- added C6: 4.7 pF, 0402, symbol SparkFun-Capacitors:6PF-0402-50V-0.5%
- added D1: D, Diode_SMD:D_SOD-523, symbol Device:D
- added P1, P2, P3: TestPoint:TestPoint_Pad_1.5x1.5mm, TestPoint:TestPoint_Pad_1.5x1.5mm, symbol conn:CONN_1
Connections:
- net labels added: GATE, VCO1, VCO2
- net labels removed: VCO
- wire segments 13 -> 16
Other:
- moved on the sheet: TP1
Changed lines of the file:
@@
 EESchema Schematic File Version 4
-EELAYER 26 0
+EELAYER 30 0
 EELAYER END
 $Descr A4 11693 8268
@@
 Strap tightly down to GND
 Wire Wire Line
-	4750 4000 4450 4000
-Wire Wire Line
 	4450 4350 4750 4350
 Connection ~ 4750 4350
-$Comp
-L w_device:DIODE D1
-U 1 1 5EAC4B0B
-P 4750 4200
-F 0 "D1" V 4866 4147 40  0000 R CNN
-F 1 "DIODE" V 4790 4147 40  0000 R CNN
-F 2 "Diode_SMD:D_SOD-523" V 4699 4147 60  0000 R CNN
-F 3 "" H 4750 4200 60  0000 C CNN
-	1    4750 4200
-	0    -1   -1   0
-$EndComp
-Wire Wire Line
-	4750 4000 4750 4100
-Wire Wire Line
-	4750 4250 4750 4350
 $Comp
 L SparkFun-Capacitors:6PF-0402-50V-0.5% C3
@@
 Wire Wire Line
 	4750 3700 5350 3700
-Wire Wire Line
-	5650 3700 5650 3850
 $Comp
 L SparkFun-Capacitors:6PF-0402-50V-0.5% C1
@@
 Wire Wire Line
 	4450 4350 4450 4300
-Connection ~ 4750 4000
 Wire Wire Line
 	5350 3700 5350 3200
@@
 	5350 3700 5650 3700
 $Comp
-L power:VCC #PWR0103
-U 1 1 5EAC60CF
-P 5350 3200
-F 0 "#PWR0103" H 5350 3300 30  0001 C CNN
-F 1 "VCC" H 5353 3328 30  0000 C CNN
-F 2 "" H 5350 3200 50  0001 C CNN
-F 3 "" H 5350 3200 50  0001 C CNN
-	1    5350 3200
-	1    0    0    -1
-$EndComp
-Text GLabel 4350 4350 0    50   Input ~ 0
-VCO
-Wire Wire Line
-	4350 4350 4450 4350
+L conn:CONN_1 P1
+U 1 1 5EAD0C12
+P 4250 4000
+F 0 "P1" H 4183 3903 40  0000 C CNN
+F 1 "TestPoint:TestPoint_Pad_1.5x1.5mm" H 4200 4040 30  0001 C CNN
+F 2 "TestPoint:TestPoint_Pad_1.5x1.5mm" H 4250 4000 50  0001 C CNN
+F 3 "" H 4250 4000 50  0001 C CNN
+	1    4250 4000
+	-1   0    0    1
+$EndComp
+$Comp
+L conn:CONN_1 P2
+U 1 1 5EAD28FF
+P 4300 4350
+F 0 "P2" H 4233 4253 40  0000 C CNN
+F 1 "TestPoint:TestPoint_Pad_1.5x1.5mm" H 4250 4390 30  0001 C CNN
+F 2 "TestPoint:TestPoint_Pad_1.5x1.5mm" H 4300 4350 50  0001 C CNN
+F 3 "" H 4300 4350 50  0001 C CNN
+	1    4300 4350
+	-1   0    0    1
+$EndComp
 Connection ~ 4450 4350
 $Comp
+L conn:CONN_1 P3
+U 1 1 5EAD30DB
+P 5200 3200
+F 0 "P3" H 5133 3103 40  0000 C CNN
+F 1 "TestPoint:TestPoint_Pad_1.5x1.5mm" H 5150 3240 30  0001 C CNN
+F 2 "TestPoint:TestPoint_Pad_1.5x1.5mm" H 5200 3200 50  0001 C CNN
+F 3 "" H 5200 3200 50  0001 C CNN
+	1    5200 3200
+	-1   0    0    1
+$EndComp
+$Comp
+L SparkFun-Capacitors:4.7UF0603 C4
+U 1 1 5EADDFB9
+P 6100 3900
+F 0 "C4" H 6208 4045 45  0000 L CNN
+F 1 "0.1 uF" H 6208 3961 45  0000 L CNN
+F 2 "0603" H 6100 4150 20  0001 C CNN
+F 3 "" H 6100 3900 50  0001 C CNN
+F 4 "CAP-08280" V 6208 3866 60  0001 L CNN "Field4"
+	1    6100 3900
+	1    0    0    -1
+$EndComp
+Wire Wire Line
+	5650 3700 6100 3700
+Connection ~ 5650 3700
+$Comp
+L power:GND #PWR0103
+U 1 1 5EAE14E0
+P 6100 4000
+F 0 "#PWR0103" H 6100 4000 30  0001 C CNN
+F 1 "GND" H 6100 3930 30  0001 C CNN
+F 2 "" H 6100 4000 50  0001 C CNN
+F 3 "" H 6100 4000 50  0001 C CNN
+	1    6100 4000
+	1    0    0    -1
+$EndComp
+$Comp
+L SparkFun-Capacitors:4.7UF0603 C5
+U 1 1 5EAE2635
+P 6550 3900
+F 0 "C5" H 6658 4045 45  0000 L CNN
+F 1 "0.1 uF" H 6658 3961 45  0000 L CNN
+F 2 "0603" H 6550 4150 20  0001 C CNN
+F 3 "" H 6550 3900 50  0001 C CNN
+F 4 "CAP-08280" V 6658 3866 60  0001 L CNN "Field4"
+	1    6550 3900
+	1    0    0    -1
+$EndComp
+Wire Wire Line
+	6550 3700 6100 3700
+Connection ~ 6100 3700
+$Comp
+L power:GND #PWR0104
+U 1 1 5EAE3489
+P 6550 4000
+F 0 "#PWR0104" H 6550 4000 30  0001 C CNN
+F 1 "GND" H 6550 3930 30  0001 C CNN
+F 2 "" H 6550 4000 50  0001 C CNN
+F 3 "" H 6550 4000 50  0001 C CNN
+	1    6550 4000
+	1    0    0    -1
+$EndComp
+Wire Wire Line
+	5650 3700 5650 4300
+$Comp
+L SparkFun-Capacitors:6PF-0402-50V-0.5% C6
+U 1 1 5EAE6A89
+P 6100 4300
+F 0 "C6" H 5993 4308 45  0000 R CNN
+F 1 "4.7 pF" H 5993 4392 45  0000 R CNN
+F 2 "0402" H 6100 4550 20  0001 C CNN
+F 3 "" H 6100 4300 50  0001 C CNN
+F 4 "" H 5993 4434 60  0000 R CNN "Field4"
+	1    6100 4300
+	0    1    -1   0
+$EndComp
+$Comp
+L SparkFun-Connectors:TEST-POINT3X4 TP1
+U 1 1 5EAC6ADE
+P 6300 4300
+F 0 "TP1" H 6364 4484 45  0000 C CNN
+F 1 "SMA" H 6364 4400 45  0000 C CNN
+F 2 "TestPoint:TestPoint_Pad_1.5x1.5mm" H 6300 4500 20  0001 C CNN
+F 3 "" H 6300 4300 50  0001 C CNN
+F 4 "" H 6364 4411 60  0000 C CNN "Field4"
+	1    6300 4300
+	1    0    0    -1
+$EndComp
+Wire Wire Line
+	6000 4300 5650 4300
+Connection ~ 5650 4300
+Wire Wire Line
+	5650 4300 5650 4450
+Text Label 5650 4000 0    50   ~ 0
+VCC
+Text Label 5150 4650 0    50   ~ 0
+GATE
+Wire Wire Line
+	4750 4000 4750 4100
+Wire Wire Line
+	4400 4000 4450 4000
+Wire Wire Line
+	4450 4000 4750 4000
+Connection ~ 4450 4000
+Connection ~ 4750 4000
+Wire Wire Line
+	4750 4300 4750 4350
+$Comp
 L SparkFun-Capacitors:6PF-0402-50V-0.5% C2
-U 1 1 5EAC63C2
+U 1 1 5EAF7D78
 P 4750 3800
 F 0 "C2" H 4643 3808 45  0000 R CNN
@@
 $EndComp
 $Comp
-L SparkFun-Connectors:TEST-POINT3X4 TP1
-U 1 1 5EAC6ADE
-P 5650 3850
-F 0 "TP1" H 5714 4034 45  0000 C CNN
-F 1 "SMA" H 5714 3950 45  0000 C CNN
-F 2 "TestPoint:TestPoint_Pad_1.5x1.5mm" H 5650 4050 20  0001 C CNN
-F 3 "" H 5650 3850 50  0001 C CNN
-F 4 "" H 5714 3961 60  0000 C CNN "Field4"
-	1    5650 3850
-	1    0    0    -1
-$EndComp
-Connection ~ 5650 3850
-Wire Wire Line
-	5650 3850 5650 4450
+L Device:D D1
+U 1 1 5EAF43A0
+P 4750 4150
+F 0 "D1" V 4704 4229 50  0000 L CNN
+F 1 "D" V 4795 4229 50  0000 L CNN
+F 2 "Diode_SMD:D_SOD-523" H 4750 4150 50  0001 C CNN
+F 3 "~" H 4750 4150 50  0001 C CNN
+	1    4750 4150
+	0    1    1    0
+$EndComp
+Text Label 4550 4350 0    50   ~ 0
+VCO1
+Text Label 4550 4000 0    50   ~ 0
+VCO2
 $EndSCHEMATC
