File: electronics/kicad/local_oscillator_v2/local_oscillator.sch (KiCad schematic (older format))
At the start: 22 parts, among them P1 TestPoint:TestPoint_Pad_1.5x1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, P2 TestPoint:TestPoint_Pad_1.5x1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, P3 TestPoint:TestPoint_Pad_1.5x1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, P4 TestPoint:TestPoint_Pad_1.5x1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, U1 CE3520K3

Commit message: Next rev.
Parts:
- removed C?: 0.1 uF, 0603, symbol SparkFun-Capacitors:4.7UF0603
- removed D4, D5, D6: D_Capacitance, Diode_SMD:D_SOD-523, symbol Device:D_Capacitance
- removed L1, L2, L3: 220 nH, 0402, symbol SparkFun-Coils:INDUCTOR-0402-3.9NH
- removed P2: TestPoint:TestPoint_Pad_1.5x1.5mm, TestPoint:TestPoint_Pad_1.5x1.5mm, symbol conn:CONN_1
- added R1, R2, R3, R4: 10k, 0402, symbol SparkFun-Resistors:RESISTOR0402
- gave numbers to parts that had none: 1
Connections:
- wire segments 15 -> 17
Other:
- moved on the sheet: C2, C3, D1, D2, D3, P1

Commit message: aaa
Parts:
- removed D2: D_Capacitance, Diode_SMD:D_SOD-523, symbol Device:D_Capacitance
Changed lines of the file:
@@
 	-1   0    0    1
-$EndComp
-$Comp
-L power:GND #PWR0107
-U 1 1 5ED14708
-P 4000 4950
-F 0 "#PWR0107" H 4000 4950 30  0001 C CNN
-F 1 "GND" H 4000 4880 30  0001 C CNN
-F 2 "" H 4000 4950 50  0001 C CNN
-F 3 "" H 4000 4950 50  0001 C CNN
-	1    4000 4950
-	1    0    0    -1
-$EndComp
-$Comp
-L Device:D_Capacitance D2
-U 1 1 5ED0FC00
-P 4000 4800
-F 0 "D2" V 3954 4879 50  0000 L CNN
-F 1 "D_Capacitance" V 4045 4879 50  0000 L CNN
-F 2 "Diode_SMD:D_SOD-523" H 4000 4800 50  0001 C CNN
-F 3 "~" H 4000 4800 50  0001 C CNN
-	1    4000 4800
-	0    1    1    0
 $EndComp
 Wire Wire Line

Commit message: Paper
Parts:
- removed D3: D_Capacitance, Diode_SMD:D_SOD-523, symbol Device:D_Capacitance
- removed R4: 10k, 0402, symbol SparkFun-Resistors:RESISTOR0402
- added C10, C7: 10 pF, 0402, symbol SparkFun-Capacitors:6PF-0402-50V-0.5%
- added C8: 0.1 uF, 0603, symbol SparkFun-Capacitors:4.7UF0603
- added D4: D_Capacitance, Diode_SMD:D_SOD-523, symbol Device:D_Capacitance
- added D5, D6: PiN, Diode_SMD:D_SOD-523, symbol Diode:1.5KExxA
- added L1: 1.2 nH, 0402, symbol SparkFun-Coils:INDUCTOR-0402-3.9NH
- added P2, P5, P6: TestPoint:TestPoint_Pad_1.5x1.5mm, TestPoint:TestPoint_Pad_1.5x1.5mm, symbol conn:CONN_1
- added Q1, Q2: BSS138, Package_TO_SOT_SMD:SOT-23, symbol Transistor_FET:BSS138
- added R5, R6: 10k, 0402, symbol SparkFun-Resistors:RESISTOR0402
- C1, C2: value 0.5 pF -> 10 pF
Connections:
- wire segments 17 -> 28
Other:
- moved on the sheet: C1, C3, C4, C5, C6, D1, L4, P1, P3, P4, R1, R3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

Commit message: LO test something more
Parts:
- removed R5: 10k, 0402, symbol SparkFun-Resistors:RESISTOR0402
- added P7: TestPoint:TestPoint_Pad_1.5x1.5mm, TestPoint:TestPoint_Pad_1.5x1.5mm, symbol conn:CONN_1
- added P8: TestPoint:TestPoint_Pad_1.5x1.5mm, TestPoint:TestPoint_Pad_D1.0mm, symbol conn:CONN_1
- added R?: 10k, 0402, symbol SparkFun-Resistors:RESISTOR0402
Connections:
- wire segments 28 -> 27
Other:
- moved on the sheet: P5, Q2
Changed lines of the file:
@@
 Wire Wire Line
 	5600 5000 5600 4900
-$Comp
-L SparkFun-Resistors:RESISTOR0402 R5
-U 1 1 5EEB120C
-P 5600 4150
-F 0 "R5" V 5695 4218 45  0000 L CNN
-F 1 "10k" V 5611 4218 45  0000 L CNN
-F 2 "0402" H 5600 4300 20  0001 C CNN
-F 3 "" H 5600 4150 60  0001 C CNN
-F 4 " " V 5516 4218 60  0000 L CNN "Field4"
-	1    5600 4150
-	0    -1   -1   0
-$EndComp
-Wire Wire Line
-	5600 4600 5600 4350
 Connection ~ 5600 4900
-Connection ~ 5600 4600
 Wire Wire Line
 	8000 4600 6750 4600
@@
 Wire Wire Line
 	2550 4600 2550 3700
-Wire Wire Line
-	2550 3700 8100 3700
 Wire Wire Line
 	8100 3700 8100 4050
@@
 L Transistor_FET:BSS138 Q2
 U 1 1 5EF335C6
-P 5700 3750
-F 0 "Q2" H 5906 3704 50  0000 L CNN
-F 1 "BSS138" H 5906 3795 50  0000 L CNN
-F 2 "Package_TO_SOT_SMD:SOT-23" H 5900 3675 50  0001 L CIN
-F 3 "https://www.fairchildsemi.com/datasheets/BS/BSS138.pdf" H 5700 3750 50  0001 L CNN
-	1    5700 3750
+P 3450 2250
+F 0 "Q2" H 3656 2204 50  0000 L CNN
+F 1 "BSS138" H 3656 2295 50  0000 L CNN
+F 2 "Package_TO_SOT_SMD:SOT-23" H 3650 2175 50  0001 L CIN
+F 3 "https://www.fairchildsemi.com/datasheets/BS/BSS138.pdf" H 3450 2250 50  0001 L CNN
+	1    3450 2250
 	-1   0    0    1
 $EndComp
@@
 L power:GND #PWR0111
 U 1 1 5EF356BF
-P 5600 3550
-F 0 "#PWR0111" H 5600 3550 30  0001 C CNN
-F 1 "GND" H 5600 3480 30  0001 C CNN
-F 2 "" H 5600 3550 50  0001 C CNN
-F 3 "" H 5600 3550 50  0001 C CNN
-	1    5600 3550
+P 3350 2050
+F 0 "#PWR0111" H 3350 2050 30  0001 C CNN
+F 1 "GND" H 3350 1980 30  0001 C CNN
+F 2 "" H 3350 2050 50  0001 C CNN
+F 3 "" H 3350 2050 50  0001 C CNN
+	1    3350 2050
 	-1   0    0    1
 $EndComp
@@
 L conn:CONN_1 P5
 U 1 1 5EF35E85
-P 6050 3750
-F 0 "P5" H 5983 3653 40  0000 C CNN
-F 1 "TestPoint:TestPoint_Pad_1.5x1.5mm" H 6000 3790 30  0001 C CNN
-F 2 "TestPoint:TestPoint_Pad_1.5x1.5mm" H 6050 3750 50  0001 C CNN
-F 3 "" H 6050 3750 50  0001 C CNN
-	1    6050 3750
+P 3800 2250
+F 0 "P5" H 3733 2153 40  0000 C CNN
+F 1 "TestPoint:TestPoint_Pad_1.5x1.5mm" H 3750 2290 30  0001 C CNN
+F 2 "TestPoint:TestPoint_Pad_1.5x1.5mm" H 3800 2250 50  0001 C CNN
+F 3 "" H 3800 2250 50  0001 C CNN
+	1    3800 2250
 	1    0    0    -1
 $EndComp
+$Comp
+L conn:CONN_1 P7
+U 1 1 5EF87253
+P 3350 2600
+F 0 "P7" H 3283 2503 40  0000 C CNN
+F 1 "TestPoint:TestPoint_Pad_1.5x1.5mm" H 3300 2640 30  0001 C CNN
+F 2 "TestPoint:TestPoint_Pad_1.5x1.5mm" H 3350 2600 50  0001 C CNN
+F 3 "" H 3350 2600 50  0001 C CNN
+	1    3350 2600
+	0    1    1    0
+$EndComp
+Wire Wire Line
+	2550 3700 8100 3700
+$Comp
+L conn:CONN_1 P8
+U 1 1 5EF94F93
+P 5600 4050
+F 0 "P8" H 5533 3953 40  0000 C CNN
+F 1 "TestPoint:TestPoint_Pad_1.5x1.5mm" H 5550 4090 30  0001 C CNN
+F 2 "TestPoint:TestPoint_Pad_D1.0mm" H 5600 4050 50  0001 C CNN
+F 3 "" H 5600 4050 50  0001 C CNN
+	1    5600 4050
+	0    -1   -1   0
+$EndComp
+$Comp
+L SparkFun-Resistors:RESISTOR0402 R?
+U 1 1 5EFB03E2
+P 5600 4400
+F 0 "R?" V 5695 4468 45  0000 L CNN
+F 1 "10k" V 5611 4468 45  0000 L CNN
+F 2 "0402" H 5600 4550 20  0001 C CNN
+F 3 "" H 5600 4400 60  0001 C CNN
+F 4 " " V 5516 4468 60  0000 L CNN "Field4"
+	1    5600 4400
+	0    -1   -1   0
+$EndComp
+Connection ~ 5600 4600
 $EndSCHEMATC

Commit message: 4-pole LO
Parts:
- removed C10, C7: 10 pF, 0402, symbol SparkFun-Capacitors:6PF-0402-50V-0.5%
- removed C8: 0.1 uF, 0603, symbol SparkFun-Capacitors:4.7UF0603
- removed D5, D6: PiN, Diode_SMD:D_SOD-523, symbol Diode:1.5KExxA
- removed P2, P5, P6, P7: TestPoint:TestPoint_Pad_1.5x1.5mm, TestPoint:TestPoint_Pad_1.5x1.5mm, symbol conn:CONN_1
- removed P8: TestPoint:TestPoint_Pad_1.5x1.5mm, TestPoint:TestPoint_Pad_D1.0mm, symbol conn:CONN_1
- removed Q1, Q2: BSS138, Package_TO_SOT_SMD:SOT-23, symbol Transistor_FET:BSS138
- removed R6, R?: 10k, 0402, symbol SparkFun-Resistors:RESISTOR0402
- added D2, D3, D5, D6: D_Capacitance, Diode_SMD:D_SOD-523, symbol Device:D_Capacitance
- added R4: 10k, 0402, symbol SparkFun-Resistors:RESISTOR0402
- L1: value 1.2 nH -> 220 nH
Connections:
- wire segments 27 -> 31
Other:
- moved on the sheet: C1, C4, C5, D1, D4, P3, R3

Commit message: SPICE
Parts:
- removed D4, D5, D6: D_Capacitance, Diode_SMD:D_SOD-523, symbol Device:D_Capacitance
- removed R4: 10k, 0402, symbol SparkFun-Resistors:RESISTOR0402
Connections:
- wire segments 31 -> 25
Other:
- moved on the sheet: D1
Changed lines of the file:
@@
-$EndComp
-$Comp
-L power:GND #PWR0107
-U 1 1 5EE0E867
-P 6900 5200
-F 0 "#PWR0107" H 6900 5200 30  0001 C CNN
-F 1 "GND" H 6900 5130 30  0001 C CNN
-F 2 "" H 6900 5200 50  0001 C CNN
-F 3 "" H 6900 5200 50  0001 C CNN
-	1    6900 5200
-	1    0    0    -1
-$EndComp
-$Comp
-L Device:D_Capacitance D4
-U 1 1 5EE0E0B0
-P 6900 5050
-F 0 "D4" V 6854 5129 50  0000 L CNN
-F 1 "D_Capacitance" V 6945 5129 50  0000 L CNN
-F 2 "Diode_SMD:D_SOD-523" H 6900 5050 50  0001 C CNN
-F 3 "~" H 6900 5050 50  0001 C CNN
-	1    6900 5050
-	0    1    1    0
-$EndComp
-$Comp
-L power:GND #PWR0106
-U 1 1 5EE0BB79
-P 7300 5200
-F 0 "#PWR0106" H 7300 5200 30  0001 C CNN
-F 1 "GND" H 7300 5130 30  0001 C CNN
-F 2 "" H 7300 5200 50  0001 C CNN
-F 3 "" H 7300 5200 50  0001 C CNN
-	1    7300 5200
-	1    0    0    -1
 $EndComp
 $Comp
 L Device:D_Capacitance D1
 U 1 1 5ED19292
-P 7300 5050
-F 0 "D1" V 7254 5129 50  0000 L CNN
-F 1 "D_Capacitance" V 7345 5129 50  0000 L CNN
-F 2 "Diode_SMD:D_SOD-523" H 7300 5050 50  0001 C CNN
-F 3 "~" H 7300 5050 50  0001 C CNN
-	1    7300 5050
-	0    1    1    0
-$EndComp
-Wire Wire Line
-	7300 4900 7300 4600
-Wire Wire Line
-	6900 4900 6900 4600
+P 7050 4600
+F 0 "D1" H 7050 4345 50  0000 C CNN
+F 1 "D_Capacitance" H 7050 4436 50  0000 C CNN
+F 2 "Diode_SMD:D_SOD-523" H 7050 4600 50  0001 C CNN
+F 3 "~" H 7050 4600 50  0001 C CNN
+	1    7050 4600
+	-1   0    0    1
+$EndComp
 $Comp
 L SparkFun-Resistors:RESISTOR0402 R3
@@
 	-1   0    0    1
 $EndComp
-Wire Wire Line
-	6900 4600 7300 4600
-Connection ~ 7300 4600
 $Comp
 L SparkFun-Capacitors:6PF-0402-50V-0.5% C2
@@
 	-1   0    0    1
 $EndComp
-$Comp
-L Device:D_Capacitance D5
-U 1 1 5F005E53
-P 5550 4600
-F 0 "D5" H 5550 4816 50  0000 C CNN
-F 1 "D_Capacitance" H 5550 4725 50  0000 C CNN
-F 2 "Diode_SMD:D_SOD-523" H 5550 4600 50  0001 C CNN
-F 3 "~" H 5550 4600 50  0001 C CNN
-	1    5550 4600
-	1    0    0    -1
-$EndComp
-$Comp
-L Device:D_Capacitance D6
-U 1 1 5F007895
-P 5850 4600
-F 0 "D6" H 5850 4345 50  0000 C CNN
-F 1 "D_Capacitance" H 5850 4436 50  0000 C CNN
-F 2 "Diode_SMD:D_SOD-523" H 5850 4600 50  0001 C CNN
-F 3 "~" H 5850 4600 50  0001 C CNN
-	1    5850 4600
-	-1   0    0    1
-$EndComp
-Wire Wire Line
-	6000 4600 6050 4600
-Connection ~ 6900 4600
 Wire Wire Line
 	4800 4600 4750 4600
@@
 	5100 4600 5100 4950
 Connection ~ 5100 4600
-Wire Wire Line
-	5700 4600 5700 4950
-Connection ~ 5700 4600
-$Comp
-L power:GND #PWR0108
-U 1 1 5F009480
-P 5700 4950
-F 0 "#PWR0108" H 5700 4950 30  0001 C CNN
-F 1 "GND" H 5700 4880 30  0001 C CNN
-F 2 "" H 5700 4950 50  0001 C CNN
-F 3 "" H 5700 4950 50  0001 C CNN
-	1    5700 4950
-	1    0    0    -1
-$EndComp
 $Comp
 L power:GND #PWR0110
@@
 	0    -1   -1   0
 $EndComp
-$Comp
-L SparkFun-Resistors:RESISTOR0402 R4
-U 1 1 5F02BE58
-P 6050 4100
-F 0 "R4" V 5955 4168 45  0000 L CNN
-F 1 "10k" V 6039 4168 45  0000 L CNN
-F 2 "0402" H 6050 4250 20  0001 C CNN
-F 3 "" H 6050 4100 60  0001 C CNN
-F 4 " " V 6134 4168 60  0000 L CNN "Field4"
-	1    6050 4100
-	0    -1   -1   0
-$EndComp
 Wire Wire Line
 	5450 3900 5450 3650
-Wire Wire Line
-	5450 3900 6050 3900
-Connection ~ 5450 3900
 Wire Wire Line
 	5450 3900 5400 3900
@@
 Wire Wire Line
 	5400 4600 5400 4300
-Connection ~ 5400 4600
-Wire Wire Line
-	6050 4300 6050 4600
-Connection ~ 6050 4600
-Wire Wire Line
-	6050 4600 6900 4600
 Wire Wire Line
 	4750 4300 4750 4600
@@
 Wire Wire Line
 	8300 4150 8300 4300
+Wire Wire Line
+	5400 4600 6900 4600
+Connection ~ 5400 4600
+Wire Wire Line
+	7200 4600 7300 4600
 $EndSCHEMATC

Commit message: SVG import improvements
Parts:
- P1: value TestPoint:TestPoint_Pad_1.5x1.5mm -> T
- P3, P4: value TestPoint:TestPoint_Pad_1.5x1.5mm -> a
Changed lines of the file:
@@
 P 9100 4300
 F 0 "P4" H 9033 4203 40  0000 C CNN
-F 1 "TestPoint:TestPoint_Pad_1.5x1.5mm" H 9050 4340 30  0001 C CNN
+F 1 "a" H 9050 4340 30  0001 C CNN
 F 2 "TestPoint:TestPoint_Pad_1.5x1.5mm" H 9100 4300 50  0001 C CNN
 F 3 "" H 9100 4300 50  0001 C CNN
@@
 P 8150 3250
 F 0 "P3" H 8083 3153 40  0000 C CNN
-F 1 "TestPoint:TestPoint_Pad_1.5x1.5mm" H 8100 3290 30  0001 C CNN
+F 1 "a" H 8100 3290 30  0001 C CNN
 F 2 "TestPoint:TestPoint_Pad_1.5x1.5mm" H 8150 3250 50  0001 C CNN
 F 3 "" H 8150 3250 50  0001 C CNN
@@
 P 5500 3500
 F 0 "P1" H 5433 3403 40  0000 C CNN
-F 1 "TestPoint:TestPoint_Pad_1.5x1.5mm" H 5450 3540 30  0001 C CNN
+F 1 "T" H 5450 3540 30  0001 C CNN
 F 2 "TestPoint:TestPoint_Pad_1.5x1.5mm" H 5500 3500 50  0001 C CNN
 F 3 "" H 5500 3500 50  0001 C CNN
