File: electronics/kicad/fdtd_test/fdtd_test.sch (KiCad schematic (older format))
At the start: 2 parts

Commit message: pvsm
Parts:
- added D1: SCHOTTKY, Diode_SMD:D_SOD-523, symbol w_device:SCHOTTKY
- gave numbers to parts that had none: 2
Connections:
- wire segments 1 -> 4
Other:
- moved on the sheet: R1
Changed lines of the file:
@@
 $EndDescr
 $Comp
-L SparkFun-Capacitors:6PF-0402-50V-0.5% C?
+L SparkFun-Capacitors:6PF-0402-50V-0.5% C1
 U 1 1 5ED41179
 P 3850 3950
-F 0 "C?" H 3958 4095 45  0000 L CNN
+F 0 "C1" H 3958 4095 45  0000 L CNN
 F 1 "c1" H 3958 4011 45  0000 L CNN
 F 2 "0402" H 3850 4200 20  0001 C CNN
@@
 $EndComp
 $Comp
-L SparkFun-Resistors:RESISTOR0402 R?
+L SparkFun-Resistors:RESISTOR0402 R1
 U 1 1 5ED4190A
-P 3650 3750
-F 0 "R?" H 3650 4050 45  0000 C CNN
-F 1 "R " H 3650 3966 45  0000 C CNN
-F 2 "0402" H 3650 3900 20  0001 C CNN
-F 3 "" H 3650 3750 60  0001 C CNN
-F 4 " " H 3650 3871 60  0000 C CNN "Field4"
-	1    3650 3750
-	1    0    0    -1
+P 3450 3950
+F 0 "R1" V 3355 4018 45  0000 L CNN
+F 1 "R " V 3439 4018 45  0000 L CNN
+F 2 "0402" H 3450 4100 20  0001 C CNN
+F 3 "" H 3450 3950 60  0001 C CNN
+F 4 " " V 3534 4018 60  0000 L CNN "Field4"
+	1    3450 3950
+	0    1    1    0
 $EndComp
 $Comp
-L power:GND #PWR?
+L power:GND #PWR0101
 U 1 1 5ED44D0E
 P 3850 4050
-F 0 "#PWR?" H 3850 4050 30  0001 C CNN
+F 0 "#PWR0101" H 3850 4050 30  0001 C CNN
 F 1 "GND" H 3850 3980 30  0001 C CNN
 F 2 "" H 3850 4050 50  0001 C CNN
@@
 	3850 3750 4150 3750
 Connection ~ 3850 3750
+Wire Wire Line
+	3450 3750 3300 3750
+$Comp
+L w_device:SCHOTTKY D1
+U 1 1 5ED46B62
+P 3200 3750
+F 0 "D1" H 3225 4023 40  0000 C CNN
+F 1 "SCHOTTKY" H 3225 3947 40  0000 C CNN
+F 2 "Diode_SMD:D_SOD-523" H 3225 3856 60  0000 C CNN
+F 3 "" H 3200 3750 60  0000 C CNN
+	1    3200 3750
+	1    0    0    -1
+$EndComp
+Wire Wire Line
+	3450 3750 3850 3750
+Connection ~ 3450 3750
+$Comp
+L power:GND #PWR0102
+U 1 1 5ED4A4E4
+P 3450 4150
+F 0 "#PWR0102" H 3450 4150 30  0001 C CNN
+F 1 "GND" H 3450 4080 30  0001 C CNN
+F 2 "" H 3450 4150 50  0001 C CNN
+F 3 "" H 3450 4150 50  0001 C CNN
+	1    3450 4150
+	1    0    0    -1
+$EndComp
+Wire Wire Line
+	3150 3750 2900 3750
 $EndSCHEMATC

Commit message: Some more documentation
Parts:
- added L? (x2): 220nH, 0402, symbol SparkFun-Coils:INDUCTOR-0402-3.9NH
- added U?: BFP620, Package_TO_SOT_SMD:SOT-343_SC-70-4, symbol 0xDBFB7:BFP620
Changed lines of the file:
@@
 Wire Wire Line
 	3150 3750 2900 3750
+$Comp
+L 0xDBFB7:BFP620 U?
+U 1 1 5EE0044F
+P 4200 2700
+F 0 "U?" H 4494 2196 50  0000 L CNN
+F 1 "BFP620" H 4494 2105 50  0000 L CNN
+F 2 "Package_TO_SOT_SMD:SOT-343_SC-70-4" H 4200 2700 50  0001 C CNN
+F 3 "" H 4200 2700 50  0001 C CNN
+	1    4200 2700
+	1    0    0    -1
+$EndComp
+$Comp
+L SparkFun-Coils:INDUCTOR-0402-3.9NH L?
+U 1 1 5EE05A6A
+P 4350 2100
+F 0 "L?" H 4402 2142 45  0000 L CNN
+F 1 "220nH" H 4402 2058 45  0000 L CNN
+F 2 "0402" H 4350 2350 20  0001 C CNN
+F 3 "" H 4350 2100 50  0001 C CNN
+F 4 "" H 4402 2016 60  0000 L CNN "Field4"
+	1    4350 2100
+	1    0    0    -1
+$EndComp
+$Comp
+L SparkFun-Coils:INDUCTOR-0402-3.9NH L?
+U 1 1 5EE0621D
+P 4350 2500
+F 0 "L?" H 4402 2542 45  0000 L CNN
+F 1 "220nH" H 4402 2458 45  0000 L CNN
+F 2 "0402" H 4350 2750 20  0001 C CNN
+F 3 "" H 4350 2500 50  0001 C CNN
+F 4 "" H 4402 2416 60  0000 L CNN "Field4"
+	1    4350 2500
+	1    0    0    -1
+$EndComp
 $EndSCHEMATC
