File: electronics/kicad/driver_card_2/driver_card.kicad_pcb (KiCad board)
At the start: 2 copper layers, 35.8 x 25.2 mm, 24 parts, among them J1 CONN_10SMD_MALE, Q1 2N7002, Q2 MMBT4401, Q3 BSS84, U2 INA194

Commit message: Spectrum analyzer progress
Parts:
- added C11: 0.1 uF, Capacitors:0603, F.Cu at (154.4, 126.5)
- added C3: 0.1 uF, Capacitors:0603, F.Cu at (154.4, 124.0)
- added C4: 10 uF, Capacitors:0603, F.Cu at (164.0, 119.2)
- added C5: 10uF, Capacitors:1206, F.Cu at (111.0, 124.0)
- added C6: 10uF, Capacitors:1206, F.Cu at (145.9, 119.7)
- added Q4: 2N7002, Package_TO_SOT_SMD:SOT-23, F.Cu at (145.2, 132.8)
- added R1: 30k, Resistor_SMD:R_0603_1608Metric, F.Cu at (162.6, 126.6)
- added R18: 10k, Resistor_SMD:R_0603_1608Metric, F.Cu at (166.6, 125.8)
- added R19: 10k, Resistor_SMD:R_0603_1608Metric, F.Cu at (162.6, 129.1)
- added R2: 10k, Resistor_SMD:R_0603_1608Metric, F.Cu at (158.1, 130.7)
- added R3: 5k, Resistor_SMD:R_0603_1608Metric, F.Cu at (126.0, 132.2)
- added R4: 1K, Resistor_SMD:R_0603_1608Metric, F.Cu at (167.9, 123.3)
- added R5: 2k, Resistor_SMD:R_0603_1608Metric, F.Cu at (157.7, 133.2)
- added R6: 2k, Resistor_SMD:R_0603_1608Metric, F.Cu at (149.4, 134.0)
- added R7: 5k, Resistor_SMD:R_0603_1608Metric, F.Cu at (171.9, 123.3)
- added R8: 5k, Resistor_SMD:R_0603_1608Metric, F.Cu at (170.1, 130.9)
- added U1: MCP4725SOT-23, Silicon-Standard:SOT23-6, F.Cu at (150.8, 120.4)
- added U3: AZ1117CH-3_3TRG1, digikey-footprints:SOT-223, F.Cu at (118.0, 121.5)
- added U4: MCP1416T-E_OT, digikey-footprints:SOT-753, F.Cu at (111.0, 127.2)
- C1, C8: value 10 uF -> 0.1 uF
- C7: value 10 uF -> 10uF; footprint Capacitors:0603 -> Capacitors:1206
- Q2: value MMBT4401 -> 2N7002; footprint digikey-footprints:SOT-23-3 -> Package_TO_SOT_SMD:SOT-23
- R10: value 1k -> 1K
- R12: value 10K -> 1k
- R14: value 1K -> 1k; footprint Resistor_SMD:R_0402_1005Metric -> Resistor_SMD:R_0603_1608Metric
- R15: value 10K -> 1k; footprint Resistor_SMD:R_0402_1005Metric -> Resistor_SMD:R_0603_1608Metric
- R16: value 2.2r -> 0.1R
- R17: value 2.2r -> 1k; footprint Resistor_SMD:R_0805_2012Metric -> Resistor_SMD:R_0603_1608Metric
- TP1: value Test_Point -> 48V
- TP2: value Test_Point -> 12V
- moved R15 54.7 mm to (166.6, 128.4), turned to 0 degrees
- moved R14 51.9 mm to (162.1, 131.6), turned to 0 degrees
- moved R17 48.4 mm to (172.2, 119.3), turned to 0 degrees
- moved C9 48.3 mm to (158.6, 124.1), turned to 0 degrees
- moved C2 47.8 mm to (159.8, 121.7), turned to 0 degrees
- moved R13 42.0 mm to (170.6, 125.8), turned to 0 degrees
- moved R10 37.1 mm to (170.6, 128.4)
- moved R11 36.7 mm to (166.1, 131.6)
- moved TP2 36.2 mm to (168.1, 120.1)
- moved C8 35.9 mm to (153.9, 128.9), turned to 0 degrees
- moved Q3 35.0 mm to (155.4, 120.3)
- moved R9 31.7 mm to (165.7, 134.1)
- moved Q2 31.3 mm to (145.2, 128.2), turned to 0 degrees
- moved TP4 31.0 mm to (158.5, 127.4)
- moved TP3 29.0 mm to (163.9, 122.5)
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Connections:
- C2 pad 2: 3.3V -> +12V
- C7 pad 1: GND -> Net-(C7-Pad1)
- C7 pad 2: source_supply_feedback -> GND
- C8 pad 2: source_supply_feedback -> Net-(C7-Pad1)
- C9 pad 1: Net-(C9-Pad1) -> GND
- C9 pad 2: GND -> Net-(C9-Pad2)
- J1 pad 5: nsource -> pulse_feedback
- Q1 pad 1: ~VARACTOR_PWM -> Net-(C4-Pad2)
- Q1 pad 3: Net-(Q1-Pad3) -> VARACTOR_OUT
- Q2 pad 1: Net-(C9-Pad1) -> VSOURCE_PWM
- Q2 pad 2: source_supply_feedback -> GND
- Q2 pad 3: 3.3V -> Net-(Q2-Pad3)
- Q3 pad 1: ~PULSE_INPUT -> Net-(Q3-Pad1)
- Q3 pad 2: source_supply_feedback -> Net-(C7-Pad1)
- R10 pad 1: VARACTOR_OUT -> GND
- R10 pad 2: Net-(Q1-Pad3) -> pulse_feedback
- R11 pad 1: VARACTOR_FEEDBACK -> GND
- R12 pad 1: ~VARACTOR_PWM -> BIAS_PWM
- R12 pad 2: 3.3V -> Net-(C9-Pad2)
- R13 pad 1: GND -> Net-(R13-Pad1)
- R13 pad 2: VARACTOR_FEEDBACK -> 3.3V
- R14 pad 1: VSOURCE_PWM -> Net-(C9-Pad2)
- R14 pad 2: Net-(C9-Pad1) -> Net-(R13-Pad1)
- R15 pad 1: 3.3V -> Net-(R15-Pad1)
- R15 pad 2: VSOURCE_PWM -> Net-(C9-Pad2)
- R17 pad 1: nsource -> GND
- R17 pad 2: Net-(Q3-Pad3) -> Net-(R15-Pad1)
- R9 pad 1: Net-(Q1-Pad3) -> VARACTOR_OUT
- TP2 pad 1: BIAS_PWM -> +12V
Routing:
- net VARACTOR_FEEDBACK: track 17.0 -> 0.00 mm
- net 3.3V: track 55.7 -> 39.2 mm, vias 3 -> 0
- net ~VARACTOR_PWM: track 12.8 -> 0.00 mm
- net Net-(C9-Pad1): track 11.6 -> 0.00 mm, vias 2 -> 0
- net nsource: track 11.6 -> 0.00 mm
- net source_supply_feedback: track 10.2 -> 0.03 mm
- net VSOURCE_PWM: track 9.74 -> 0.00 mm
- net Net-(Q2-Pad1): track 0.00 -> 7.67 mm
- net CURRENT_SENSE: track 22.3 -> 16.4 mm, vias 2 -> 0
- net ~PULSE_INPUT: track 17.9 -> 12.1 mm, vias 2 -> 0
- net GND: track 5.73 -> 0.00 mm
- net VARACTOR_OUT: track 4.32 -> 0.00 mm
- removed copper zone on F.Cu, net GND
- removed copper zone on F.Cu, net Net-(Q3-Pad3)
- removed copper zone on F.Cu, net nsource
- removed copper zone on F.Cu, net source_supply_feedback
Other:
- outline, holes or cut-outs redrawn
