File: electronics/kicad/lil_driver/lil_driver.kicad_pcb (KiCad board)
At the start: 2 copper layers, 23 parts, among them J1 CONN_06SMD, Q1 2N7002, Q2 2N7002, Q3 BSS84, U1 MCP4725SOT-23

Commit message: Manual ops
Parts:
- moved U1 0.63 mm to (173.8, 100.2)
Changed lines of the file:
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@@
   )
   (module Silicon-Standard:SOT23-6 (layer F.Cu)
-    (at 174.4 100)
+    (at 173.8 100.2)
     (descr SOT23-6)
     (tags SOT23-6)
