File: electronics/kicad/eppenwolf_bottom/eppenwolf_bottom.kicad_pcb (KiCad board)
At the start: 2 copper layers, 68 x 56 mm, 0 parts

Commit message: Eppenwolf milled out
Parts:
- added C1: 100 pF, Capacitor_SMD:C_0402_1005Metric, F.Cu at (44.8, 85.5)
- added C2: 100 pF, Capacitor_SMD:C_0402_1005Metric, F.Cu at (42.8, 23.2)
- added C3: 100 pF, Capacitor_SMD:C_0402_1005Metric, F.Cu at (40.1, 29.1)
- added C4: 100 pF, Capacitor_SMD:C_0402_1005Metric, F.Cu at (43.1, 82.5)
- added C5: 100 pF, Capacitor_SMD:C_0402_1005Metric, F.Cu at (40.4, 87.8)
- added C6: 100 pF, Capacitor_SMD:C_0402_1005Metric, F.Cu at (44.6, 27.3)
- added D1: BAT15-04, Package_TO_SOT_SMD:SOT-23, F.Cu at (42.3, 25.4)
- added D2: BAT15-04, Package_TO_SOT_SMD:SOT-23, F.Cu at (42.4, 28.6)
- added D3: BAT15-04, Package_TO_SOT_SMD:SOT-23, F.Cu at (42.5, 84.5)
- added D4: BAT15-04, Package_TO_SOT_SMD:SOT-23, F.Cu at (42.5, 87.3)
- added Q1: MOSFET-NCH-FDD8780, Silicon-Standard:DPAK, F.Cu at (55.8, 88.9)
- added R10: 10k, Capacitors:0402, F.Cu at (42.6, 22.0)
- added R11: 10k, Capacitors:0402, F.Cu at (39.1, 29.0)
- added R12: 10k, Capacitors:0402, F.Cu at (43.0, 81.2)
- added R13: 10k, Capacitors:0402, F.Cu at (39.1, 87.8)
- added R6: 1k, Resistor_SMD:R_0603_1608Metric, F.Cu at (56.0, 94.2)
- added R9: 50R, Capacitors:0805, F.Cu at (46.0, 87.2)
- added TP1: capacitance_sensing, TestPoint:TestPoint_Pad_1.5x1.5mm, F.Cu at (38.8, 24.5)
- added TP3: capacitance_sensing, TestPoint:TestPoint_Pad_1.5x1.5mm, F.Cu at (37.2, 28.9)
- added TP4: capacitance_sensing, TestPoint:TestPoint_Pad_1.5x1.5mm, F.Cu at (39.5, 84.0)
- added TP5: capacitance_sensing, TestPoint:TestPoint_Pad_1.5x1.5mm, F.Cu at (39.8, 89.5)
Routing:
- net RF_input: track 0.00 -> 65.0 mm
- net high_current_trace: track 0.00 -> 63.3 mm
- net (no net): track 0.00 -> 53.0 mm, vias 0 -> 1
- net GND: track 0.00 -> 23.2 mm
- net input_power_sense_2: track 0.00 -> 7.16 mm
- net terminated_end_power_sense_2: track 0.00 -> 6.61 mm
- net input_power_sense_1: track 0.00 -> 5.02 mm
- net terminated_end_power_sense_1: track 0.00 -> 4.81 mm
- net Net-(C6-Pad1): track 0.00 -> 1.91 mm
- net Net-(Q1-Pad1): track 0.00 -> 1.67 mm
- added copper zone on F.Cu, net GND
Other:
- board outline removed
- net class Default: trace_width 0.25 -> 0.5
