File: electronics/kicad/eppenwolf_bottom/eppenwolf_bottom.sch (KiCad schematic (older format))
At the start: 28 parts, among them J1 CONN_06SMD

Commit message: gosh writing papers is addictive, have to stop
Parts:
- added bolometer_power: (no value), TestPoint:TestPoint_Pad_1.5x1.5mm, symbol Connector:Test_Point
Changed lines of the file:
@@
 	1    0    0    -1
 $EndComp
+$Comp
+L SparkFun-PowerSymbols:3.3V #SUPPLY?
+U 1 1 5F496F4D
+P 2150 2550
+F 0 "#SUPPLY?" H 2200 2550 45  0001 L BNN
+F 1 "3.3V" H 2150 2720 45  0000 C CNN
+F 2 "" H 2150 2731 60  0000 C CNN
+F 3 "" H 2150 2550 60  0001 C CNN
+	1    2150 2550
+	1    0    0    -1
+$EndComp
+$Comp
+L Connector:Test_Point bolometer_power
+U 1 1 5F4972C7
+P 2150 2550
+F 0 "bolometer_power" H 2208 2668 50  0000 L CNN
+F 1 " " H 2208 2577 50  0000 L CNN
+F 2 "TestPoint:TestPoint_Pad_1.5x1.5mm" H 2350 2550 50  0001 C CNN
+F 3 "~" H 2350 2550 50  0001 C CNN
+	1    2150 2550
+	-1   0    0    1
+$EndComp
 $EndSCHEMATC

Commit message: Eppenwolf milled out
Parts:
- removed C? (x4): 100 pF, 0402, symbol SparkFun-Capacitors:6PF-0402-50V-0.5%
- removed D?: BAT15-04, Package_TO_SOT_SMD:SOT-23, symbol Diode:BAS40-04
- removed J1: CONN_06SMD, 1X06-SMD_RA_MALE, symbol SparkFun-Connectors:CONN_06SMD
- removed R?: 180, Resistor_SMD:R_0603_1608Metric, symbol SparkFun-Resistors:RESISTOR0402
- removed R?: THERM, Resistor_SMD:R_0603_1608Metric, symbol SparkFun-Resistors:RESISTOR0402
- removed R?: 10k, Resistor_SMD:R_0603_1608Metric, symbol SparkFun-Resistors:RESISTOR0402
- removed TP?: capacitance_sensing, TestPoint:TestPoint_Pad_1.5x1.5mm, symbol Connector:Test_Point
- added C1, C2, C3, C4, C5, C6: 100 pF, Capacitor_SMD:C_0402_1005Metric, symbol SparkFun-Capacitors:6PF-0402-50V-0.5%
- added D4: BAT15-04, Package_TO_SOT_SMD:SOT-23, symbol Diode:BAS40-04
- added TP1, TP3, TP4, TP5: capacitance_sensing, TestPoint:TestPoint_Pad_1.5x1.5mm, symbol Connector:Test_Point
- R6: renamed from R?; value 180 -> 1k
- R7: renamed from R?; value 180 -> 330
- gave numbers to parts that had none: 13
- renumbered bolometer_SCL to bolometer_SCL1, bolometer_SDA to bolometer_SDA1, bolometer_power to bolometer_power1
Connections:
- net labels added: RF_input, high_current_trace, input_power_sense_1, input_power_sense_2, terminated_end, terminated_end_power_sense_1, terminated_end_power_sense_2
- net labels removed: far_end, far_end_power_sense_1, far_end_power_sense_2, near_end, thermistor
- wire segments 11 -> 16
Other:
- moved on the sheet: D1, D2, Q1, R1, R10, R11, R6, R9, bolometer_SDA1, bolometer_power1
