File: electronics/kicad/lil_driver_2/lil_driver_2.kicad_pcb (KiCad board)
At the start: 2 copper layers, 35 parts, among them J1 CONN_01, J2 CONN_01, J3 CONN_01, J4 CONN_01, J5 CONN_01, J6 CONN_01, J7 CONN_01, Q3 BSS84, U1 LM358, U2 V_REG_LM1117SOT223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

Commit message: Driver built
Other:
- board outline added: 38.5 x 46 mm
Changed lines of the file:
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@@
   (general
     (thickness 1.6)
-    (drawings 0)
+    (drawings 4)
     (tracks 121)
     (zones 0)
@@
     )
   )
+  (gr_line (start 148.5 83.5) (end 110 83.5) (layer Edge.Cuts) (width 0.05))
+  (gr_line (start 148.5 129.5) (end 148.5 83.5) (layer Edge.Cuts) (width 0.05))
+  (gr_line (start 110 129.5) (end 148.5 129.5) (layer Edge.Cuts) (width 0.05))
+  (gr_line (start 110 83.5) (end 110 129.5) (layer Edge.Cuts) (width 0.05))
   (segment (start 129.0625 117.15) (end 129.2125 117) (width 0.5) (layer F.Cu) (net 1))
   (segment (start 123.2125 116.5) (end 123.5 116.7875) (width 0.5) (layer F.Cu) (net 1))
