File: electronics/kicad/lil_driver_2/lil_driver_2.sch (KiCad schematic (older format))
At the start: 35 parts, among them J1 CONN_01, J2 CONN_01, J3 CONN_01, J4 CONN_01, J5 CONN_01, J6 CONN_01, J7 CONN_01, Q3 BSS84, U1 LM358, U2 V_REG_LM1117SOT223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

Commit message: Driver built
Parts:
- U1: value LM358 -> TS912IDT
Changed lines of the file:
@@
 P 2500 5950
 F 0 "U1" H 2500 6304 45  0000 C CNN
-F 1 "LM358" H 2500 6220 45  0000 C CNN
+F 1 "TS912IDT" H 2500 6220 45  0000 C CNN
 F 2 "Package_SO:SOIC-8_3.9x4.9mm_P1.27mm" H 2500 6300 20  0001 C CNN
 F 3 "" H 2500 5950 50  0001 C CNN
@@
 P 7600 5850
 F 0 "U1" H 7728 5892 45  0000 L CNN
-F 1 "LM358" H 7728 5808 45  0000 L CNN
+F 1 "TS912IDT" H 7728 5808 45  0000 L CNN
 F 2 "Package_SO:SOIC-8_3.9x4.9mm_P1.27mm" H 7600 6200 20  0001 C CNN
 F 3 "" H 7600 5850 50  0001 C CNN
