File: electronics/kicad/sig_gen/sig_gen.kicad_pcb (KiCad board)
At the start: 2 copper layers, 25 parts, among them J1 PDSE1, J2 CONN_01, J3 CONN_01, J4 CONN_01, J5 CONN_01, J6 CONN_01, J7 CONN_01, J8 CONN_01, J9 CONN_01, U1 L7805CV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

Commit message: HMC732
Parts:
- removed R12: 1k, Resistor_SMD:R_0603_1608Metric
- added C8: 0.1 uF, Capacitors:0603, F.Cu at (87.8, 103.3)
- added C9: 10 nF, Capacitors:0402, F.Cu at (100.0, 104.2)
- U1: value L7805CV -> LM7805; footprint digikey-footprints:TO-220-3 -> digikey-footprints:SOT-223
- moved R6 35.9 mm to (87.7, 77.8)
- moved R8 33.0 mm to (92.6, 77.9), turned to 90 degrees
- moved C4 31.8 mm to (57.2, 105.8)
- moved J5 31.5 mm to (66.2, 103.8)
- moved J9 21.9 mm to (91.8, 94.0)
- moved C7 18.5 mm to (95.2, 110.9)
- moved R10 14.5 mm to (83.5, 119.5)
- moved U1 11.0 mm to (78.2, 105.3)
- moved C1 10.6 mm to (78.7, 111.8)
- moved U5 9.17 mm to (87.1, 77.8), turned to 90 degrees
- moved C2 4.85 mm to (78.5, 113.8)
- moved J3 1.10 mm to (105.1, 104.2)
Connections:
- J3 pad 1: Net-(J3-Pad1) -> Net-(C9-Pad1)
- R8 pad 1: Net-(R12-Pad2) -> Vtune
- U2 pad 15: Net-(J3-Pad1) -> Net-(C9-Pad2)
- U5 pad 1: Net-(R12-Pad2) -> Vtune
Routing:
- net Net-(J3-Pad1): track 8.13 -> 0.00 mm
- net Net-(C9-Pad1): track 0.00 -> 4.10 mm
- net Net-(C9-Pad2): track 0.00 -> 3.25 mm
- removed copper zone on F.Cu, net GND

Commit message: VCO board done
Parts:
- removed C2, C3, C8: 0.1 uF, Capacitors:0603
- removed C4: 10 uF, Capacitors:0603
- removed J4, J5, J6, J7, J8, J9: CONN_01, Connectors2:1X01
- removed R10, R6: 1k, Resistor_SMD:R_0603_1608Metric
- removed R8: 10k, Resistor_SMD:R_0603_1608Metric
- removed U1: LM7805, digikey-footprints:SOT-223
- removed U3: MCP4725SOT-23, Silicon-Standard:SOT23-6
- removed U4: BA78M20FP, digikey-footprints:TO-252-3
- removed U5: TLV2172IDR, Package_SO:SOIC-8_3.9x4.9mm_P1.27mm
- C1: value 10uF -> 0.1 uF; footprint Capacitors:1206 -> Capacitors:0603
- C5: footprint Capacitors:0402 -> Capacitor_SMD:C_0402_1005Metric
- J1: value PDSE1 -> CONN_01; footprint Connectors2:1X04_SMD_RA_FEMALE -> TestPoint:TestPoint_Pad_1.5x1.5mm
- J2: footprint Connectors2:1X01 -> TestPoint:TestPoint_Pad_1.5x1.5mm
- moved C6 37.1 mm to (95.9, 113.8), turned to 0 degrees
- moved J1 27.9 mm to (94.5, 115.7)
- moved J2 16.0 mm to (85.1, 104.2)
- moved C5 13.6 mm to (94.7, 107.4)
- moved C1 10.7 mm to (87.0, 105.1), turned to 270 degrees
- moved C7 0.32 mm to (95.3, 111.2)
Connections:
- C1 pad 1: 20V -> Vtune
- J1 pad 1: GND -> 5V
- J2 pad 1: 12V -> Vtune
Routing:
- net 5V: track 0.00 -> 9.84 mm
- net GND: track 5.15 -> 14.1 mm
- net Vtune: track 0.00 -> 6.14 mm
- added copper zone on F.Cu, net GND
