File: electronics/kicad/sig_gen/sig_gen.sch (KiCad schematic (older format))
At the start: 26 parts, among them J1 PDSE1, J2 CONN_01, J3 CONN_01, J4 CONN_01, J5 CONN_01, J6 CONN_01, J7 CONN_01, J8 CONN_01, J9 CONN_01, U1 LM7805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

Commit message: VCO board done
Parts:
- removed C1: 10uF, 1206, symbol SparkFun-Capacitors:1.0UF-1206-50V-10%
- removed C2, C3, C8: 0.1 uF, 0603, symbol SparkFun-Capacitors:0.1UF-0603-25V-5%
- removed C4: 10 uF, 0603, symbol SparkFun-Capacitors:0.1UF-0603-25V-5%
- removed J1: PDSE1, Connectors2:1X04_SMD_RA_FEMALE, symbol w_connectors:HEADER_4
- removed J4, J5, J6, J7, J8, J9: CONN_01, 1X01, symbol SparkFun-Connectors:CONN_01
- removed R10, R6: 1k, Resistor_SMD:R_0603_1608Metric, symbol SparkFun-Resistors:RESISTOR0402
- removed R8: 10k, Resistor_SMD:R_0603_1608Metric, symbol SparkFun-Resistors:RESISTOR0402
- removed U1: LM7805, digikey-footprints:SOT-223, symbol dk_PMIC-Voltage-Regulators-Linear:LM7812CT_LTB
- removed U3: MCP4725SOT-23, SOT23-6, symbol SparkFun-IC-Conversion:MCP4725SOT-23
- removed U4: BA78M20FP, digikey-footprints:TO-252-3, symbol dk_PMIC-Voltage-Regulators-Linear:MC7805BDTRKG
- removed U5: TLV2172IDR, Package_SO:SOIC-8_3.9x4.9mm_P1.27mm, symbol SparkFun-IC-Amplifiers:LM358
- added C1: 0.1 uF, 0603, symbol SparkFun-Capacitors:0.1UF-0603-25V-5%
- added J1: CONN_01, TestPoint:TestPoint_Pad_1.5x1.5mm, symbol SparkFun-Connectors:CONN_01
- C5: footprint 0402 -> Capacitor_SMD:C_0402_1005Metric
- J2: footprint 1X01 -> TestPoint:TestPoint_Pad_1.5x1.5mm
Connections:
- net labels removed: 12V, 20V, 24V, 3.3V, varactor_pwm_input
- wire segments 9 -> 1
Other:
- note added: "On this part the N/C pins are truly not connected; for ease of layout they're manually set to ground on the PCB."
- moved on the sheet: C6, C7
