File: electronics/kicad/sig_gen_driver/sig_gen_driver.sch (KiCad schematic (older format))
At the start: 26 parts, among them J1 PDSE1, J2 CONN_01, J3 CONN_01, J4 CONN_01, J5 CONN_01, J6 CONN_01, J7 CONN_01, J8 CONN_01, J9 CONN_01, U1 LM7805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

Commit message: HMC732
Parts:
- removed C5, C9: 10 nF, 0402, symbol SparkFun-Capacitors:6PF-0402-50V-0.5%
- removed J3: CONN_01, TestPoint:TestPoint_Pad_1.5x1.5mm, symbol SparkFun-Connectors:CONN_01
- removed U2: HMC732, Package_DFN_QFN:QFN-24-1EP_4x4mm_P0.5mm_EP2.6x2.6mm, symbol 0xDBFB7:HMC732
Connections:
- wire segments 9 -> 8
Changed lines of the file:
@@
 Text GLabel 10200 1900 2    50   Input ~ 0
 20V
-$Comp
-L 0xDBFB7:HMC732 U2
-U 1 1 5F7369B2
-P 3800 2800
-F 0 "U2" H 3775 2765 50  0000 C CNN
-F 1 "HMC732" H 3775 2674 50  0000 C CNN
-F 2 "Package_DFN_QFN:QFN-24-1EP_4x4mm_P0.5mm_EP2.6x2.6mm" H 3800 2800 50  0001 C CNN
-F 3 "" H 3800 2800 50  0001 C CNN
-	1    3800 2800
-	1    0    0    -1
-$EndComp
 Connection ~ 7750 1450
 Wire Wire Line
@@
 	8100 1450 8150 1450
 $Comp
-L SparkFun-Capacitors:6PF-0402-50V-0.5% C5
-U 1 1 5F7AC4E2
-P 2850 3350
-F 0 "C5" H 2958 3442 45  0000 L CNN
-F 1 "10 nF" H 2958 3358 45  0000 L CNN
-F 2 "0402" H 2850 3600 20  0001 C CNN
-F 3 "" H 2850 3350 50  0001 C CNN
-F 4 "" H 2958 3316 60  0000 L CNN "Field4"
-	1    2850 3350
-	1    0    0    -1
-$EndComp
-$Comp
-L SparkFun-PowerSymbols:5V #SUPPLY0104
-U 1 1 5F7ADBAB
-P 3350 3250
-F 0 "#SUPPLY0104" H 3400 3250 45  0001 L BNN
-F 1 "5V" V 3350 3377 45  0000 L CNN
-F 2 "" V 3392 3378 60  0000 L CNN
-F 3 "" H 3350 3250 60  0001 C CNN
-	1    3350 3250
-	0    -1   -1   0
-$EndComp
-$Comp
-L SparkFun-PowerSymbols:5V #SUPPLY0105
-U 1 1 5F7AF25B
-P 2850 3150
-F 0 "#SUPPLY0105" H 2900 3150 45  0001 L BNN
-F 1 "5V" V 2850 3277 45  0000 L CNN
-F 2 "" V 2892 3278 60  0000 L CNN
-F 3 "" H 2850 3150 60  0001 C CNN
-	1    2850 3150
-	0    -1   -1   0
-$EndComp
-$Comp
 L SparkFun-Capacitors:1.0UF-1206-50V-10% C6
 U 1 1 5F7B2CE4
@@
 	0    1    -1   0
 $EndComp
-$Comp
-L power:GND #PWR0111
-U 1 1 5F7B3DBB
-P 3350 3350
-F 0 "#PWR0111" H 3350 3350 30  0001 C CNN
-F 1 "GND" H 3350 3280 30  0001 C CNN
-F 2 "" H 3350 3350 50  0001 C CNN
-F 3 "" H 3350 3350 50  0001 C CNN
-	1    3350 3350
-	0    1    1    0
-$EndComp
-$Comp
-L power:GND #PWR0112
-U 1 1 5F7B43A4
-P 3350 3450
-F 0 "#PWR0112" H 3350 3450 30  0001 C CNN
-F 1 "GND" H 3350 3380 30  0001 C CNN
-F 2 "" H 3350 3450 50  0001 C CNN
-F 3 "" H 3350 3450 50  0001 C CNN
-	1    3350 3450
-	0    1    1    0
-$EndComp
-Text GLabel 3350 3100 0    50   Input ~ 0
-Vtune
-$Comp
-L power:GND #PWR0114
-U 1 1 5F7B5B6D
-P 2850 3450
-F 0 "#PWR0114" H 2850 3450 30  0001 C CNN
-F 1 "GND" H 2850 3380 30  0001 C CNN
-F 2 "" H 2850 3450 50  0001 C CNN
-F 3 "" H 2850 3450 50  0001 C CNN
-	1    2850 3450
-	1    0    0    -1
-$EndComp
-$Comp
-L SparkFun-Connectors:CONN_01 J3
-U 1 1 5F7B6DAF
-P 4800 3250
-F 0 "J3" H 4758 3454 45  0000 C CNN
-F 1 "CONN_01" H 4758 3370 45  0000 C CNN
-F 2 "TestPoint:TestPoint_Pad_1.5x1.5mm" H 4800 3450 20  0001 C CNN
-F 3 "" H 4800 3250 50  0001 C CNN
-F 4 "" H 4758 3381 60  0000 C CNN "Field4"
-	1    4800 3250
-	-1   0    0    1
-$EndComp
-Wire Wire Line
-	4200 3250 4400 3250
 $Comp
 L SparkFun-PowerSymbols:3.3V #SUPPLY0108
@@
 	1    0    0    -1
 $EndComp
-$Comp
-L SparkFun-Capacitors:6PF-0402-50V-0.5% C9
-U 1 1 5F7EE8B4
-P 4500 3250
-F 0 "C9" H 4608 3342 45  0000 L CNN
-F 1 "10 nF" H 4608 3258 45  0000 L CNN
-F 2 "0402" H 4500 3500 20  0001 C CNN
-F 3 "" H 4500 3250 50  0001 C CNN
-F 4 "" H 4608 3216 60  0000 L CNN "Field4"
-	1    4500 3250
-	0    1    1    0
-$EndComp
 $EndSCHEMATC

Commit message: VCO board done
Parts:
- removed C6: 10uF, 1206, symbol SparkFun-Capacitors:1.0UF-1206-50V-10%
- added J10, J3: CONN_01, TestPoint:TestPoint_Pad_1.5x1.5mm, symbol SparkFun-Connectors:CONN_01
Connections:
- net 5V: now also J3.1
- net Vtune: now also J10.1
Other:
- moved on the sheet: C7
Changed lines of the file:
@@
 	8100 1450 8150 1450
-$Comp
-L SparkFun-Capacitors:1.0UF-1206-50V-10% C6
-U 1 1 5F7B2CE4
-P 3250 1500
-F 0 "C6" H 3358 1592 45  0000 L CNN
-F 1 "10uF" H 3358 1508 45  0000 L CNN
-F 2 "1206" H 3250 1750 20  0001 C CNN
-F 3 "" H 3250 1500 50  0001 C CNN
-F 4 "" H 3358 1466 60  0000 L CNN "Field4"
-	1    3250 1500
-	1    0    0    -1
-$EndComp
 $Comp
 L SparkFun-Capacitors:0.1UF-0603-25V-5% C7
 U 1 1 5F7B2CEB
-P 3700 1500
-F 0 "C7" H 3808 1592 45  0000 L CNN
-F 1 "0.1 uF" H 3808 1508 45  0000 L CNN
-F 2 "0603" H 3700 1750 20  0001 C CNN
-F 3 "" H 3700 1500 50  0001 C CNN
-F 4 "" H 3808 1466 60  0000 L CNN "Field4"
-	1    3700 1500
-	1    0    0    -1
-$EndComp
-$Comp
-L power:GND #PWR0102
-U 1 1 5F7B2CF1
-P 3250 1600
-F 0 "#PWR0102" H 3250 1600 30  0001 C CNN
-F 1 "GND" H 3250 1530 30  0001 C CNN
-F 2 "" H 3250 1600 50  0001 C CNN
-F 3 "" H 3250 1600 50  0001 C CNN
-	1    3250 1600
+P 3400 1500
+F 0 "C7" H 3508 1592 45  0000 L CNN
+F 1 "0.1 uF" H 3508 1508 45  0000 L CNN
+F 2 "0603" H 3400 1750 20  0001 C CNN
+F 3 "" H 3400 1500 50  0001 C CNN
+F 4 "" H 3508 1466 60  0000 L CNN "Field4"
+	1    3400 1500
 	1    0    0    -1
 $EndComp
@@
 L power:GND #PWR0103
 U 1 1 5F7B2CF7
-P 3700 1600
-F 0 "#PWR0103" H 3700 1600 30  0001 C CNN
-F 1 "GND" H 3700 1530 30  0001 C CNN
-F 2 "" H 3700 1600 50  0001 C CNN
-F 3 "" H 3700 1600 50  0001 C CNN
-	1    3700 1600
+P 3400 1600
+F 0 "#PWR0103" H 3400 1600 30  0001 C CNN
+F 1 "GND" H 3400 1530 30  0001 C CNN
+F 2 "" H 3400 1600 50  0001 C CNN
+F 3 "" H 3400 1600 50  0001 C CNN
+	1    3400 1600
 	1    0    0    -1
 $EndComp
@@
 L SparkFun-PowerSymbols:5V #SUPPLY0106
 U 1 1 5F7B2D77
-P 3700 1300
-F 0 "#SUPPLY0106" H 3750 1300 45  0001 L BNN
-F 1 "5V" V 3700 1428 45  0000 L CNN
-F 2 "" V 3742 1428 60  0000 L CNN
-F 3 "" H 3700 1300 60  0001 C CNN
-	1    3700 1300
-	0    1    -1   0
-$EndComp
-$Comp
-L SparkFun-PowerSymbols:5V #SUPPLY0107
-U 1 1 5F7B326C
-P 3250 1300
-F 0 "#SUPPLY0107" H 3300 1300 45  0001 L BNN
-F 1 "5V" V 3250 1428 45  0000 L CNN
-F 2 "" V 3292 1428 60  0000 L CNN
-F 3 "" H 3250 1300 60  0001 C CNN
-	1    3250 1300
+P 3400 1300
+F 0 "#SUPPLY0106" H 3450 1300 45  0001 L BNN
+F 1 "5V" V 3400 1428 45  0000 L CNN
+F 2 "" V 3442 1428 60  0000 L CNN
+F 3 "" H 3400 1300 60  0001 C CNN
+	1    3400 1300
 	0    1    -1   0
 $EndComp
@@
 	1    0    0    -1
 $EndComp
+$Comp
+L SparkFun-Connectors:CONN_01 J10
+U 1 1 5F819631
+P 9650 1350
+F 0 "J10" H 9608 1554 45  0000 C CNN
+F 1 "CONN_01" H 9608 1470 45  0000 C CNN
+F 2 "TestPoint:TestPoint_Pad_1.5x1.5mm" H 9650 1550 20  0001 C CNN
+F 3 "" H 9650 1350 50  0001 C CNN
+F 4 "" H 9608 1481 60  0000 C CNN "Field4"
+	1    9650 1350
+	-1   0    0    -1
+$EndComp
+Text GLabel 9550 1350 0    50   Input ~ 0
+Vtune
+$Comp
+L SparkFun-Connectors:CONN_01 J3
+U 1 1 5F81A425
+P 3850 1950
+F 0 "J3" H 3808 2154 45  0000 C CNN
+F 1 "CONN_01" H 3808 2070 45  0000 C CNN
+F 2 "TestPoint:TestPoint_Pad_1.5x1.5mm" H 3850 2150 20  0001 C CNN
+F 3 "" H 3850 1950 50  0001 C CNN
+F 4 "" H 3808 2081 60  0000 C CNN "Field4"
+	1    3850 1950
+	-1   0    0    -1
+$EndComp
+$Comp
+L SparkFun-PowerSymbols:5V #SUPPLY0104
+U 1 1 5F81BBA7
+P 3750 1950
+F 0 "#SUPPLY0104" H 3800 1950 45  0001 L BNN
+F 1 "5V" V 3750 2078 45  0000 L CNN
+F 2 "" V 3792 2078 60  0000 L CNN
+F 3 "" H 3750 1950 60  0001 C CNN
+	1    3750 1950
+	0    -1   1    0
+$EndComp
 $EndSCHEMATC
