File: electronics/kicad/amplifier/amplifier.kicad_pcb (KiCad board)
At the start: 2 copper layers, 10 parts, among them J1 CONSMA001-SMD-G, U1 BFP620

Commit message: Amplifier
Parts:
- added C1: 100 nF, Capacitors:0603, F.Cu at (148.1, 109.0)
- added U2: CE3520K3, 0xDBFB7:4-Micro-X, F.Cu at (162.7, 82.7)
- C3: value 0.1 uF -> 100 nF
- R1: value RESISTOR0402 -> 10k
- moved C3 19.3 mm to (153.1, 100.6), turned to 180 degrees
- moved J1 17.5 mm to (141.5, 106.6)
- moved R1 16.7 mm to (147.2, 107.5), turned to 270 degrees
- moved TPOP1 16.3 mm to (159.8, 104.6)
- moved TPSO2 15.5 mm to (147.2, 113.2)
- moved U1 10.2 mm to (150.3, 105.5), turned to 90 degrees
- moved C4 8.72 mm to (155.1, 104.6)
- moved TPSO1 7.04 mm to (150.8, 100.3)
- moved L2 5.27 mm to (151.0, 101.9), turned to 270 degrees
- moved L3 4.88 mm to (151.0, 103.5), turned to 270 degrees
Connections:
- J1 pad 1: Net-(J1-Pad1) -> GND
Routing:
- net GND: track 0.00 -> 37.2 mm
- net Net-(J1-Pad2): track 0.00 -> 7.65 mm
- net Net-(C1-Pad1): track 0.00 -> 5.19 mm
- net Net-(C4-Pad2): track 0.00 -> 3.45 mm
- net Net-(C4-Pad1): track 0.00 -> 2.95 mm
- net Net-(L2-Pad2): track 0.00 -> 0.63 mm
- added copper zone on F.Cu, net GND

Commit message: S2p
Parts:
- moved U2 21.0 mm to (164.0, 103.6)
Changed lines of the file:
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@@
   )
   (module 0xDBFB7:4-Micro-X (layer F.Cu)
-    (at 162.65 82.65)
+    (at 164 103.6)
     (fp_text reference U2 (at 0 5.072) (layer F.SilkS)
       (effects (font (size 1 1) (thickness 0.15)))
