File: electronics/kicad/amplifier_stage_2/amplifier.sch (KiCad schematic (older format))
At the start: 10 parts, among them U1 BFP620, U2 CE3520K3

Commit message: Pulser working fine
Parts:
- gave numbers to parts that had none: 1
Changed lines of the file:
@@
 $EndComp
 $Comp
-L Connector:Test_Point TPOP?
+L Connector:Test_Point TPOP2
 U 1 1 5F97D0D2
 P 2950 2900
-F 0 "TPOP?" V 3145 2972 50  0000 C CNN
+F 0 "TPOP2" V 3145 2972 50  0000 C CNN
 F 1 "Voutput" V 3054 2972 50  0000 C CNN
 F 2 "TestPoint:TestPoint_Pad_1.5x1.5mm" H 3150 2900 50  0001 C CNN
