File: electronics/kicad/coplanar_amplifier/coplanar_amplifier.sch (KiCad schematic (older format))
At the start: 11 parts, among them U2 CE3520K3

Commit message: Writing the protocol
Parts:
- gave numbers to parts that had none: 1
Other:
- note removed: "The small gap between the board and this SMD connector is\na bit concerning; some sort of resonance could probably be set up\nin there."
Changed lines of the file:
@@
 	1    0    0    -1
 $EndComp
-Text Notes 1100 4350 0    50   ~ 0
-The small gap between the board and this SMD connector is\na bit concerning; some sort of resonance could probably be set up\nin there.
 $Comp
 L 0xDBFB7:CE3520K3 U2
@@
 $EndComp
 $Comp
-L SparkFun-Capacitors:4.7UF0603 C?
+L SparkFun-Capacitors:4.7UF0603 C5
 U 1 1 5F355F2B
 P 4150 2300
-F 0 "C?" V 3916 2350 45  0000 C CNN
+F 0 "C5" V 3916 2350 45  0000 C CNN
 F 1 "100 nF" V 4000 2350 45  0000 C CNN
 F 2 "Resistor_SMD:R_0402_1005Metric" H 4150 2550 20  0001 C CNN
@@
 $EndComp
 $Comp
-L power:GND #PWR?
+L power:GND #PWR0103
 U 1 1 5F3567EF
 P 4350 2300
-F 0 "#PWR?" H 4350 2300 30  0001 C CNN
+F 0 "#PWR0103" H 4350 2300 30  0001 C CNN
 F 1 "GND" H 4350 2230 30  0001 C CNN
 F 2 "" H 4350 2300 50  0001 C CNN
