File: electronics/kicad/freq_prescaler/freq_prescaler.kicad_pcb (KiCad board)
At the start: 2 copper layers, 38 parts, among them P1 CONN_1, P2 OUTPUT, P3 OUTPUT, P4 OUTPUT, P5 OUTPUT, U1 SY100EP, U2 HMC363, U3 SY100EP, U4 SY100EP, U5 SKY65013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

Commit message: Amplifier
Parts:
- moved P4 0.60 mm to (101.5, 78.1)
Routing:
- net 5V: track 4.87 -> 6.92 mm
- net Net-(C7-Pad2): track 0.00 -> 1.94 mm
- net Net-(U3-Pad3): track 0.00 -> 1.27 mm
- net Net-(C4-Pad1): track 4.74 -> 6.01 mm
- net Net-(C9-Pad2): track 5.08 -> 6.14 mm
- net Net-(C10-Pad2): track 2.36 -> 3.14 mm
Changed lines of the file:
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@@
     (thickness 1.6)
     (drawings 0)
-    (tracks 98)
+    (tracks 108)
     (zones 0)
     (modules 38)
@@
       (creategerberjobfile false)
       (excludeedgelayer true)
-      (linewidth 0.010000)
+      (linewidth 0.150000)
       (plotframeref false)
       (viasonmask false)
@@
   )
   (module Connector_PinHeader_2.54mm:PinHeader_1x01_P2.54mm_Vertical (layer F.Cu)
-    (at 102.1 78.1)
+    (at 101.5 78.1)
     (descr "Through hole straight pin header, 1x01, 2.54mm pitch, single row")
     (tags "Through hole pin header THT 1x01 2.54mm single row")
@@
   (segment (start 96.614999 67.05588) (end 97.520879 66.15) (width 0.4) (layer F.Cu) (net 7))
   (segment (start 96.614999 68.200001) (end 96.614999 67.05588) (width 0.4) (layer F.Cu) (net 7))
+  (segment (start 95.344999 68.200001) (end 96.614999 68.200001) (width 0.25) (layer F.Cu) (net 7))
   (segment (start 87.23844 84.30656) (end 87.245 84.3) (width 0.4) (layer F.Cu) (net 8))
   (segment (start 85.65 84.30656) (end 87.23844 84.30656) (width 0.4) (layer F.Cu) (net 8))
@@
   (segment (start 84.75089 74.70089) (end 84.1 74.05) (width 0.4) (layer F.Cu) (net 8))
   (segment (start 84.75089 76.151551) (end 84.75089 74.70089) (width 0.4) (layer F.Cu) (net 8))
+  (segment (start 81.03588 63.635) (end 80.95 63.72088) (width 0.4) (layer F.Cu) (net 9))
+  (segment (start 82.85 63.635) (end 81.03588 63.635) (width 0.4) (layer F.Cu) (net 9))
   (segment (start 88.45 57.45) (end 90.45 59.45) (width 1.5) (layer F.Cu) (net 10))
   (segment (start 88.45 55.2) (end 88.45 57.45) (width 1.5) (layer F.Cu) (net 10))
+  (segment (start 90.55 59.55) (end 90.45 59.45) (width 0.4) (layer F.Cu) (net 10))
+  (segment (start 90.55 60.47088) (end 90.55 59.55) (width 0.4) (layer F.Cu) (net 10))
   (segment (start 90.55 62.37912) (end 90.57088 62.4) (width 0.4) (layer F.Cu) (net 11))
   (segment (start 90.53588 62.365) (end 90.57088 62.4) (width 0.4) (layer F.Cu) (net 11))
   (segment (start 88.25 62.365) (end 90.53588 62.365) (width 0.4) (layer F.Cu) (net 11))
+  (segment (start 90.57088 61.65) (end 90.55 61.62912) (width 0.4) (layer F.Cu) (net 11))
+  (segment (start 90.57088 62.4) (end 90.57088 61.65) (width 0.4) (layer F.Cu) (net 11))
   (segment (start 93.29 62.4) (end 93.35 62.46) (width 0.4) (layer F.Cu) (net 12))
   (segment (start 91.72912 62.4) (end 93.29 62.4) (width 0.4) (layer F.Cu) (net 12))
@@
   (segment (start 98.75 56.95164) (end 98.69836 56.9) (width 0.4) (layer F.Cu) (net 13))
   (segment (start 98.75 58.40084) (end 98.75 56.95164) (width 0.4) (layer F.Cu) (net 13))
+  (segment (start 86.805 59.65) (end 88.25 61.095) (width 0.4) (layer F.Cu) (net 13))
+  (segment (start 86.79836 59.65) (end 86.805 59.65) (width 0.4) (layer F.Cu) (net 13))
   (segment (start 98.75 64.12088) (end 98.7 64.17088) (width 0.4) (layer F.Cu) (net 14))
   (segment (start 98.75 62.67912) (end 98.75 64.12088) (width 0.4) (layer F.Cu) (net 14))
@@
   (segment (start 88.515 82.385841) (end 88.50084 82.400001) (width 0.4) (layer F.Cu) (net 22))
   (segment (start 88.515 80.55) (end 88.515 82.385841) (width 0.4) (layer F.Cu) (net 22))
+  (segment (start 95.345 77.4) (end 96.615 77.4) (width 0.25) (layer F.Cu) (net 26))
   (segment (start 91.055 89.7) (end 89.785 89.7) (width 0.4) (layer F.Cu) (net 32))
   (segment (start 89.785 80.55) (end 91.055 80.55) (width 0.4) (layer F.Cu) (net 35))
@@
     (polygon
       (pts
-        (xy 103.975 98.3) (xy 73.125 98.3) (xy 73.075 49.2) (xy 104.025 49.2)
+        (xy 105.1 94.8) (xy 69 94.9) (xy 68.9 64.8) (xy 75.2 64.8) (xy 75.1 62.1)
+        (xy 79.7 62.1) (xy 79.7 63.7) (xy 82.2 63.7) (xy 82.15 54.4) (xy 84.85 54.4)
+        (xy 84.9 61) (xy 93.8 61) (xy 93.8 54.4) (xy 105 54.4)
       )
     )

Commit message: Progress
Parts:
- removed C1, C3, C5, C9: 100 pF, Capacitors:0402
- removed HACKRF1: HACKRF, TestPoint:TestPoint_Pad_1.5x1.5mm
- moved P1 37.1 mm to (77.6, 97.3), turned to 90 degrees
- moved P3 36.1 mm to (72.6, 77.7), turned to 90 degrees
- moved P2 34.9 mm to (96.9, 106.0), turned to 90 degrees
- moved C2 31.7 mm to (77.6, 92.7), turned to 270 degrees
- moved R2 31.4 mm to (75.6, 90.5), turned to 90 degrees
- moved C15 29.5 mm to (99.8, 101.9), turned to 90 degrees
- moved C12 25.8 mm to (73.4, 65.2), turned to 270 degrees
- moved C16 24.5 mm to (76.2, 82.2), turned to 270 degrees
- moved R5 23.5 mm to (75.8, 64.2), turned to 180 degrees
- moved U7 23.4 mm to (96.2, 100.2), turned to 270 degrees
- moved C7 22.9 mm to (80.8, 87.2), turned to 180 degrees
- moved P5 22.3 mm to (103.5, 82.2), turned to 270 degrees
- moved U2 20.5 mm to (79.5, 82.5), turned to 270 degrees
- moved L1 20.3 mm to (78.6, 64.2), turned to 0 degrees
- moved C14 19.6 mm to (79.2, 62.8), turned to 270 degrees
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Connections:
- R2 pad 2: Net-(C3-Pad1) -> Net-(R2-Pad2)
- U2 pad 5: Net-(C3-Pad2) -> Net-(R2-Pad2)
Routing:
- net GND: track 4.31 -> 41.6 mm
- net 3.3V: track 75.0 -> 52.7 mm
- net 5V: track 6.92 -> 24.9 mm
- net Net-(R8-Pad1): track 17.9 -> 3.80 mm
- net DIV8_OUT: track 3.21 -> 13.9 mm
- net Net-(C1-Pad2): track 8.70 -> 0.00 mm
- net Net-(C9-Pad2): track 6.14 -> 0.00 mm
- net Net-(C10-Pad1): track 1.65 -> 6.46 mm
- net Net-(R2-Pad2): track 0.00 -> 3.69 mm
- net Net-(C3-Pad2): track 2.07 -> 0.00 mm
- net Net-(C3-Pad1): track 1.62 -> 0.00 mm
- net Net-(C14-Pad2): track 4.00 -> 2.52 mm
- net Net-(C4-Pad1): track 6.01 -> 4.81 mm
- net Net-(C10-Pad2): track 3.14 -> 2.36 mm

Commit message: coplanarizing further
Parts:
- removed P3: OUTPUT, Connector_PinHeader_2.54mm:PinHeader_1x01_P2.54mm_Vertical
- added C1: 1 nF, Capacitor_SMD:C_0402_1005Metric, F.Cu at (93.1, 33.3)
- added C17: 1 nF, Capacitor_SMD:C_0402_1005Metric, F.Cu at (99.8, 55.8)
- added C18: 1 nF, Capacitor_SMD:C_0402_1005Metric, F.Cu at (99.8, 64.8)
- added C19: 1 nF, Capacitor_SMD:C_0402_1005Metric, F.Cu at (99.8, 74.1)
- added C20: 1 nF, Capacitor_SMD:C_0402_1005Metric, F.Cu at (99.8, 83.2)
- added C21: 1 nF, Capacitor_SMD:C_0402_1005Metric, F.Cu at (99.8, 92.3)
- added C22: 1 nF, Capacitor_SMD:C_0402_1005Metric, F.Cu at (82.5, 34.4)
- added C23: 1 nF, Capacitor_SMD:C_0402_1005Metric, F.Cu at (85.0, 34.4)
- added C3: 1 nF, Capacitor_SMD:C_0402_1005Metric, F.Cu at (94.7, 35.6)
- added C35: 100 nF, Capacitors:0603, F.Cu at (84.2, 27.5)
- added C36: 1 nF, Resistor_SMD:R_0402_1005Metric, F.Cu at (83.7, 31.3)
- added C5: 1 nF, Capacitor_SMD:C_0402_1005Metric, F.Cu at (97.8, 45.1)
- added C9: 1 nF, Capacitor_SMD:C_0402_1005Metric, F.Cu at (96.2, 47.7)
- added D3: BAT15-04, Package_TO_SOT_SMD:SOT-23, F.Cu at (83.7, 33.3)
- added P6: CONN_1, TestPoint:TestPoint_Pad_1.5x1.5mm, F.Cu at (104.9, 55.0)
- added P7: CONN_1, TestPoint:TestPoint_Pad_1.5x1.5mm, F.Cu at (91.1, 32.7)
- added P8: a, TestPoint:TestPoint_Pad_1.5x1.5mm, F.Cu at (82.1, 27.4)
- added R18: 10k, Resistor_SMD:R_0402_1005Metric, F.Cu at (83.7, 30.2)
- added R3: 10k, Resistor_SMD:R_0402_1005Metric, F.Cu at (83.2, 28.7)
- C10, C14, C2, C7: value 100 pF -> 1 nF; footprint Capacitors:0402 -> Capacitor_SMD:C_0402_1005Metric
- L1, R1: footprint Capacitors:0402 -> Capacitor_SMD:C_0402_1005Metric
- P1: footprint TestPoint:TestPoint_Pad_1.5x1.5mm -> TestPoint:TestPoint_Pad_1.0x1.0mm
- P5: value OUTPUT -> CONN_1; footprint Connector_PinHeader_2.54mm:PinHeader_1x01_P2.54mm_Vertical -> TestPoint:TestPoint_Pad_1.5x1.5mm
- R6, R7, R8, R9: value 50 -> 100
- moved P1 63.0 mm to (75.6, 34.3), turned to 0 degrees
- moved C2 58.3 mm to (78.3, 34.3), turned to 180 degrees
- moved R2 58.3 mm to (79.6, 32.3), turned to 0 degrees
- moved C16 51.1 mm to (89.0, 32.7), turned to 180 degrees
- moved C7 50.5 mm to (86.2, 36.9)
- moved U2 47.6 mm to (90.4, 36.3), turned to 180 degrees
- moved R4 40.3 mm to (94.5, 39.1), turned to 90 degrees
- moved P5 39.7 mm to (103.5, 42.5), turned to 0 degrees
- moved C10 38.9 mm to (99.6, 44.1)
- moved U5 38.5 mm to (99.8, 37.1), turned to 0 degrees
- moved C12 36.1 mm to (102.3, 43.6)
- moved R5 32.8 mm to (100.5, 42.7), turned to 0 degrees
- moved C14 29.6 mm to (99.7, 41.3)
- moved L1 29.3 mm to (98.5, 42.7), turned to 180 degrees
- moved P4 13.4 mm to (92.8, 54.8)
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Connections:
- C10 pad 2: Net-(C10-Pad2) -> GND
- C11 pad 1: 3.3V -> 5V
- C13 pad 1: 3.3V -> 5V
- C14 pad 1: DIV8_OUT -> GND
- C14 pad 2: Net-(C14-Pad2) -> Net-(C10-Pad1)
- C15 pad 1: 3.3V -> 5V
- C6 pad 1: 3.3V -> 5V
- C7 pad 1: GND -> Net-(C7-Pad1)
- C7 pad 2: Net-(C7-Pad2) -> GND
- C8 pad 1: 3.3V -> 5V
- L1 pad 1: Net-(L1-Pad1) -> Net-(C10-Pad1)
- L1 pad 2: Net-(C14-Pad2) -> Net-(C5-Pad2)
- P5 pad 1: 3.3V -> 5V
- R2 pad 2: Net-(R2-Pad2) -> Net-(C22-Pad2)
- R5 pad 1: Net-(L1-Pad1) -> Net-(C10-Pad1)
- U1 pad 8: 3.3V -> 5V
- U2 pad 3: Net-(C10-Pad2) -> Net-(C3-Pad2)
- U2 pad 5: Net-(R2-Pad2) -> Net-(C23-Pad1)
- U2 pad 7: Net-(C7-Pad2) -> Net-(C7-Pad1)
- U3 pad 8: 3.3V -> 5V
- U4 pad 8: 3.3V -> 5V
- U5 pad 1: Net-(C10-Pad1) -> Net-(C3-Pad1)
- U5 pad 3: Net-(C14-Pad2) -> Net-(C5-Pad2)
- U6 pad 8: 3.3V -> 5V
- U7 pad 8: 3.3V -> 5V
Routing:
- net 3.3V: track 52.7 -> 0.00 mm
- net 5V: track 24.9 -> 74.4 mm
- net GND: track 41.6 -> 6.36 mm
- net DIV8_OUT: track 13.9 -> 4.06 mm
- net Net-(C10-Pad1): track 6.46 -> 0.00 mm
- net Net-(C5-Pad2): track 0.00 -> 5.65 mm
- net Net-(R2-Pad2): track 3.69 -> 0.00 mm
- net Net-(C36-Pad1): track 0.00 -> 3.31 mm
- net Net-(C14-Pad2): track 2.52 -> 0.00 mm
- net Net-(C3-Pad1): track 0.00 -> 2.39 mm
- net Net-(C10-Pad2): track 2.36 -> 0.00 mm
- net Net-(C23-Pad1): track 0.00 -> 2.24 mm
- net Net-(C7-Pad2): track 1.94 -> 0.00 mm
- net Net-(C2-Pad2): track 3.40 -> 1.90 mm
- net Net-(L1-Pad1): track 1.32 -> 0.00 mm
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
Commit message: d
Parts:
- removed C2, C23: 1 nF, Capacitor_SMD:C_0402_1005Metric
- removed R2: PAT1220, 0xDBFB7:PAT1220
- P2, P4: footprint Connector_PinHeader_2.54mm:PinHeader_1x01_P2.54mm_Vertical -> TestPoint:TestPoint_Pad_2.5x2.5mm
- P5, P7, P8: footprint TestPoint:TestPoint_Pad_1.5x1.5mm -> TestPoint:TestPoint_Pad_2.5x2.5mm
- moved P1 4.06 mm to (79.6, 34.3)
- moved P7 0.99 mm to (91.2, 31.7)
- moved P8 0.43 mm to (81.9, 27.0)
- moved C12 0.30 mm to (102.3, 43.9)
Connections:
- D3 pad 1: GND -> Net-(D3-Pad1)
- P1 pad 1: Net-(C2-Pad2) -> Net-(C22-Pad2)
- U2 pad 5: Net-(C23-Pad1) -> Net-(C22-Pad1)
Routing:
- net Net-(C22-Pad1): track 0.00 -> 3.65 mm
- net Net-(C23-Pad1): track 2.24 -> 0.00 mm
- net 5V: track 74.4 -> 76.6 mm
- net Net-(C2-Pad2): track 1.90 -> 0.00 mm
- net Net-(C22-Pad2): track 0.86 -> 1.91 mm
- net Net-(C2-Pad1): track 0.84 -> 0.00 mm
