File: electronics/kicad/freq_prescaler/freq_prescaler.sch (KiCad schematic (older format))
At the start: 38 parts, among them P1 CONN_1, P2 OUTPUT, P3 OUTPUT, P4 OUTPUT, P5 OUTPUT, U1 SY100EP, U2 HMC363, U3 SY100EP, U4 SY100EP, U5 SKY65013, U6 SY100EP, U7 SY100EP

Commit message: Progress
Parts:
- removed C1, C3, C5, C9: 100 pF, 0402, symbol SparkFun-Capacitors:6PF-0402-50V-0.5%
- removed HACKRF1: HACKRF, TestPoint:TestPoint_Pad_1.5x1.5mm, symbol conn:CONN_1
Connections:
- net at U2.5 (IN): now also R2.2
Other:
- moved on the sheet: C2, P1, R2
Changed lines of the file:
@@
 L 0xDBFB7:attenuator R2
 U 1 1 5F838885
-P 2100 2250
-F 0 "R2" H 2125 2465 50  0000 C CNN
-F 1 "PAT1220" H 2125 2374 50  0000 C CNN
-F 2 "0xDBFB7:PAT1220" H 2100 2250 50  0001 C CNN
-F 3 "" H 2100 2250 50  0001 C CNN
-F 4 "-10 dBm" H 2125 2283 50  0000 C CNN "Field4"
-	1    2100 2250
+P 2400 2250
+F 0 "R2" H 2425 2465 50  0000 C CNN
+F 1 "PAT1220" H 2425 2374 50  0000 C CNN
+F 2 "0xDBFB7:PAT1220" H 2400 2250 50  0001 C CNN
+F 3 "" H 2400 2250 50  0001 C CNN
+F 4 "-10 dBm" H 2425 2283 50  0000 C CNN "Field4"
+	1    2400 2250
 	1    0    0    -1
 $EndComp
@@
 $EndComp
 $Comp
-L SparkFun-Capacitors:6PF-0402-50V-0.5% C9
-U 1 1 5F83E862
-P 4600 2250
-F 0 "C9" H 4492 2258 45  0000 R CNN
-F 1 "100 pF" H 4492 2342 45  0000 R CNN
-F 2 "0402" H 4600 2500 20  0001 C CNN
-F 3 "" H 4600 2250 50  0001 C CNN
-F 4 "" V 4439 2300 60  0000 C CNN "Field4"
-	1    4600 2250
-	-1   0    0    1
-$EndComp
-$Comp
-L conn:CONN_1 HACKRF1
-U 1 1 5F83F2CD
-P 4600 1700
-F 0 "HACKRF1" V 4533 1641 40  0000 R CNN
-F 1 "HACKRF" H 4550 1740 30  0001 C CNN
-F 2 "TestPoint:TestPoint_Pad_1.5x1.5mm" H 4600 1700 50  0001 C CNN
-F 3 "" H 4600 1700 50  0001 C CNN
-	1    4600 1700
-	0    -1   -1   0
-$EndComp
-$Comp
 L SparkFun-PowerSymbols:5V #SUPPLY0101
 U 1 1 5F83FB00
@@
 L power:GND #PWR0103
 U 1 1 5F842A34
-P 1900 2500
-F 0 "#PWR0103" H 1900 2500 30  0001 C CNN
-F 1 "GND" H 1900 2430 30  0001 C CNN
-F 2 "" H 1900 2500 50  0001 C CNN
-F 3 "" H 1900 2500 50  0001 C CNN
-	1    1900 2500
-	0    1    1    0
-$EndComp
-Wire Wire Line
-	4600 2150 4600 1850
-Wire Wire Line
-	4600 2450 5100 2450
+P 2200 2500
+F 0 "#PWR0103" H 2200 2500 30  0001 C CNN
+F 1 "GND" H 2200 2430 30  0001 C CNN
+F 2 "" H 2200 2500 50  0001 C CNN
+F 3 "" H 2200 2500 50  0001 C CNN
+	1    2200 2500
+	0    1    1    0
+$EndComp
 Wire Wire Line
 	5400 2450 5550 2450
 Text Notes 950  3550 0    50   ~ 0
 O/P is -9 to -6 dBm, too low for the logic levels of the \nSY.
-Wire Wire Line
-	4150 2450 4600 2450
-Connection ~ 4600 2450
 $Comp
 L conn:CONN_1 P1
 U 1 1 5F844EAC
-P 800 2350
-F 0 "P1" H 733 2253 40  0000 C CNN
-F 1 "CONN_1" H 750 2390 30  0001 C CNN
-F 2 "TestPoint:TestPoint_Pad_1.5x1.5mm" H 800 2350 50  0001 C CNN
-F 3 "" H 800 2350 50  0001 C CNN
-	1    800  2350
+P 1100 2350
+F 0 "P1" H 1033 2253 40  0000 C CNN
+F 1 "CONN_1" H 1050 2390 30  0001 C CNN
+F 2 "TestPoint:TestPoint_Pad_1.5x1.5mm" H 1100 2350 50  0001 C CNN
+F 3 "" H 1100 2350 50  0001 C CNN
+	1    1100 2350
 	-1   0    0    1
 $EndComp
@@
 L SparkFun-Capacitors:6PF-0402-50V-0.5% C2
 U 1 1 5F84D039
-P 1550 2350
-F 0 "C2" V 1400 2400 45  0000 C CNN
-F 1 "100 pF" V 1316 2400 45  0000 C CNN
-F 2 "0402" H 1550 2600 20  0001 C CNN
-F 3 "" H 1550 2350 50  0001 C CNN
-F 4 "" V 1389 2400 60  0000 C CNN "Field4"
-	1    1550 2350
+P 1850 2350
+F 0 "C2" V 1700 2400 45  0000 C CNN
+F 1 "100 pF" V 1616 2400 45  0000 C CNN
+F 2 "0402" H 1850 2600 20  0001 C CNN
+F 3 "" H 1850 2350 50  0001 C CNN
+F 4 "" V 1689 2400 60  0000 C CNN "Field4"
+	1    1850 2350
 	0    1    -1   0
 $EndComp
-$Comp
-L SparkFun-Capacitors:6PF-0402-50V-0.5% C1
-U 1 1 5F84DFD2
-P 1450 2150
-F 0 "C1" H 1558 2158 45  0000 L CNN
-F 1 "100 pF" H 1558 2242 45  0000 L CNN
-F 2 "0402" H 1450 2400 20  0001 C CNN
-F 3 "" H 1450 2150 50  0001 C CNN
-F 4 "" V 1289 2200 60  0000 C CNN "Field4"
-	1    1450 2150
-	-1   0    0    1
-$EndComp
-$Comp
-L SparkFun-Capacitors:6PF-0402-50V-0.5% C5
-U 1 1 5F84F096
-P 2650 2150
-F 0 "C5" H 2542 2158 45  0000 R CNN
-F 1 "100 pF" H 2542 2242 45  0000 R CNN
-F 2 "0402" H 2650 2400 20  0001 C CNN
-F 3 "" H 2650 2150 50  0001 C CNN
-F 4 "" V 2489 2200 60  0000 C CNN "Field4"
-	1    2650 2150
-	-1   0    0    1
-$EndComp
-$Comp
-L SparkFun-Capacitors:6PF-0402-50V-0.5% C3
-U 1 1 5F8558E2
-P 2550 2350
-F 0 "C3" V 2400 2400 45  0000 C CNN
-F 1 "100 pF" V 2316 2400 45  0000 C CNN
-F 2 "0402" H 2550 2600 20  0001 C CNN
-F 3 "" H 2550 2350 50  0001 C CNN
-F 4 "" V 2389 2400 60  0000 C CNN "Field4"
-	1    2550 2350
-	0    -1   -1   0
-$EndComp
-Connection ~ 2650 2350
-Wire Wire Line
-	1900 2350 1750 2350
-Wire Wire Line
-	1450 1950 2650 1950
+Wire Wire Line
+	2200 2350 2050 2350
 $Comp
 L power:GND #PWR0104
@@
 $EndComp
 Wire Wire Line
-	2650 2050 2650 1950
-Wire Wire Line
-	1450 2050 1450 1950
-Wire Wire Line
-	950  2350 1450 2350
-Connection ~ 1450 2350
+	1250 2350 1750 2350
 $Comp
 L SparkFun-Resistors:0.22OHM-0805-1_4W-1% R4
@@
 	1    0    0    -1
 $EndComp
+Wire Wire Line
+	4150 2450 5100 2450
 $EndSCHEMATC

Commit message: coplanarizing further
Parts:
- removed P3: OUTPUT, Connector_PinHeader_2.54mm:PinHeader_1x01_P2.54mm_Vertical, symbol conn:CONN_1
- added C1, C17, C18, C19, C20, C21, C22, C23, C3, C5, C9: 1 nF, Capacitor_SMD:C_0402_1005Metric, symbol SparkFun-Capacitors:6PF-0402-50V-0.5%
- added C35: 100 nF, 0603, symbol SparkFun-Capacitors:4.7UF0603
- added C36: 1 nF, Resistor_SMD:R_0402_1005Metric, symbol SparkFun-Capacitors:6PF-0402-50V-0.5%
- added D3: BAT15-04, Package_TO_SOT_SMD:SOT-23, symbol Diode:BAS40-04
- added P6, P7: CONN_1, TestPoint:TestPoint_Pad_1.5x1.5mm, symbol conn:CONN_1
- added P8: a, TestPoint:TestPoint_Pad_1.5x1.5mm, symbol conn:CONN_1
- added R18, R3: 10k, Resistor_SMD:R_0402_1005Metric, symbol SparkFun-Resistors:RESISTOR0402
- C10, C14, C2, C7: value 100 pF -> 1 nF; footprint 0402 -> Capacitor_SMD:C_0402_1005Metric
- L1, R1: footprint 0402 -> Capacitor_SMD:C_0402_1005Metric
- P1: footprint TestPoint:TestPoint_Pad_1.5x1.5mm -> TestPoint:TestPoint_Pad_1.0x1.0mm
- P5: value OUTPUT -> CONN_1; footprint Connector_PinHeader_2.54mm:PinHeader_1x01_P2.54mm_Vertical -> TestPoint:TestPoint_Pad_1.5x1.5mm
- R6, R7, R8, R9: value 50 -> 100
Connections:
- net 3.3V is gone; now on net 5V: C11.1, C13.1, C15.1, C6.1, C8.1, P5.1, U1.8 (VCC), U3.8 (VCC), U4.8 (VCC), U6.8 (VCC), U7.8 (VCC)
- net 5V: now also C1.2, C17.2, C18.2, C19.2, C20.2, C21.2, P6.1, P7.1
- net DIV8_OUT: now also C5.1; no longer C14.1
- net GND: now also C10.2, C14.1, C7.2, C1.1, C17.1, C18.1, C19.1, C20.1, C21.1, C35.2, C36.2, C9.1, D3.1, R18.2; no longer C7.1
- net at U2.3 (OUT): now also C3.2; no longer C10.2
- net at R2.2: now also C22.2; no longer U2.5 (IN)
- net at U2.7 (~IN): now also C7.1; no longer C7.2
- net at U5.1 (INPUT): now also C3.1; no longer C10.1
- net at L1.2, U5.3 (OUT+VCC): now also C5.2; no longer C14.2
- net at L1.1, R5.1: now also C10.1, C14.2
- net at C4.1, R1.2, U1.3 (~CLK)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: now also C9.2
- new net: C36.1, D3.2, R18.1, R3.1
- new net: C22.1, C23.2, D3.3
- new net: C35.1, P8.1, R3.2
- new net: C23.1, U2.5 (IN)
Other:
- moved on the sheet: C11, C12, C13, C15, C16, C2, C4, C6, C8, L1, P1, P2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

Commit message: d
Parts:
- removed C2, C23: 1 nF, Capacitor_SMD:C_0402_1005Metric, symbol SparkFun-Capacitors:6PF-0402-50V-0.5%
- removed R2: PAT1220, 0xDBFB7:PAT1220, symbol 0xDBFB7:attenuator
- P2, P4: footprint Connector_PinHeader_2.54mm:PinHeader_1x01_P2.54mm_Vertical -> TestPoint:TestPoint_Pad_2.5x2.5mm
- P5, P7, P8: footprint TestPoint:TestPoint_Pad_1.5x1.5mm -> TestPoint:TestPoint_Pad_2.5x2.5mm
Connections:
- net GND: no longer D3.1
- net at C22.1, D3.3: now also U2.5 (IN)
- net at C22.2: now also P1.1
Other:
- moved on the sheet: P1
Changed lines of the file:
@@
 Input power range of the HMC. is max. +5 dBm across the spectrum, 0 dBm recommended.\n
-$Comp
-L 0xDBFB7:attenuator R2
-U 1 1 5F838885
-P 1900 2700
-F 0 "R2" H 1925 2915 50  0000 C CNN
-F 1 "PAT1220" H 1925 2824 50  0000 C CNN
-F 2 "0xDBFB7:PAT1220" H 1900 2700 50  0001 C CNN
-F 3 "" H 1900 2700 50  0001 C CNN
-F 4 "-10 dBm" H 1925 2733 50  0000 C CNN "Field4"
-	1    1900 2700
-	1    0    0    -1
-$EndComp
 $Comp
 L 0xDBFB7:SKY65013 U5
@@
 	1    0    0    -1
 $EndComp
-$Comp
-L power:GND #PWR0103
-U 1 1 5F842A34
-P 1700 2950
-F 0 "#PWR0103" H 1700 2950 30  0001 C CNN
-F 1 "GND" H 1700 2880 30  0001 C CNN
-F 2 "" H 1700 2950 50  0001 C CNN
-F 3 "" H 1700 2950 50  0001 C CNN
-	1    1700 2950
-	0    1    1    0
-$EndComp
-Wire Wire Line
-	6150 2900 6300 2900
 Text Notes 1250 4000 0    50   ~ 0
 O/P is -9 to -6 dBm, too low for the logic levels of the \nSY.
@@
 L conn:CONN_1 P1
 U 1 1 5F844EAC
-P 600 2800
-F 0 "P1" H 533 2703 40  0000 C CNN
-F 1 "CONN_1" H 550 2840 30  0001 C CNN
-F 2 "TestPoint:TestPoint_Pad_1.0x1.0mm" H 600 2800 50  0001 C CNN
-F 3 "" H 600 2800 50  0001 C CNN
-	1    600  2800
+P 1500 2800
+F 0 "P1" H 1433 2703 40  0000 C CNN
+F 1 "CONN_1" H 1450 2840 30  0001 C CNN
+F 2 "TestPoint:TestPoint_Pad_1.0x1.0mm" H 1500 2800 50  0001 C CNN
+F 3 "" H 1500 2800 50  0001 C CNN
+	1    1500 2800
 	-1   0    0    1
 $EndComp
-$Comp
-L SparkFun-Capacitors:6PF-0402-50V-0.5% C2
-U 1 1 5F84D039
-P 1350 2800
-F 0 "C2" V 1200 2850 45  0000 C CNN
-F 1 "1 nF" V 1116 2850 45  0000 C CNN
-F 2 "Capacitor_SMD:C_0402_1005Metric" H 1350 3050 20  0001 C CNN
-F 3 "" H 1350 2800 50  0001 C CNN
-F 4 "" V 1189 2850 60  0000 C CNN "Field4"
-	1    1350 2800
-	0    1    -1   0
-$EndComp
-Wire Wire Line
-	1700 2800 1550 2800
 $Comp
 L power:GND #PWR0104
@@
 	0    1    1    0
 $EndComp
-Wire Wire Line
-	750  2800 1250 2800
 $Comp
 L SparkFun-Resistors:0.22OHM-0805-1_4W-1% R4
@@
 F 0 "P2" H 9158 5250 40  0000 L CNN
 F 1 "OUTPUT" H 9050 5290 30  0001 C CNN
-F 2 "Connector_PinHeader_2.54mm:PinHeader_1x01_P2.54mm_Vertical" H 9100 5250 50  0001 C CNN
+F 2 "TestPoint:TestPoint_Pad_2.5x2.5mm" H 9100 5250 50  0001 C CNN
 F 3 "" H 9100 5250 50  0001 C CNN
 	1    9100 5250
@@
 F 0 "P4" V 8932 6309 40  0000 L CNN
 F 1 "OUTPUT" H 8950 6290 30  0001 C CNN
-F 2 "Connector_PinHeader_2.54mm:PinHeader_1x01_P2.54mm_Vertical" H 9000 6250 50  0001 C CNN
+F 2 "TestPoint:TestPoint_Pad_2.5x2.5mm" H 9000 6250 50  0001 C CNN
 F 3 "" H 9000 6250 50  0001 C CNN
 	1    9000 6250
@@
 	1    0    0    -1
 $EndComp
-Wire Wire Line
-	4900 2900 5850 2900
 $Comp
 L SparkFun-Capacitors:6PF-0402-50V-0.5% C3
@@
 F 0 "P7" H 7283 2003 40  0000 C CNN
 F 1 "CONN_1" H 7300 2140 30  0001 C CNN
-F 2 "TestPoint:TestPoint_Pad_1.5x1.5mm" H 7350 2100 50  0001 C CNN
+F 2 "TestPoint:TestPoint_Pad_2.5x2.5mm" H 7350 2100 50  0001 C CNN
 F 3 "" H 7350 2100 50  0001 C CNN
 	1    7350 2100
@@
 F 0 "P5" H 3083 5903 40  0000 C CNN
 F 1 "CONN_1" H 3100 6040 30  0001 C CNN
-F 2 "TestPoint:TestPoint_Pad_1.5x1.5mm" H 3150 6000 50  0001 C CNN
+F 2 "TestPoint:TestPoint_Pad_2.5x2.5mm" H 3150 6000 50  0001 C CNN
 F 3 "" H 3150 6000 50  0001 C CNN
 	1    3150 6000
@@
 F 0 "P8" H 2933 -47 40  0000 C CNN
 F 1 "a" H 2950 90  30  0001 C CNN
-F 2 "TestPoint:TestPoint_Pad_1.5x1.5mm" H 3000 50  50  0001 C CNN
+F 2 "TestPoint:TestPoint_Pad_2.5x2.5mm" H 3000 50  50  0001 C CNN
 F 3 "" H 3000 50  50  0001 C CNN
 	1    3000 50
@@
 Wire Wire Line
 	3000 200  3000 500
-$Comp
-L power:GND #PWR0138
-U 1 1 5F4843B8
-P 3000 2400
-F 0 "#PWR0138" H 3000 2400 30  0001 C CNN
-F 1 "GND" H 3000 2330 30  0001 C CNN
-F 2 "" H 3000 2400 50  0001 C CNN
-F 3 "" H 3000 2400 50  0001 C CNN
-	1    3000 2400
-	1    0    0    -1
-$EndComp
 $Comp
 L SparkFun-Capacitors:6PF-0402-50V-0.5% C22
@@
 $EndComp
 $Comp
-L SparkFun-Capacitors:6PF-0402-50V-0.5% C23
-U 1 1 5F6850C4
-P 3300 2800
-F 0 "C23" V 3150 2850 45  0000 C CNN
-F 1 "1 nF" V 3066 2850 45  0000 C CNN
-F 2 "Capacitor_SMD:C_0402_1005Metric" H 3300 3050 20  0001 C CNN
-F 3 "" H 3300 2800 50  0001 C CNN
-F 4 "" V 3139 2850 60  0000 C CNN "Field4"
-	1    3300 2800
-	0    1    -1   0
-$EndComp
-Connection ~ 3200 2800
-Wire Wire Line
-	3500 2800 4100 2800
-Wire Wire Line
-	2150 2800 2900 2800
-$Comp
 L SparkFun-Resistors:RESISTOR0402 R3
 U 1 1 5F6D38E6
@@
 	0    -1   -1   0
 $EndComp
+Wire Wire Line
+	1650 2800 2900 2800
+Wire Wire Line
+	3200 2800 4100 2800
+Connection ~ 3200 2800
+Wire Wire Line
+	4900 2900 5850 2900
+Wire Wire Line
+	6150 2900 6300 2900
 $EndSCHEMATC
