File: electronics/kicad/integrated_amp/integrated_amp.sch (KiCad schematic (older format))
At the start: 1 part

Commit message: Protocol
Parts:
- removed U?: MCP3422, Package_SO:SOIC-8_3.9x4.9mm_P1.27mm, symbol Analog_ADC:MCP3422
- added C1, C13, C21, C3, C5, C8, C9: 0.1 uF, 0603, symbol SparkFun-Capacitors:0.1UF-0603-25V-5%
- added C10, C12, C20, C4, C7: 2.2 uF, 0603, symbol SparkFun-Capacitors:0.1UF-0603-25V-5%
- added C11, C16, C19, C24, C25: 1 nF, Capacitor_SMD:C_0402_1005Metric, symbol SparkFun-Capacitors:6PF-0402-50V-0.5%
- added C14, C15: 1 nF, Resistor_SMD:R_0402_1005Metric, symbol SparkFun-Capacitors:6PF-0402-50V-0.5%
- added C17, C22: 1 nF, Capacitor_SMD:C_0603_1608Metric, symbol SparkFun-Capacitors:6PF-0402-50V-0.5%
- added C18, C23, C6: 1 nF, Capacitor_SMD:C_0603_1005Metric, symbol SparkFun-Capacitors:6PF-0402-50V-0.5%
- added C2: 10uF, 1206, symbol SparkFun-Capacitors:1.0UF-1206-50V-10%
- added D1: BAT15-04, Package_TO_SOT_SMD:SOT-323_SC-70, symbol Diode:BAS40-04
- added D2: LED, symbol Device:LED
- added J1: CONN_01, 1X01, symbol SparkFun-Connectors:CONN_01
- added J13: CONN_02, 1X02, symbol SparkFun-Connectors:CONN_02
- added J2: PDSE1, Connectors2:1X04_SMD_RA_FEMALE, symbol w_connectors:HEADER_4
- added P1: a, TestPoint:TestPoint_Pad_1.5x1.5mm, symbol conn:CONN_1
- added Q1, Q2: DMP3099L, Package_TO_SOT_SMD:SOT-23, symbol Transistor_FET:BSS84
- added R1, R3, R7: 10k, Resistor_SMD:R_0603_1608Metric, symbol SparkFun-Resistors:RESISTOR0402
- added R10, R11, R13, R14, R15, R2, R4, R6: 1k, Resistor_SMD:R_0603_1608Metric, symbol SparkFun-Resistors:RESISTOR0402
- added R12: 330, Resistor_SMD:R_0603_1608Metric, symbol SparkFun-Resistors:RESISTOR0402
- added R16, R17: 4.7k, Resistor_SMD:R_0603_1608Metric, symbol SparkFun-Resistors:RESISTOR0402
- added R5: 0.1r, 0805, symbol SparkFun-Resistors:0.75OHM-0805-1_4W-1%
- added R8, R9: 10k, Resistor_SMD:R_0402_1005Metric, symbol SparkFun-Resistors:RESISTOR0402
- added U1: LM7805, digikey-footprints:SOT-223, symbol dk_PMIC-Voltage-Regulators-Linear:LM7812CT_LTB
- added U10: HMC732, Package_DFN_QFN:QFN-24-1EP_4x4mm_P0.5mm_EP2.6x2.6mm, symbol 0xDBFB7:HMC732
- added U11: HMC996, symbol 0xDBFB7:HMC996
- added U12: TSL2571FN, Silicon-Standard:DFN-6-2X2, symbol 0xDBFB7:TSL2571FN
- added U13: MAX4915, Package_TO_SOT_SMD:SOT-23-5_HandSoldering, symbol 0xDBFB7:MAX4915
- added U14, U16, U6: MCP4725SOT-23, SOT23-6, symbol SparkFun-IC-Conversion:MCP4725SOT-23
- added U15: TS912IDT, Package_SO:SOIC-8_3.9x4.9mm_P1.27mm, symbol SparkFun-IC-Amplifiers:LM358
- added U17, U18: 74HC595, symbol 74xx:74HC595
- added U19: CD74HC4067M, Package_SO:SOIC-24W_7.5x15.4mm_P1.27mm, symbol 74xx:CD74HC4067M
- added U2: ADS1115IDGS, snapeda:IC_ADS1115IRUGR, symbol Analog_ADC:ADS1115IDGS
- added U20, U9: MCP1416T-E_OT, digikey-footprints:SOT-753, symbol dk_PMIC-Gate-Drivers:MCP1416T-E_OT
- added U3: BA78M20FP, digikey-footprints:TO-252-3, symbol dk_PMIC-Voltage-Regulators-Linear:MC7805BDTRKG
- added U4: NCP1117-3.3_TO252, Package_TO_SOT_SMD:TO-252-2, symbol Regulator_Linear:NCP1117-3.3_TO252
- added U5: LM2776, Package_TO_SOT_SMD:SOT-23-6, symbol Regulator_SwitchedCapacitor:LM2776
- added U7: TLV2172IDR, Package_SO:SOIC-8_3.9x4.9mm_P1.27mm, symbol SparkFun-IC-Amplifiers:LM358
- added U8: INA194, Package_TO_SOT_SMD:SOT-23-5, symbol Amplifier_Current:INA194
Connections:
- net labels added: -5V, 12V, 20V, 24V, 3.3V, 5V, AMP_DRAIN_SUPPLY, AMP_GAIN_CONTROL, AMP_GATE_CONTROL, GAIN_DAC_I2C_SELECT, GATE_DAC_I2C_SELECT, GND, SCL, SDA, TUNING_DAC_I2C_SELECT, VCO_POWER, Vtune, current_sense_output, ~AMP_DRAIN_CONTROL, ~VCO_POWER_CONTROL
- wire segments 0 -> 51
Other:
- note added: ""Application Notes_Bias and RF Sequencing for GaN and LDMOS RF Power Devices",\n"Remark: Power devices are particularly\nunstable at low drain voltages. This is the\nreason why [the device must be in] pinch-off when Vds is lower than\n the recommended operating Vds value""
- note added: "Because \n- the diode detector output is so close to the RF trace, \n- the far-end output has to travel parallel to the trace,\n- and filtering might affect the RF impedance\nit helps to digitize the output immediately; hence the ADCs.\n\nAlso, since initial impedance measurements have to be taken with a\n low-power signal so as to not destroy the virus, the programmable-gain amp also helps a lot."
- note added: "I2c multiplexer see https://electronics.stackexchange.com/a/392155/25599"
- note added: "The SDA pin could be used for the LED, LED as pullup, through the 4076. 4067 resistance is 200 ohms, however. \nTeensy setSCL(), setSDA(); needed because 17 and 16 do 20 mA."
- note added: "see https://www.analog.com/en/app-notes/an-1363.html\n"

Commit message: Simple absorption/reflection calc
Parts:
- removed D2: LED, symbol Device:LED
- removed R12: 330, Resistor_SMD:R_0603_1608Metric, symbol SparkFun-Resistors:RESISTOR0402
- removed R8: 10k, Resistor_SMD:R_0402_1005Metric, symbol SparkFun-Resistors:RESISTOR0402
- removed U12: TSL2571FN, Silicon-Standard:DFN-6-2X2, symbol 0xDBFB7:TSL2571FN
- removed U17, U18: 74HC595, symbol 74xx:74HC595
- removed U19: CD74HC4067M, Package_SO:SOIC-24W_7.5x15.4mm_P1.27mm, symbol 74xx:CD74HC4067M
- added C26: 1 nF, Capacitor_SMD:C_0603_1608Metric, symbol SparkFun-Capacitors:6PF-0402-50V-0.5%
- added C27: 1 nF, Capacitor_SMD:C_0603_1005Metric, symbol SparkFun-Capacitors:6PF-0402-50V-0.5%
- added C28, C29: 1 nF, Capacitor_SMD:C_0402_1005Metric, symbol SparkFun-Capacitors:6PF-0402-50V-0.5%
- added J3: Conn_01x04, Connector_PinHeader_2.54mm:PinHeader_1x04_P2.54mm_Vertical_SMD_Pin1Left, symbol Connector_Generic:Conn_01x04
- C18, C6: footprint Capacitor_SMD:C_0603_1005Metric -> Capacitor_SMD:C_0603_1608Metric
- U11: footprint (none) -> Package_DFN_QFN:QFN-24-1EP_4x4mm_P0.5mm_EP2.6x2.6mm
Connections:
- wire segments 51 -> 55
Other:
- note removed: "The SDA pin could be used for the LED, LED as pullup, through the 4076. 4067 resistance is 200 ohms, however. \nTeensy setSCL(), setSDA(); needed because 17 and 16 do 20 mA."
- moved on the sheet: C14, C15, D1, J13, P1, R16, R17, R9, U2

Commit message: Integrated amp progress
Parts:
- removed C23: 1 nF, Capacitor_SMD:C_0603_1005Metric, symbol SparkFun-Capacitors:6PF-0402-50V-0.5%
- removed C6: 1 nF, Capacitor_SMD:C_0603_1608Metric, symbol SparkFun-Capacitors:6PF-0402-50V-0.5%
- added C30, C31, C34: 0.1 uF, Capacitor_SMD:C_0603_1608Metric, symbol SparkFun-Capacitors:6PF-0402-50V-0.5%
- added C36, C38, C40, C41: 1 nF, Capacitor_SMD:C_0402_1005Metric, symbol SparkFun-Capacitors:6PF-0402-50V-0.5%
- added C42, C43, C44, C45, C48: 1 nF, Resistor_SMD:R_0402_1005Metric, symbol SparkFun-Capacitors:6PF-0402-50V-0.5%
- added C49, C50, C53, C55, C57: 2.2 uF, 0603, symbol SparkFun-Capacitors:0.1UF-0603-25V-5%
- added C51, C52: 1 nF, Capacitor_SMD:C_0603_1608Metric, symbol SparkFun-Capacitors:6PF-0402-50V-0.5%
- added C54, C56: 0.1 uF, 0603, symbol SparkFun-Capacitors:0.1UF-0603-25V-5%
- added D2, D3: BAT15-04, Package_TO_SOT_SMD:SOT-323_SC-70, symbol Diode:BAS40-04
- added J4: CONN_02, Connectors2:1X04_SMD_RA_FEMALE, symbol SparkFun-Connectors:CONN_04
- added JP1, JP3, JP4, JP5: Jumper, 0xDBFB7:JUMPER_5102, symbol Device:Jumper
- added JP2: Jumper, symbol Device:Jumper
- added P2: CONN_1, TestPoint:TestPoint_Pad_2.5x2.5mm, symbol conn:CONN_1
- added P3: CONN_1, Connector_PinHeader_2.54mm:PinHeader_1x02_P2.54mm_Vertical_SMD_Pin1Left, symbol conn:CONN_1
- added P4, P5: CONN_6, Connectors2:1X06-SMD_RA_MALE, symbol conn:CONN_6
- added R12, R18, R23, R24, R8: 10k, Resistor_SMD:R_0402_1005Metric, symbol SparkFun-Resistors:RESISTOR0402
- added R21: attenuator, 0xDBFB7:PAT1220, symbol 0xDBFB7:attenuator
- added R22: 50r, 0805, symbol SparkFun-Resistors:RESISTOR0805
- added U12: ADS1115IDGS, snapeda:IC_ADS1115IRUGR, symbol Analog_ADC:ADS1115IDGS
- added U17: HMC363, Package_SO:SOIC-8_3.9x4.9mm_P1.27mm, symbol 0xDBFB7:HMC363
- J13: footprint 1X02 -> Connectors2:1X04_SMD_RA_FEMALE; symbol SparkFun-Connectors:CONN_02 -> SparkFun-Connectors:CONN_04
- P1: value a -> CONN_1; footprint TestPoint:TestPoint_Pad_1.5x1.5mm -> TestPoint:TestPoint_Pad_1.0x1.0mm
Connections:
- net labels added: AMP_DRAIN_CONTROL_, AMP_GAIN_CONTROL_, AMP_GATE_CONTROL_, VCO_POWER_CONTROL_
- wire segments 55 -> 87
Other:
- moved on the sheet: C14, C15, C16, C8, C9, D1, R15, R5, R6, R7, R9, U10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

Commit message: Penetration depth
Parts:
- removed C1, C21, C3, C54: 0.1 uF, 0603, symbol SparkFun-Capacitors:0.1UF-0603-25V-5%
- removed C12, C20, C7: 2.2 uF, 0603, symbol SparkFun-Capacitors:0.1UF-0603-25V-5%
- removed C2: 10uF, 1206, symbol SparkFun-Capacitors:1.0UF-1206-50V-10%
- removed J1: CONN_01, 1X01, symbol SparkFun-Connectors:CONN_01
- removed J13, J4: CONN_02, Connectors2:1X04_SMD_RA_FEMALE, symbol SparkFun-Connectors:CONN_04
- removed J2: PDSE1, Connectors2:1X04_SMD_RA_FEMALE, symbol w_connectors:HEADER_4
- removed J3: Conn_01x04, Connector_PinHeader_2.54mm:PinHeader_1x04_P2.54mm_Vertical_SMD_Pin1Left, symbol Connector_Generic:Conn_01x04
- removed JP2: Jumper, symbol Device:Jumper
- removed P2: CONN_1, TestPoint:TestPoint_Pad_2.5x2.5mm, symbol conn:CONN_1
- removed P3: CONN_1, Connector_PinHeader_2.54mm:PinHeader_1x02_P2.54mm_Vertical_SMD_Pin1Left, symbol conn:CONN_1
- removed R1, R3: 10k, Resistor_SMD:R_0603_1608Metric, symbol SparkFun-Resistors:RESISTOR0402
- removed R10, R11, R13, R14, R15, R2, R4, R6: 1k, Resistor_SMD:R_0603_1608Metric, symbol SparkFun-Resistors:RESISTOR0402
- removed R16, R17: 4.7k, Resistor_SMD:R_0603_1608Metric, symbol SparkFun-Resistors:RESISTOR0402
- removed R5: 0.1r, 0805, symbol SparkFun-Resistors:0.75OHM-0805-1_4W-1%
- removed U1: LM7805, digikey-footprints:SOT-223, symbol dk_PMIC-Voltage-Regulators-Linear:LM7812CT_LTB
- removed U14, U16, U6: MCP4725SOT-23, SOT23-6, symbol SparkFun-IC-Conversion:MCP4725SOT-23
- removed U15: TS912IDT, Package_SO:SOIC-8_3.9x4.9mm_P1.27mm, symbol SparkFun-IC-Amplifiers:LM358
- removed U20, U9: MCP1416T-E_OT, digikey-footprints:SOT-753, symbol dk_PMIC-Gate-Drivers:MCP1416T-E_OT
- removed U3: BA78M20FP, digikey-footprints:TO-252-3, symbol dk_PMIC-Voltage-Regulators-Linear:MC7805BDTRKG
- removed U4: NCP1117-3.3_TO252, Package_TO_SOT_SMD:TO-252-2, symbol Regulator_Linear:NCP1117-3.3_TO252
- removed U5: LM2776, Package_TO_SOT_SMD:SOT-23-6, symbol Regulator_SwitchedCapacitor:LM2776
- removed U7: TLV2172IDR, Package_SO:SOIC-8_3.9x4.9mm_P1.27mm, symbol SparkFun-IC-Amplifiers:LM358
- removed U8: INA194, Package_TO_SOT_SMD:SOT-23-5, symbol Amplifier_Current:INA194
Connections:
- net labels removed: -5V, 12V, 20V, 24V, GAIN_DAC_I2C_SELECT, GATE_DAC_I2C_SELECT, TUNING_DAC_I2C_SELECT, current_sense_output, ~AMP_DRAIN_CONTROL, ~VCO_POWER_CONTROL
- wire segments 87 -> 57
Other:
- moved on the sheet: C11, C17, C18, C19, C4, C5, Q1
