File: electronics/kicad/integrated_amp/integrated_amp.kicad_pcb (KiCad board)
At the start: 2 copper layers, 63 parts, among them J1 CONN_01, J13 CONN_02, J2 PDSE1, P1 a, Q1 DMP3099L, Q2 DMP3099L, U1 LM7805, U10 HMC732, U12 TSL2571FN, U13 MAX4915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

Commit message: Simple absorption/reflection calc
Parts:
- removed R12: 330, Resistor_SMD:R_0603_1608Metric
- removed R8: 10k, Resistor_SMD:R_0402_1005Metric
- removed U12: TSL2571FN, Silicon-Standard:DFN-6-2X2
- removed U19: CD74HC4067M, Package_SO:SOIC-24W_7.5x15.4mm_P1.27mm
- added C18: 1 nF, Capacitor_SMD:C_0603_1608Metric, F.Cu at (123.5, 114.7)
- added C26: 1 nF, Capacitor_SMD:C_0603_1608Metric, F.Cu at (124.8, 104.1)
- added C28: 1 nF, Capacitor_SMD:C_0402_1005Metric, F.Cu at (125.1, 105.7)
- added C29: 1 nF, Capacitor_SMD:C_0402_1005Metric, F.Cu at (126.1, 105.1)
- added C6: 1 nF, Capacitor_SMD:C_0603_1608Metric, F.Cu at (109.8, 110.9)
- added J3: Conn_01x04, Connector_PinHeader_2.54mm:PinHeader_1x04_P2.54mm_Vertical_SMD_Pin1Left, F.Cu at (143.6, 90.9)
- added U11: HMC996, Package_DFN_QFN:QFN-24-1EP_4x4mm_P0.5mm_EP2.6x2.6mm, F.Cu at (126.9, 109.0)
- moved U9 104.7 mm to (108.1, 119.5)
- moved C17 92.7 mm to (121.9, 113.6)
- moved C5 91.5 mm to (125.7, 118.1)
- moved C8 87.7 mm to (112.7, 91.5)
- moved C4 83.5 mm to (125.7, 119.5)
- moved C16 83.4 mm to (118.4, 109.7), turned to 90 degrees
- moved C10 80.9 mm to (117.6, 101.6), turned to 270 degrees
- moved C13 76.9 mm to (119.0, 101.6), turned to 270 degrees
- moved R5 76.7 mm to (115.5, 100.7)
- moved C19 75.7 mm to (123.2, 111.9), turned to 180 degrees
- moved C22 72.8 mm to (128.9, 104.1), turned to 180 degrees
- moved C24 71.4 mm to (127.7, 105.7)
- moved C25 71.4 mm to (128.6, 105.0)
- moved Q2 68.9 mm to (125.6, 101.8), turned to 270 degrees
- moved U13 67.3 mm to (122.1, 101.7)
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Connections:
- U13 pad 3: 5V -> Net-(C10-Pad1)
Routing:
- net Net-(C8-Pad2): track 10.3 -> 0.00 mm
- net AMP_DRAIN_SUPPLY: track 0.00 -> 7.22 mm
- net (no net): track 6.03 -> 0.00 mm
- net VCO_POWER: track 0.00 -> 3.96 mm
- net 5V: track 3.96 -> 0.00 mm
- net Net-(C16-Pad2): track 0.00 -> 2.38 mm
- net Net-(C11-Pad1): track 2.38 -> 0.00 mm
- net Net-(U10-Pad15): track 2.71 -> 1.18 mm
- net GND: track 0.00 -> 0.50 mm

Commit message: Integrated amp progress
Parts:
- removed C6: 1 nF, Capacitor_SMD:C_0603_1608Metric
- added C30: 0.1 uF, Capacitor_SMD:C_0603_1608Metric, F.Cu at (128.2, 117.1)
- added C31: 0.1 uF, Capacitor_SMD:C_0603_1608Metric, F.Cu at (124.7, 116.4)
- added C34: 0.1 uF, Capacitor_SMD:C_0603_1608Metric, F.Cu at (131.0, 116.7)
- added C36: 1 nF, Capacitor_SMD:C_0402_1005Metric, F.Cu at (127.1, 112.4)
- added C38: 1 nF, Capacitor_SMD:C_0402_1005Metric, F.Cu at (129.3, 112.4)
- added C40: 1 nF, Capacitor_SMD:C_0402_1005Metric, F.Cu at (126.2, 114.1)
- added C41: 1 nF, Capacitor_SMD:C_0402_1005Metric, F.Cu at (125.2, 112.3)
- added C42: 1 nF, Resistor_SMD:R_0402_1005Metric, F.Cu at (135.4, 111.4)
- added C43: 1 nF, Resistor_SMD:R_0402_1005Metric, F.Cu at (148.4, 109.2)
- added C44: 1 nF, Resistor_SMD:R_0402_1005Metric, F.Cu at (152.5, 111.4)
- added C45: 1 nF, Resistor_SMD:R_0402_1005Metric, F.Cu at (152.8, 109.2)
- added C48: 1 nF, Resistor_SMD:R_0402_1005Metric, F.Cu at (157.8, 109.2)
- added C49: 2.2 uF, Capacitors:0603, F.Cu at (128.5, 122.9)
- added C50: 2.2 uF, Capacitors:0603, F.Cu at (122.4, 119.5)
- added C51: 1 nF, Capacitor_SMD:C_0603_1608Metric, F.Cu at (158.8, 112.5)
- added C52: 1 nF, Capacitor_SMD:C_0603_1608Metric, F.Cu at (167.1, 107.9)
- added C53: 2.2 uF, Capacitors:0603, F.Cu at (167.0, 106.3)
- added C54: 0.1 uF, Capacitors:0603, F.Cu at (275.1, 70.1)
- added C55: 2.2 uF, Capacitors:0603, F.Cu at (275.1, 72.5)
- added C56: 0.1 uF, Capacitors:0603, F.Cu at (155.9, 113.0)
- added C57: 2.2 uF, Capacitors:0603, F.Cu at (157.8, 115.1)
- added D2: BAT15-04, Package_TO_SOT_SMD:SOT-323_SC-70, F.Cu at (136.8, 110.5)
- added D3: BAT15-04, Package_TO_SOT_SMD:SOT-323_SC-70, F.Cu at (150.6, 110.2)
- added J4: CONN_02, Connectors2:1X04_SMD_RA_FEMALE, F.Cu at (259.2, 82.3)
- added JP1: Jumper, 0xDBFB7:JUMPER_5102, F.Cu at (124.6, 120.3)
- added JP3: Jumper, 0xDBFB7:JUMPER_5102, F.Cu at (155.0, 117.7)
- added JP4: Jumper, 0xDBFB7:JUMPER_5102, F.Cu at (151.2, 117.8)
- added JP5: Jumper, 0xDBFB7:JUMPER_5102, F.Cu at (137.7, 118.3)
- added P2: CONN_1, TestPoint:TestPoint_Pad_2.5x2.5mm, F.Cu at (219.7, 105.4)
- added P3: CONN_1, Connector_PinHeader_2.54mm:PinHeader_1x02_P2.54mm_Vertical_SMD_Pin1Left, F.Cu at (246.6, 116.6)
- added P4: CONN_6, Connectors2:1X06-SMD_RA_MALE, F.Cu at (103.7, 106.7)
- added P5: CONN_6, Connectors2:1X06-SMD_RA_MALE, F.Cu at (103.7, 121.9)
- added R12: 10k, Resistor_SMD:R_0402_1005Metric, F.Cu at (133.5, 112.1)
- added R18: 10k, Resistor_SMD:R_0402_1005Metric, F.Cu at (152.5, 112.4)
- added R21: attenuator, 0xDBFB7:PAT1220, F.Cu at (154.6, 107.2)
- added R22: 50r, Capacitors:0805, F.Cu at (168.0, 114.0)
- added R23: 10k, Resistor_SMD:R_0402_1005Metric, F.Cu at (126.4, 123.0)
- added R24: 10k, Resistor_SMD:R_0402_1005Metric, F.Cu at (120.6, 120.3)
- added R8: 10k, Resistor_SMD:R_0402_1005Metric, F.Cu at (134.7, 112.1)
- added U12: ADS1115IDGS, snapeda:IC_ADS1115IRUGR, F.Cu at (152.9, 114.2)
- added U17: HMC363, Package_SO:SOIC-8_3.9x4.9mm_P1.27mm, F.Cu at (163.3, 111.1)
- J13: footprint Connectors2:1X02 -> Connectors2:1X04_SMD_RA_FEMALE
- P1: value a -> CONN_1; footprint TestPoint:TestPoint_Pad_1.5x1.5mm -> TestPoint:TestPoint_Pad_1.0x1.0mm
- moved R5 176.9 mm to (292.1, 110.5)
- moved U9 145.5 mm to (253.2, 108.7), turned to 270 degrees
- moved U16 114.6 mm to (305.3, 114.3)
- moved U6 106.1 mm to (308.6, 93.3)
- moved C2 106.1 mm to (303.7, 94.1)
- moved J13 106.1 mm to (276.7, 112.0)
- moved R10 106.1 mm to (300.3, 111.5)
- moved R4 106.1 mm to (301.1, 109.0)
- moved U3 106.1 mm to (262.1, 101.8)
- moved U7 106.1 mm to (293.5, 102.2)
- moved U8 106.1 mm to (292.2, 107.7)
- moved C20 106.1 mm to (304.6, 70.9)
- moved C21 106.1 mm to (299.1, 77.9)
- moved C7 106.1 mm to (294.8, 75.6)
- moved J1 106.1 mm to (312.3, 104.8)
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Connections:
- net Net-(Q1-Pad1) renamed VCO_POWER_CONTROL_
- net Net-(Q2-Pad1) renamed AMP_DRAIN_CONTROL_
- C10 pad 1: Net-(C10-Pad1) -> 5V
- C13 pad 1: Net-(C10-Pad1) -> 5V
- J13 pad 2: Net-(J13-Pad2) -> Net-(C14-Pad1)
- P1 pad 1: Net-(C14-Pad1) -> Net-(P1-Pad1)
- R13 pad 2: AMP_GATE_CONTROL -> Net-(R13-Pad2)
- R14 pad 2: AMP_GAIN_CONTROL -> Net-(R14-Pad2)
- R5 pad 2: Net-(C10-Pad1) -> Net-(R5-Pad2)
- U13 pad 1: Net-(C10-Pad1) -> 5V
- U13 pad 3: Net-(C10-Pad1) -> 5V
- U15 pad 1: AMP_GAIN_CONTROL -> Net-(R14-Pad2)
- U15 pad 7: AMP_GATE_CONTROL -> Net-(R13-Pad2)
- U2 pad 5: Net-(U2-Pad5) -> Net-(C14-Pad1)
- U8 pad 4: Net-(C10-Pad1) -> Net-(R5-Pad2)
Routing:
- net 5V: track 0.00 -> 109.5 mm
- net SCL: track 0.00 -> 78.6 mm
- net 3.3V: track 0.00 -> 71.1 mm
- net SDA: track 0.00 -> 56.7 mm
- net AMP_GATE_CONTROL: track 0.00 -> 23.8 mm
- net AMP_DRAIN_CONTROL_: track 0.00 -> 22.1 mm
- net AMP_DRAIN_SUPPLY: track 7.22 -> 26.2 mm
- net AMP_GAIN_CONTROL_: track 0.00 -> 18.2 mm
- net Net-(C15-Pad1): track 0.00 -> 13.1 mm
- net AMP_GAIN_CONTROL: track 0.00 -> 12.9 mm
- net AMP_GATE_CONTROL_: track 0.00 -> 12.4 mm
- net VCO_POWER_CONTROL_: track 0.00 -> 11.1 mm
- net Vtune: track 0.00 -> 6.51 mm
- net Net-(P1-Pad1): track 0.00 -> 5.89 mm
- net Net-(C44-Pad1): track 0.00 -> 4.22 mm, vias 0 -> 1
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
Commit message: Penetration depth
Parts:
- removed C1, C21, C3, C54: 0.1 uF, Capacitors:0603
- removed C12, C20, C55, C7: 2.2 uF, Capacitors:0603
- removed C2: 10uF, Capacitors:1206
- removed J1: CONN_01, Connectors2:1X01
- removed J13, J4: CONN_02, Connectors2:1X04_SMD_RA_FEMALE
- removed J2: PDSE1, Connectors2:1X04_SMD_RA_FEMALE
- removed J3: Conn_01x04, Connector_PinHeader_2.54mm:PinHeader_1x04_P2.54mm_Vertical_SMD_Pin1Left
- removed P2: CONN_1, TestPoint:TestPoint_Pad_2.5x2.5mm
- removed P3: CONN_1, Connector_PinHeader_2.54mm:PinHeader_1x02_P2.54mm_Vertical_SMD_Pin1Left
- removed R1, R3: 10k, Resistor_SMD:R_0603_1608Metric
- removed R10, R11, R13, R14, R15, R2, R4, R6: 1k, Resistor_SMD:R_0603_1608Metric
- removed R16, R17: 4.7k, Resistor_SMD:R_0603_1608Metric
- removed R5: 0.1r, Capacitors:0805
- removed U1: LM7805, digikey-footprints:SOT-223
- removed U14, U16, U6: MCP4725SOT-23, Silicon-Standard:SOT23-6
- removed U15: TS912IDT, Package_SO:SOIC-8_3.9x4.9mm_P1.27mm
- removed U20, U9: MCP1416T-E_OT, digikey-footprints:SOT-753
- removed U3: BA78M20FP, digikey-footprints:TO-252-3
- removed U4: NCP1117-3.3_TO252, Package_TO_SOT_SMD:TO-252-2
- removed U5: LM2776, Package_TO_SOT_SMD:SOT-23-6
- removed U7: TLV2172IDR, Package_SO:SOIC-8_3.9x4.9mm_P1.27mm
- removed U8: INA194, Package_TO_SOT_SMD:SOT-23-5
- moved P1 59.6 mm to (130.1, 152.9), turned to 270 degrees
- moved R22 54.2 mm to (126.6, 149.0), turned to 180 degrees
- moved C53 53.1 mm to (134.3, 148.1), turned to 270 degrees
- moved C52 52.9 mm to (132.7, 148.1), turned to 90 degrees
- moved U17 47.4 mm to (129.5, 144.4), turned to 90 degrees
- moved C51 41.0 mm to (128.1, 139.8), turned to 180 degrees
- moved P5 40.1 mm to (118.7, 84.7), turned to 180 degrees
- moved C57 40.1 mm to (125.5, 138.8), turned to 90 degrees
- moved C48 39.7 mm to (131.4, 138.9), turned to 90 degrees
- moved P4 37.4 mm to (133.9, 84.7), turned to 180 degrees
- moved C56 37.0 mm to (127.6, 136.9), turned to 270 degrees
- moved JP3 37.0 mm to (122.9, 136.0), turned to 180 degrees
- moved R21 35.4 mm to (133.4, 135.6), turned to 270 degrees
- moved U12 33.1 mm to (126.4, 134.0), turned to 180 degrees
- moved C45 32.6 mm to (131.4, 133.8), turned to 90 degrees
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Connections:
- R12 pad 2: Net-(C42-Pad1) -> Net-(R12-Pad2)
Routing:
- net Net-(C51-Pad1): track 0.00 -> 1.88 mm
Other:
- board outline added: 13.2 x 11.2 mm

Commit message: Amp built
Routing:
- net (no net): vias 4 -> 7
Other:
- board size 13.2 x 11.2 mm -> 32.7 x 30.2 mm
