File: electronics/kicad/integrated_amp_driver_2/integrated_amp_driver.kicad_pcb (KiCad board)
At the start: 2 copper layers, 35 parts, among them J1 CONN_04, J5 CONN_03, P1 CONN_6, P3 CONN_6, P4 CONN_6, P5 CONN_6, U1 LM7805, U14 MCP4725SOT-23, U15 TS912IDT, U16 MCP4725SOT-23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

Commit message: more garbage
Parts:
- removed C16: 10uF, Capacitors:1206
- removed C17: 0.1 uF, Capacitors:0603
- removed JP1: Jumper, 0xDBFB7:JUMPER_5102
- removed P1, P3, P4, P5: CONN_6, Connectors2:1X06-SMD_RA_MALE
- removed U1: LM7805, digikey-footprints:SOT-223
- added C1: 0.1 uF, Capacitors:0603, F.Cu at (228.7, 79.0)
- added C2: 0.1 uF, Capacitors:0603, F.Cu at (249.1, 82.4)
- added J10: CONN_02, Connector_PinHeader_2.54mm:PinHeader_1x02_P2.54mm_Vertical_SMD_Pin1Left, F.Cu at (225.8, 43.9)
- added J13: CONN_02, Connector_PinHeader_2.54mm:PinHeader_1x03_P2.54mm_Vertical_SMD_Pin1Left, F.Cu at (245.5, 45.2)
- added J14: CONN_02, Connector_PinHeader_2.54mm:PinHeader_1x03_P2.54mm_Vertical_SMD_Pin1Left, F.Cu at (226.3, 62.0)
- added J2: CONN_02, Connector_PinHeader_2.54mm:PinHeader_1x03_P2.54mm_Vertical_SMD_Pin1Left, F.Cu at (247.7, 75.0)
- added J3: CONN_02, Connector_PinHeader_2.54mm:PinHeader_1x03_P2.54mm_Vertical_SMD_Pin1Left, F.Cu at (220.1, 80.4)
- added J4: CONN_02, Connector_PinHeader_2.54mm:PinHeader_1x02_P2.54mm_Vertical_SMD_Pin1Left, F.Cu at (236.2, 74.9)
- added J6: CONN_02, Connector_PinHeader_2.54mm:PinHeader_1x03_P2.54mm_Vertical_SMD_Pin1Left, F.Cu at (238.3, 58.3)
- added J7: CONN_02, Connector_PinHeader_2.54mm:PinHeader_1x02_P2.54mm_Vertical_SMD_Pin1Left, F.Cu at (234.3, 43.9)
- added J8: CONN_02, Connector_PinHeader_2.54mm:PinHeader_1x02_P2.54mm_Vertical_SMD_Pin1Left, F.Cu at (238.8, 43.9)
- added J9: CONN_02, Connector_PinHeader_2.54mm:PinHeader_1x02_P2.54mm_Vertical_SMD_Pin1Left, F.Cu at (230.1, 43.9)
- J1: value CONN_04 -> CONN_02; footprint Connectors2:1X06-SMD-FEMALE -> Connector_PinHeader_2.54mm:PinHeader_1x02_P2.54mm_Vertical_SMD_Pin1Left
- J5: value CONN_03 -> CONN_02; footprint Connectors2:1X03_SMD_RA_MALE -> Connector_PinHeader_2.54mm:PinHeader_1x02_P2.54mm_Vertical_SMD_Pin1Left
- moved J5 136.1 mm to (248.7, 58.5), turned to 0 degrees
- moved C14 118.0 mm to (231.8, 54.2), turned to 0 degrees
- moved R17 117.1 mm to (238.9, 41.9), turned to 90 degrees
- moved U9 115.2 mm to (233.0, 56.7), turned to 270 degrees
- moved R16 114.9 mm to (238.9, 46.1), turned to 270 degrees
- moved R5 114.3 mm to (243.1, 56.9), turned to 180 degrees
- moved C12 114.0 mm to (239.4, 88.9), turned to 90 degrees
- moved C15 112.0 mm to (233.3, 59.3), turned to 0 degrees
- moved U8 110.7 mm to (243.2, 59.3), turned to 180 degrees
- moved U5 110.4 mm to (236.3, 89.4), turned to 0 degrees
- moved C21 108.5 mm to (236.1, 87.0), turned to 0 degrees
- moved C13 108.5 mm to (240.5, 78.0), turned to 90 degrees
- moved U20 108.1 mm to (233.0, 61.8), turned to 270 degrees
- moved C20 107.7 mm to (236.1, 85.4), turned to 0 degrees
- moved C7 106.9 mm to (233.4, 90.0), turned to 90 degrees
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Connections:
- J1 pad 1: GND -> 5V
- J1 pad 2: 5V -> GND
- J5 pad 1: GND -> 5V
- J5 pad 2: 12V -> GND
Routing:
- net GND: track 9.56 -> 94.9 mm
- net 5V: track 151.8 -> 105.1 mm
- net TUNING_DAC_I2C_SELECT: track 27.0 -> 0.00 mm, vias 1 -> 0
- net 3.3V: track 30.7 -> 54.7 mm
- net Vtune: track 23.5 -> 0.00 mm
- net current_sense_output: track 34.9 -> 24.6 mm
- net 12V: track 7.86 -> 0.00 mm
- net AMP_GAIN_CONTROL_: track 16.6 -> 8.77 mm
- net AMP_GATE_CONTROL_: track 14.9 -> 8.03 mm
- net GAIN_DAC_I2C_SELECT: track 7.88 -> 3.29 mm, vias 2 -> 0
- net SCL: track 29.6 -> 26.4 mm, vias 3 -> 0
- net SDA: track 31.2 -> 28.2 mm, vias 3 -> 0
- net ~VCO_POWER_CONTROL: track 7.30 -> 9.88 mm, vias 2 -> 0
- net GATE_DAC_I2C_SELECT: track 3.86 -> 1.89 mm, vias 1 -> 0
- net ~AMP_DRAIN_CONTROL: track 8.18 -> 9.51 mm, vias 2 -> 0
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Other:
- board outline added: 73.7 x 92.1 mm
