File: electronics/kicad/integrated_amp_driver_2/integrated_amp_driver.sch (KiCad schematic (older format))
At the start: 35 parts, among them J1 CONN_04, J5 CONN_03, P1 CONN_6, P3 CONN_6, P4 CONN_6, P5 CONN_6, U1 LM7805, U14 MCP4725SOT-23, U15 TS912IDT, U16 MCP4725SOT-23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

Commit message: more garbage
Parts:
- removed C16: 10uF, 1206, symbol SparkFun-Capacitors:1.0UF-1206-50V-10%
- removed C17: 0.1 uF, 0603, symbol SparkFun-Capacitors:0.1UF-0603-25V-5%
- removed J1: CONN_04, Connectors2:1X06-SMD-FEMALE, symbol conn:CONN_6
- removed J5: CONN_03, Connectors2:1X03_SMD_RA_MALE, symbol SparkFun-Connectors:CONN_03
- removed JP1: Jumper, 0xDBFB7:JUMPER_5102, symbol Device:Jumper
- removed P1, P3, P4, P5: CONN_6, Connectors2:1X06-SMD_RA_MALE, symbol conn:CONN_6
- removed U1: LM7805, digikey-footprints:SOT-223, symbol dk_PMIC-Voltage-Regulators-Linear:LM7812CT_LTB
- added C1, C2: 0.1 uF, 0603, symbol SparkFun-Capacitors:0.1UF-0603-25V-5%
- added J1, J10, J11, J12, J15, J16, J17, J18, J4, J5, J7, J8, J9: CONN_02, Connector_PinHeader_2.54mm:PinHeader_1x02_P2.54mm_Vertical_SMD_Pin1Left, symbol SparkFun-Connectors:CONN_02
- added J13, J14, J2, J3, J6: CONN_02, Connector_PinHeader_2.54mm:PinHeader_1x03_P2.54mm_Vertical_SMD_Pin1Left, symbol conn:CONN_3
Connections:
- net 3.3V: now also J13.1 (P1)
- net 5V: now also C1.1, C2.1, J1.1, J15.1, J16.1, J17.1, J18.1, J5.1
- net AMP_DRAIN_CONTROL_: now also J6.3 (P3)
- net AMP_DRAIN_SUPPLY: now also J6.2 (PM)
- net AMP_GAIN_CONTROL_: now also J4.1
- net AMP_GATE_CONTROL_: now also J4.2
- net GAIN_DAC_I2C_SELECT: now also J3.1 (P1)
- net GATE_DAC_I2C_SELECT: now also J2.1 (P1)
- net GND: now also C1.2, C2.2, J1.2, J15.2, J16.2, J17.2, J18.2, J5.2
- net SCL: now also J10.1, J11.1, J12.1, J13.2 (PM), J2.2 (PM), J3.2 (PM), J7.1, J8.1, J9.1
- net SDA: now also J10.2, J11.2, J12.2, J13.3 (P3), J2.3 (P3), J3.3 (P3), J7.2, J8.2, J9.2
- net VCO_POWER_CONTROL_: now also J6.1 (P1)
- net current_sense_output: now also J14.3 (P3)
- net ~AMP_DRAIN_CONTROL: now also J14.2 (PM)
- net ~VCO_POWER_CONTROL: now also J14.1 (P1)
Other:
- moved on the sheet: C11, C13, C14, C15, R15, R16, R17, R5, R6, U20, U8, U9
