File: electronics/kicad/turbidimeter/LED_segment.sch (KiCad schematic (older format))
At the start: 2 parts

Commit message: turbidimeter
Changed lines of the file:
@@
 $Descr A4 11693 8268
 encoding utf-8
-Sheet 2 33
+Sheet 6 17
 Title ""
 Date ""
@@
 AR Path="/5FC2BBFC/5FC1DAB1" Ref="R15"  Part="1"
 AR Path="/5FC2BBFF/5FC1DAB1" Ref="R16"  Part="1"
-F 0 "R16" V 3205 4068 45  0000 L CNN
+F 0 "R5" V 3205 4068 45  0000 L CNN
 F 1 "330" V 3289 4068 45  0000 L CNN
 F 2 "Resistor_SMD:R_0603_1608Metric" H 3300 4150 20  0001 C CNN
@@
 AR Path="/5FC2BBFC/5FC1FCC6" Ref="#PWR0117"  Part="1"
 AR Path="/5FC2BBFF/5FC1FCC6" Ref="#PWR0118"  Part="1"
-F 0 "#PWR0118" H 3300 4200 30  0001 C CNN
+F 0 "#PWR0107" H 3300 4200 30  0001 C CNN
 F 1 "GND" H 3300 4130 30  0001 C CNN
 F 2 "" H 3300 4200 50  0001 C CNN
@@
 AR Path="/5FC2BBFC/5FC32F33" Ref="D15"  Part="1"
 AR Path="/5FC2BBFF/5FC32F33" Ref="D16"  Part="1"
-F 0 "D16" H 3378 3592 45  0000 L CNN
+F 0 "D5" H 3378 3592 45  0000 L CNN
 F 1 "LED-GREEN1206-BOTTOM" H 3378 3508 45  0000 L CNN
 F 2 "LED-1206-BOTTOM" V 3100 3600 20  0001 C CNN
