File: electronics/kicad/horizontal_sweep_gen/horizontal_sweep_gen.sch (KiCad schematic (older format))
At the start: 2 parts

Commit message: pdftex
Parts:
- added C? (x4): 0.1 uF, Capacitor_SMD:C_0603_1608Metric, symbol SparkFun-Capacitors:0.1UF-KIT-EZ-50V-20%
- added C?: 50 pF, Capacitor_SMD:C_1206_3216Metric, symbol SparkFun-Capacitors:0.1UF-KIT-EZ-50V-20%
- added D? (x2): D_TVS, Diode_SMD:D_SMA, symbol Device:D_TVS
- added J?: TEENSY, Connectors2:1X03_SMD_RA_MALE, symbol w_connectors:HEADER_3
- added J?: TESTPOINT, symbol w_connectors:HEADER_2
- added J?: DEFLECTION, Connectors2:1X03_SMD_RA_MALE, symbol w_connectors:HEADER_3
- added J?: CONN_08SMD-MALE, 1X08_SMD_MALE, symbol SparkFun-Connectors:CONN_08SMD-MALE
- added Q3: BSS84, Package_TO_SOT_SMD:SOT-23, symbol Transistor_FET:BSS84
- added R4, R? (x2): 100k, Resistor_SMD:R_2512_6332Metric, symbol SparkFun-Resistors:RESISTOR1206
- added U?: DS1100Z-500, SOIC127P600X175-8N, symbol 0xDBFB7:DS1100Z-500
- added U?: MCP1416T-E_OT, digikey-footprints:SOT-753, symbol dk_PMIC-Gate-Drivers:MCP1416T-E_OT
- Q?: footprint (none) -> Connectors2:1X03_SMD_RA_MALE
Connections:
- net TRIG: now reaches U?.1 (IN)
- net TRIG: now also J?.2, U?.1 (IN)
- net GND: now reaches U?.14 (*P/S)
- net GND: now also Q?.S, U?.8 (GND), C?.2, C?.2, C?.2, C?.2, C?.2, D?.1 (A1), D?.2 (A2), J?.1, R?.2, U?.4 (GND), U?.4 (GND)
- net SWEEP_TRIGGER: now reaches U?.15 (OUT/*OUT)
- net SWEEP_TRIGGER: now also U?.3 (IN)
- net 5V: now reaches U?.16 (VCC)
- net 5V: now also U?.2 (LE), C?.1, C?.1, J?.3, U?.8 (VCC)
- net SWEEP: now reaches Q?.D
- net SWEEP: now also J?.1, J?.2, J?.3, R4.2
- net at Q?.G: now also Q3.3 (D)
- new net: D?.1 (A1), Q3.1 (G), U?.5 (OUT)
- new net 12V: C?.1, U?.2 (VDD)
- new net HV: C?.1, R4.1, R?.1
- new net HV_CENTER: J?.1, J?.2, R?.1, R?.2
- new net P0: J?.1
- new net P1: J?.2
- new net P2: J?.3
- new net P3: J?.4
- new net P4: J?.5
- new net P5: J?.6
- new net P6: J?.7
- new net PULSE_TRIGGER: U?.2 (TAP2)
- new net VSWEEP_SLOPE: C?.1, D?.2 (A2), Q3.2 (S)
Other:
- note added: "coax"
- note added: "ramp generator based on Baker and Johnson"
- moved on the sheet: Q?, U?
