File: electronics/kicad/delay_line/delay_line.kicad_pcb (KiCad board)
At the start: 2 copper layers, 13 parts, among them J1 TEENSY, J2 TEENSY, P1 CONN_2, U1 DS1023S-50, U2 DS1100Z-500, U3 MCP1416T-E_OT, U4 74AHC1G00, U5 74AHC1G08, U6 MCP1416T-E_OT

Commit message: Delay line functioning great
Parts:
- added C4: 0.1UF-0603-25V-5%, Capacitors:0603, F.Cu at (112.1, 102.4)
- added R1: 50 ohm, Capacitors:0805, F.Cu at (111.2, 100.0)
Routing:
- net Net-(C4-Pad2): track 0.00 -> 12.2 mm
- net Net-(C4-Pad1): track 24.6 -> 13.8 mm
- net COAX: track 13.9 -> 15.4 mm
